File: can_board/can_board.kicad_pcb (KiCad board)
At the start: 2 copper layers, 20.1 x 20.3 mm, 8 parts, among them J1 Conn_01x06_Male, U1 SN65HVD230

Commit message: added jlc string to canboard
Other:
- board text added: "JLCJLCJLCJLC"
Changed lines of the file:
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@@
   )
   (gr_rect (start 136.271 113.095) (end 156.337 133.415) (layer "Edge.Cuts") (width 0.1) (fill none))
+  (gr_text "JLCJLCJLCJLC" (at 147.828 129.54) (layer "B.SilkS")
+    (effects (font (size 1.5 1.5) (thickness 0.3)) (justify mirror))
+  )
   (gr_text "SDM CAN\nBoard v1.0" (at 147.447 118.683) (layer "B.SilkS")
     (effects (font (size 1.5 1.5) (thickness 0.3)) (justify mirror))
