File: yaw_probe_stm32/yaw_probe_stm32.kicad_pcb (KiCad board)
At the start: 2 copper layers, 58.4 x 73.7 mm, 40 parts, among them J1 CONN_CAN, J2 Conn_01x04_Male, J3 USB_B_Micro, SW1 SW_SPDT, U1 STM32F072C8Tx, U2 SN65HVD230_CAN_Transceiver, U3 AMS1117-3.3, U4 MS4525DO, U5 MS4525DO, Y1 16MHz

Commit message: imu box
Parts:
- moved R1 2.68 mm to (162.2, 69.0)
Changed lines of the file:
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@@
   )
   (footprint "Resistor_SMD:R_0402_1005Metric" (layer "F.Cu")
-    (at 162.269 66.316)
+    (at 162.25 69)
     (descr "Resistor SMD 0402 (1005 Metric), square (rectangular) end terminal, IPC_7351 nominal, (Body size source: IPC-SM-782 page 72, https://www.pcb-3d.com/wordpress/wp-content/uploads/ipc-sm-782a_amendment_1_and_2.pdf), generated with kicad-footprint-generator")
     (tags "resistor")
