File: sdm23main/sdm23main.kicad_sch (KiCad schematic)
At the start: 14 parts, among them J1 Haltech_CAN, J2 AES_CAN, J3 AES_CAN, J4 AES_CAN, J5 AES_CAN, J6 AES_CAN, U1 Teensy4.1, U2 Haltech Transceiver, U3 AES Transceiver, U4 Pololu_5V_2.5A_SD_Regulator

Commit message: initial draft for main board sdm23
Parts:
- added U5: GPS_ADA746, Connector_PinSocket_2.54mm:PinSocket_1x09_P2.54mm_Vertical, symbol SDM:GPS_ADA746
Connections:
- net GND: now also U5.7 (GND)
- net +3V3: now reaches U1.15 (3V3)
- net +3V3: now also U5.8 (VIN)
- net TX6: now reaches U1.16 (24_A10_TX6_SCL2)
- net TX6: now also U5.6 (RX)
- net RX6: now reaches U1.17 (25_A11_RX6_SDA2)
- net RX6: now also U5.5 (TX)
- no-connect marks 60 -> 62
Other:
- note added: "5V Regulator"
- note added: "AES CAN Bus"
- note added: "GPS Module"
- note added: "Haltech CAN Bus"
- note added: "Mounting Holes"
- note added: "Teensy 4.1"
- moved on the sheet: H1, H2, H3, H4, J2, J3, J4, J5, J6, U1, U4

Commit message: sdm23main: rearranging layout
Connections:
- net RX7: now reaches U1.20 (28_RX7)
- net RX7: now also U5.5 (TX)
- net TX7: now reaches U1.21 (29_TX7)
- net TX7: now also U5.6 (RX)
- net RX6: no longer names the net of U1.17 (25_A11_RX6_SDA2)
- net RX6: no longer U5.5 (TX)
- net TX6: no longer names the net of U1.16 (24_A10_TX6_SCL2)
- net TX6: no longer U5.6 (RX)
Changed lines of the file:
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@@
   (no_connect (at 132.08 130.81))
   (no_connect (at 187.96 99.06))
-  (no_connect (at 132.08 111.76))
   (no_connect (at 187.96 86.36))
   (no_connect (at 187.96 83.82))
@@
   (no_connect (at 132.08 78.74))
   (no_connect (at 187.96 138.43))
+  (no_connect (at 132.08 99.06))
+  (no_connect (at 132.08 101.6))
   (no_connect (at 187.96 101.6))
   (no_connect (at 132.08 86.36))
@@
   (no_connect (at 187.96 106.68))
   (no_connect (at 187.96 119.38))
-  (no_connect (at 132.08 109.22))
   (no_connect (at 132.08 127))
   (no_connect (at 240.03 91.44))
@@
     (stroke (width 0) (type default) (color 0 0 0 0))
   )
+  (wire (pts (xy 124.46 109.22) (xy 132.08 109.22))
+    (stroke (width 0) (type default) (color 0 0 0 0))
+  )
   (wire (pts (xy 62.23 132.08) (xy 72.39 132.08))
     (stroke (width 0) (type default) (color 0 0 0 0))
@@
     (stroke (width 0) (type default) (color 0 0 0 0))
   )
-  (wire (pts (xy 124.46 99.06) (xy 132.08 99.06))
-    (stroke (width 0) (type default) (color 0 0 0 0))
-  )
   (polyline (pts (xy 24.13 198.12) (xy 107.95 198.12))
     (stroke (width 0) (type default) (color 0 0 0 0))
@@
     (stroke (width 0) (type default) (color 0 0 0 0))
   )
+  (wire (pts (xy 124.46 111.76) (xy 132.08 111.76))
+    (stroke (width 0) (type default) (color 0 0 0 0))
+  )
   (wire (pts (xy 203.2 63.5) (xy 203.2 67.31))
     (stroke (width 0) (type default) (color 0 0 0 0))
@@
     (stroke (width 0) (type default) (color 0 0 0 0))
   )
-  (wire (pts (xy 124.46 101.6) (xy 132.08 101.6))
-    (stroke (width 0) (type default) (color 0 0 0 0))
-  )
   (wire (pts (xy 43.18 123.19) (xy 45.72 123.19))
     (stroke (width 0) (type default) (color 0 0 0 0))
@@
     (effects (font (size 1.27 1.27)) (justify left bottom))
   )
-  (label "TX6" (at 124.46 99.06 0)
+  (label "TX7" (at 124.46 111.76 0)
     (effects (font (size 1.27 1.27)) (justify left bottom))
   )
@@
     (effects (font (size 1.27 1.27)) (justify left bottom))
   )
-  (label "TX6" (at 219.71 99.06 0)
+  (label "TX7" (at 219.71 99.06 0)
     (effects (font (size 1.27 1.27)) (justify left bottom))
   )
@@
     (effects (font (size 1.27 1.27)) (justify left bottom))
   )
-  (label "RX6" (at 124.46 101.6 0)
-    (effects (font (size 1.27 1.27)) (justify left bottom))
-  )
-  (label "RX6" (at 242.57 96.52 0)
-    (effects (font (size 1.27 1.27)) (justify left bottom))
-  )
+  (label "RX7" (at 124.46 109.22 0)
+    (effects (font (size 1.27 1.27)) (justify left bottom))
+  )
+  (label "RX7" (at 242.57 96.52 0)
+    (effects (font (size 1.27 1.27)) (justify left bottom))
+  )

Commit message: uploading yaw probe draft
Parts:
- added D1: GREEN, LED_THT:LED_D5.0mm, symbol Device:LED
- added J7: Conn_01x06_Female, Connector_PinSocket_2.00mm:PinSocket_1x06_P2.00mm_Vertical, symbol Connector:Conn_01x06_Female
- added R1: R, Resistor_THT:R_Axial_DIN0204_L3.6mm_D1.6mm_P7.62mm_Horizontal, symbol Device:R
- J2, J3, J4, J5, J6: value AES_CAN -> DAQ_CAN
- U2: footprint Connector_PinSocket_2.54mm:PinSocket_1x06_P2.54mm_Vertical -> SDM:SDM_CANBoard_v1
- U3: value AES Transceiver -> DAQ Transceiver; footprint Connector_PinSocket_2.54mm:PinSocket_1x06_P2.54mm_Vertical -> SDM:SDM_CANBoard_v1
Connections:
- net +3.3V: now also U3.3 (3V3), J7.1 (Pin_1); no longer U2.1 (3V3), U3.1 (3V3)
- net +3V3: now also U2.3 (3V3)
- net +5V: now also R1.1
- net CRX1: now also U3.4 (CRX); no longer U2.4 (CRX)
- net CTX1: now also U3.1 (CTX); no longer U2.3 (CTX)
- net GND: now also D1.1 (K), J7.6 (Pin_6)
- net CRX2: now reaches U1.2 (0_RX1_CRX2_CS1)
- net CRX2: now also U2.4 (CRX)
- net CTX2: now reaches U1.3 (1_TX1_CTX2_MISO1)
- net CTX2: now also U2.1 (CTX)
- net A0: now reaches U1.36 (14_A0_TX3_SPDIF_OUT)
- net A0: now also J7.5 (Pin_5)
- net A1: now reaches U1.37 (15_A1_RX3_SPDIF_IN)
- net A1: now also J7.4 (Pin_4)
- net SCL1: now reaches U1.38 (16_A2_RX4_SCL1)
- net SCL1: now also J7.3 (Pin_3)
- net SDA1: now reaches U1.39 (17_A3_TX4_SDA1)
- net SDA1: now also J7.2 (Pin_2)
- net AES_CANH renamed DAQ_CANH
- net AES_CANL renamed DAQ_CANL
- net CRX3: no longer names the net of U1.22 (30_CRX3)
- net CRX3: no longer U3.4 (CRX)
- net CTX3: no longer names the net of U1.23 (31_CTX3)
- net CTX3: no longer U3.3 (CTX)
- net HALTECH_CANH renamed HALTECH_CAN+
- net HALTECH_CANL renamed HALTECH_CAN-
- new net: D1.2 (A), R1.2
- no-connect marks 62 -> 58
Other:
- note added: "DAQ CAN Bus"
- note added: "Extra Connectors"
- note removed: "AES CAN Bus"
- moved on the sheet: H1, H2, H3, H4, U5

Commit message: imu box
Parts:
- removed J7: Conn_01x06_Female, Connector_PinSocket_2.00mm:PinSocket_1x06_P2.00mm_Vertical, symbol Connector:Conn_01x06_Female
- added J7: Conn_01x08_Female, Connector_PinSocket_2.54mm:PinSocket_1x08_P2.54mm_Vertical, symbol Connector:Conn_01x08_Female
- U4: footprint Connector_PinSocket_2.54mm:PinSocket_1x05_P2.54mm_Vertical -> Connector_PinHeader_2.54mm:PinHeader_1x05_P2.54mm_Vertical
- U5: footprint Connector_PinSocket_2.54mm:PinSocket_1x09_P2.54mm_Vertical -> Connector_PinHeader_2.54mm:PinHeader_1x09_P2.54mm_Vertical
Connections:
- net +3.3V: now also J7.1 (Pin_1)
- net A0: now also J7.7 (Pin_7)
- net A1: now also J7.6 (Pin_6)
- net GND: now also J7.8 (Pin_8)
- net SCL1: now also J7.5 (Pin_5)
- net SDA1: now also J7.4 (Pin_4)
- net SDA0: now reaches U1.40 (18_A4_SDA)
- net SDA0: now also J7.3 (Pin_3)
- net SCL0: now reaches U1.41 (19_A5_SCL)
- net SCL0: now also J7.2 (Pin_2)
- net HALTECH_CAN+ renamed HALTECH_CANH
- net HALTECH_CAN- renamed HALTECH_CANL
- no-connect marks 58 -> 56
Other:
- moved on the sheet: H1, H2, H3, H4

Commit message: silkscreen additions
Other:
- company: Sun Devil Motorsports -> Sun Devil Motorsports - Data Acquisition
Changed lines of the file:
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@@
   (title_block
     (title "SDM-23 DAQ Main Board")
-    (date "2022-11-05")
+    (date "2023-01-11")
     (rev "v1")
-    (company "Sun Devil Motorsports")
+    (company "Sun Devil Motorsports - Data Acquisition")
   )
   (junction (at 54.61 115.57) (diameter 0) (color 0 0 0 0)

Commit message: start sg amplifier
Other:
- company: Sun Devil Motorsports - Data Acquisition -> (none)
Changed lines of the file:
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@@
     (date "2023-01-11")
     (rev "v1")
-    (company "Sun Devil Motorsports - Data Acquisition")
   )
   (junction (at 54.61 115.57) (diameter 0) (color 0 0 0 0)

Commit message: various improvements
Parts:
- added C1: 0.33uF, Capacitor_THT:C_Disc_D3.0mm_W2.0mm_P2.50mm, symbol Device:C_Small
- added C2: 0.1uF, Capacitor_THT:C_Disc_D3.0mm_W2.0mm_P2.50mm, symbol Device:C_Small
- added U6: L78L05_TO92, Package_TO_SOT_THT:TO-220-3_Vertical, symbol Regulator_Linear:L78L05_TO92
- J7: value Conn_01x08_Female -> Extra Pinouts
- R1: value R -> 330
Connections:
- net +5V: now also C2.2, U6.1 (VO)
- net GND: now also C1.2, C2.1, U6.2 (GND)
- net VCC: now also C1.1, U6.3 (VI)
Other:
- note removed: "Extra Connectors"
- moved on the sheet: J7, U4

Commit message: sent JLC order
Parts:
- added R2: 10k, Resistor_THT:R_Axial_DIN0204_L3.6mm_D1.6mm_P7.62mm_Horizontal, symbol Device:R
- added SW1: Button, TerminalBlock_TE-Connectivity:TerminalBlock_TE_282834-2_1x02_P2.54mm_Horizontal, symbol Switch:SW_Push
Connections:
- net +3.3V: now also SW1.2
- net GND: now also R2.1
- net BUTTON: now reaches U1.25 (33_MCLK2)
- net BUTTON: now also R2.2, SW1.1
- no-connect marks 56 -> 55
Other:
- note added: "Backup regulator"
Changed lines of the file:
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@@
   (title_block
     (title "SDM-23 DAQ Main Board")
-    (date "2023-01-22")
+    (date "2023-01-25")
     (rev "v1")
   )
@@
   )
   (junction (at 81.28 36.83) (diameter 0) (color 0 0 0 0)
+  )
+  (junction (at 207.01 115.57) (diameter 0) (color 0 0 0 0)
   )
   (junction (at 199.39 66.04) (diameter 0) (color 0 0 0 0)
@@
   (no_connect (at 132.08 93.98))
   (no_connect (at 132.08 124.46))
-  (no_connect (at 187.96 119.38))
   (no_connect (at 152.4 148.59))
   (no_connect (at 187.96 73.66))
@@
     (stroke (width 0) (type default) (color 0 0 0 0))
   )
+  (wire (pts (xy 199.39 119.38) (xy 199.39 115.57))
+    (stroke (width 0) (type default) (color 0 0 0 0))
+  )
   (wire (pts (xy 187.96 63.5) (xy 203.2 63.5))
     (stroke (width 0) (type default) (color 0 0 0 0))
@@
     (stroke (width 0) (type default) (color 0 0 0 0))
   )
+  (wire (pts (xy 207.01 115.57) (xy 207.01 116.84))
+    (stroke (width 0) (type default) (color 0 0 0 0))
+  )
   (wire (pts (xy 124.46 63.5) (xy 132.08 63.5))
     (stroke (width 0) (type default) (color 0 0 0 0))
@@
     (stroke (width 0) (type default) (color 0 0 0 0))
   )
+  (wire (pts (xy 199.39 115.57) (xy 207.01 115.57))
+    (stroke (width 0) (type default) (color 0 0 0 0))
+  )
   (wire (pts (xy 187.96 86.36) (xy 200.66 86.36))
     (stroke (width 0) (type default) (color 0 0 0 0))
@@
     (stroke (width 0) (type default) (color 0 0 0 0))
   )
+  (wire (pts (xy 207.01 115.57) (xy 207.01 113.03))
+    (stroke (width 0) (type default) (color 0 0 0 0))
+  )
   (wire (pts (xy 187.96 68.58) (xy 191.77 68.58))
     (stroke (width 0) (type default) (color 0 0 0 0))
   )
+  (wire (pts (xy 207.01 124.46) (xy 207.01 129.54))
+    (stroke (width 0) (type default) (color 0 0 0 0))
+  )
   (wire (pts (xy 96.52 133.35) (xy 101.6 133.35))
     (stroke (width 0) (type default) (color 0 0 0 0))
@@
     (stroke (width 0) (type default) (color 0 0 0 0))
   )
+  (wire (pts (xy 187.96 119.38) (xy 199.39 119.38))
+    (stroke (width 0) (type default) (color 0 0 0 0))
+  )
   (wire (pts (xy 43.18 148.59) (xy 53.34 148.59))
     (stroke (width 0) (type default) (color 0 0 0 0))
@@
     (stroke (width 0) (type default) (color 0 0 0 0))
   )
+  (wire (pts (xy 212.09 100.33) (xy 212.09 97.79))
+    (stroke (width 0) (type default) (color 0 0 0 0))
+  )
   (polyline (pts (xy 237.49 148.59) (xy 257.81 148.59))
     (stroke (width 0) (type default) (color 0 0 0 0))
@@
     (stroke (width 0) (type default) (color 0 0 0 0))
   )
+  (wire (pts (xy 207.01 100.33) (xy 207.01 102.87))
+    (stroke (width 0) (type default) (color 0 0 0 0))
+  )
   (wire (pts (xy 81.28 34.29) (xy 81.28 36.83))
     (stroke (width 0) (type default) (color 0 0 0 0))
@@
     (stroke (width 0) (type default) (color 0 0 0 0))
   )
+  (wire (pts (xy 207.01 100.33) (xy 212.09 100.33))
+    (stroke (width 0) (type default) (color 0 0 0 0))
+  )
   (polyline (pts (xy 107.95 105.41) (xy 107.95 198.12))
     (stroke (width 0) (type default) (color 0 0 0 0))
@@
   )
   (text "5V Regulator" (at 87.63 54.61 0)
+    (effects (font (size 1.27 1.27)) (justify left bottom))
+  )
+  (text "Backup regulator" (at 30.48 24.13 0)
     (effects (font (size 1.27 1.27)) (justify left bottom))
   )
@@
   (label "SDA0" (at 193.04 81.28 0)
     (effects (font (size 1.27 1.27)) (justify left bottom))
+  )
+  (label "BUTTON" (at 194.31 119.38 0)
+    (effects (font (size 0.64 0.64)) (justify left bottom))
   )
   (label "CRX2" (at 91.44 78.74 0)
@@
     (pin "5")
     (pin "6")
+  )
+  (symbol (lib_id "power:GND") (at 207.01 129.54 0) (unit 1)
+    (in_bom yes) (on_board yes) (fields_autoplaced)
+    (property "Reference" "#PWR0123" (id 0) (at 207.01 135.89 0)
+      (effects (font (size 1.27 1.27)) hide)
+    )
+    (property "Value" "GND" (id 1) (at 207.01 134.62 0))
+    (property "Footprint" "" (id 2) (at 207.01 129.54 0)
+      (effects (font (size 1.27 1.27)) hide)
+    )
+    (property "Datasheet" "" (id 3) (at 207.01 129.54 0)
+      (effects (font (size 1.27 1.27)) hide)
+    )
+    (pin "1")
   )
   (symbol (lib_id "power:GND") (at 195.58 97.79 0) (unit 1)
@@
     (pin "4")
   )
+  (symbol (lib_id "Device:R") (at 207.01 120.65 180) (unit 1)
+    (in_bom yes) (on_board yes) (fields_autoplaced)
+    (property "Reference" "R2" (id 0) (at 209.55 119.3799 0)
+      (effects (font (size 1.27 1.27)) (justify right))
+    )
+    (property "Value" "10k" (id 1) (at 209.55 121.9199 0)
+      (effects (font (size 1.27 1.27)) (justify right))
+    )
+    (property "Footprint" "Resistor_THT:R_Axial_DIN0204_L3.6mm_D1.6mm_P7.62mm_Horizontal" (id 2) (at 208.788 120.65 90)
+      (effects (font (size 1.27 1.27)) hide)
+    )
+    (property "Datasheet" "~" (id 3) (at 207.01 120.65 0)
+      (effects (font (size 1.27 1.27)) hide)
+    )
+    (pin "1")
+    (pin "2")
+  )
   (symbol (lib_id "power:GND") (at 95.25 46.99 0) (unit 1)
     (in_bom yes) (on_board yes)
@@
     (pin "1")
   )
+  (symbol (lib_id "Switch:SW_Push") (at 207.01 107.95 90) (unit 1)
+    (in_bom yes) (on_board yes) (fields_autoplaced)
+    (property "Reference" "SW1" (id 0) (at 208.28 106.6799 90)
+      (effects (font (size 1.27 1.27)) (justify right))
+    )
+    (property "Value" "Button" (id 1) (at 208.28 109.2199 90)
+      (effects (font (size 1.27 1.27)) (justify right))
+    )
+    (property "Footprint" "TerminalBlock_TE-Connectivity:TerminalBlock_TE_282834-2_1x02_P2.54mm_Horizontal" (id 2) (at 201.93 107.95 0)
+      (effects (font (size 1.27 1.27)) hide)
+    )
+    (property "Datasheet" "~" (id 3) (at 201.93 107.95 0)
+      (effects (font (size 1.27 1.27)) hide)
+    )
+    (pin "1")
+    (pin "2")
+  )
   (symbol (lib_id "power:+5V") (at 54.61 113.03 0) (unit 1)
     (in_bom yes) (on_board yes) (fields_autoplaced)
@@
     )
     (property "Datasheet" "" (id 3) (at 81.28 34.29 0)
+      (effects (font (size 1.27 1.27)) hide)
+    )
+    (pin "1")
+  )
+  (symbol (lib_id "power:+3.3V") (at 212.09 97.79 0) (unit 1)
+    (in_bom yes) (on_board yes)
+    (property "Reference" "#PWR0124" (id 0) (at 212.09 101.6 0)
+      (effects (font (size 1.27 1.27)) hide)
+    )
+    (property "Value" "+3.3V" (id 1) (at 212.09 93.98 0))
+    (property "Footprint" "" (id 2) (at 212.09 97.79 0)
+      (effects (font (size 1.27 1.27)) hide)
+    )
+    (property "Datasheet" "" (id 3) (at 212.09 97.79 0)
       (effects (font (size 1.27 1.27)) hide)
     )
@@
       (reference "#PWR0122") (unit 1) (value "VCC") (footprint "")
     )
+    (path "/32601aac-5dc4-4263-bb64-859c4d5f5d81"
+      (reference "#PWR0123") (unit 1) (value "GND") (footprint "")
+    )
+    (path "/f135c5fa-ca14-4de7-a37f-a0aa5844d96f"
+      (reference "#PWR0124") (unit 1) (value "+3.3V") (footprint "")
+    )
     (path "/228c9f17-cdd8-444a-93b8-27bfd2de802a"
       (reference "C1") (unit 1) (value "0.33uF") (footprint "Capacitor_THT:C_Disc_D3.0mm_W2.0mm_P2.50mm")
@@
       (reference "R1") (unit 1) (value "330") (footprint "Resistor_THT:R_Axial_DIN0204_L3.6mm_D1.6mm_P7.62mm_Horizontal")
     )
+    (path "/825899bf-0b35-4d92-8eaf-078dfcc00dc8"
+      (reference "R2") (unit 1) (value "10k") (footprint "Resistor_THT:R_Axial_DIN0204_L3.6mm_D1.6mm_P7.62mm_Horizontal")
+    )
+    (path "/bd70d64f-4a95-45d9-8eff-d44066989b2b"
+      (reference "SW1") (unit 1) (value "Button") (footprint "TerminalBlock_TE-Connectivity:TerminalBlock_TE_282834-2_1x02_P2.54mm_Horizontal")
+    )
     (path "/3e12ac96-45d2-4d0f-97aa-6fd800466c2b"
