File: sdm24logger/memory.kicad_sch (KiCad schematic)
At the start: 5 parts, among them J1 Molex_47219-2001, U6 M24128-BRDW6TP, U7 ST_EMIF06-MSD02N16

Commit message: updating repo
Parts:
- removed J1: Molex_47219-2001, Library:Molex_uSD-47219-2001, symbol Connector:Micro_SD_Card
- added J3: Molex_1040310811, symbol Connector:Micro_SD_Card_Det2
Connections:
- net +3.3V: now also U7.16 (RDATA_VCC), J3.4 (VDD)
- net GND: now also J3.11 (SHIELD), J3.6 (VSS); no longer U7.2 (RDAT3_GND)
- net at U7.14 (DAT2_EX): now also J3.1 (DAT2)
- net at U7.13 (DAT3_EX): now also J3.2 (DAT3/CD)
- net at U7.12 (CMD_EX): now also J3.3 (CMD)
- net at U7.11 (CLK_EX): now also J3.5 (CLK)
- net at U7.10 (DAT0_EX): now also J3.7 (DAT0)
- net at U7.9 (DAT1_EX): now also J3.8 (DAT1)
- net CD: now reaches U7.1 (WP/CD)
- net CD: now also J3.10 (DET_A), J3.9 (DET_B)
- no-connect marks 2 -> 1
Changed lines of the file:
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@@
   (title_block
     (title "SDM-24 Data Logger")
-    (date "2023-06-11")
+    (date "2023-07-30")
     (rev "v1")
     (company "Sun Devil Motorsports")
@@
   (junction (at 134.62 113.03) (diameter 0) (color 0 0 0 0)
   )
+  (junction (at 140.97 88.9) (diameter 0) (color 0 0 0 0)
+  )
   (junction (at 134.62 111.76) (diameter 0) (color 0 0 0 0)
   )
@@
   (junction (at 138.43 53.34) (diameter 0) (color 0 0 0 0)
   )
+  (junction (at 138.43 60.96) (diameter 0) (color 0 0 0 0)
+  )
   (junction (at 140.97 86.36) (diameter 0) (color 0 0 0 0)
   )
-  (junction (at 140.97 87.63) (diameter 0) (color 0 0 0 0)
-  )
-  (junction (at 118.11 86.36) (diameter 0) (color 0 0 0 0)
-  )
   (junction (at 121.92 123.19) (diameter 0) (color 0 0 0 0)
   )
-  (no_connect (at 104.14 58.42))
-  (no_connect (at 137.16 60.96))
+  (junction (at 143.51 81.28) (diameter 0) (color 0 0 0 0)
+  )
+  (no_connect (at 104.14 60.96))
+  (wire (pts (xy 189.23 82.55) (xy 189.23 88.9))
+    (stroke (width 0) (type default))
+  )
   (wire (pts (xy 134.62 111.76) (xy 134.62 113.03))
     (stroke (width 0) (type default))
@@
     (stroke (width 0) (type default))
   )
-  (wire (pts (xy 104.14 60.96) (xy 102.87 60.96))
-    (stroke (width 0) (type default))
-  )
-  (wire (pts (xy 186.69 82.55) (xy 190.5 82.55))
+  (wire (pts (xy 138.43 60.96) (xy 138.43 53.34))
+    (stroke (width 0) (type default))
+  )
+  (wire (pts (xy 186.69 82.55) (xy 189.23 82.55))
     (stroke (width 0) (type default))
   )
@@
     (stroke (width 0) (type default))
   )
+  (wire (pts (xy 143.51 80.01) (xy 143.51 81.28))
+    (stroke (width 0) (type default))
+  )
   (wire (pts (xy 137.16 76.2) (xy 139.7 76.2))
     (stroke (width 0) (type default))
@@
     (stroke (width 0) (type default))
   )
+  (wire (pts (xy 140.97 88.9) (xy 140.97 91.44))
+    (stroke (width 0) (type default))
+  )
   (wire (pts (xy 148.59 114.3) (xy 148.59 111.76))
     (stroke (width 0) (type default))
@@
     (stroke (width 0) (type default))
   )
-  (wire (pts (xy 138.43 67.31) (xy 138.43 53.34))
+  (wire (pts (xy 138.43 67.31) (xy 138.43 60.96))
     (stroke (width 0) (type default))
   )
@@
     (stroke (width 0) (type default))
   )
+  (wire (pts (xy 137.16 60.96) (xy 138.43 60.96))
+    (stroke (width 0) (type default))
+  )
   (wire (pts (xy 139.7 59.69) (xy 143.51 59.69))
     (stroke (width 0) (type default))
@@
     (stroke (width 0) (type default))
   )
-  (wire (pts (xy 140.97 86.36) (xy 140.97 87.63))
-    (stroke (width 0) (type default))
-  )
-  (wire (pts (xy 102.87 86.36) (xy 118.11 86.36))
+  (wire (pts (xy 140.97 86.36) (xy 140.97 88.9))
+    (stroke (width 0) (type default))
+  )
+  (wire (pts (xy 135.89 81.28) (xy 143.51 81.28))
     (stroke (width 0) (type default))
   )
@@
     (stroke (width 0) (type default))
   )
+  (wire (pts (xy 143.51 81.28) (xy 143.51 82.55))
+    (stroke (width 0) (type default))
+  )
   (wire (pts (xy 115.57 113.03) (xy 134.62 113.03))
     (stroke (width 0) (type default))
@@
     (stroke (width 0) (type default))
   )
-  (wire (pts (xy 190.5 82.55) (xy 190.5 87.63))
-    (stroke (width 0) (type default))
-  )
-  (wire (pts (xy 140.97 87.63) (xy 140.97 91.44))
-    (stroke (width 0) (type default))
-  )
   (wire (pts (xy 137.16 73.66) (xy 142.24 73.66))
     (stroke (width 0) (type default))
@@
     (stroke (width 0) (type default))
   )
+  (wire (pts (xy 101.6 58.42) (xy 104.14 58.42))
+    (stroke (width 0) (type default))
+  )
   (wire (pts (xy 140.97 72.39) (xy 140.97 86.36))
     (stroke (width 0) (type default))
@@
     (stroke (width 0) (type default))
   )
-  (wire (pts (xy 102.87 60.96) (xy 102.87 86.36))
-    (stroke (width 0) (type default))
-  )
   (wire (pts (xy 132.08 134.62) (xy 132.08 135.89))
     (stroke (width 0) (type default))
@@
     (stroke (width 0) (type default))
   )
-  (wire (pts (xy 190.5 87.63) (xy 140.97 87.63))
+  (wire (pts (xy 189.23 88.9) (xy 140.97 88.9))
     (stroke (width 0) (type default))
   )
@@
   )
   (text "TODO: \n~{WC} could be conn. to GND\n" (at 96.52 138.43 0)
+    (effects (font (size 1.27 1.27)) (justify left bottom))
+  )
+  (label "CD" (at 101.6 58.42 180) (fields_autoplaced)
+    (effects (font (size 1.27 1.27)) (justify right bottom))
+  )
+  (label "CD" (at 135.89 81.28 0) (fields_autoplaced)
     (effects (font (size 1.27 1.27)) (justify left bottom))
   )
@@
     )
   )
-  (symbol (lib_id "Connector:Micro_SD_Card") (at 166.37 67.31 0) (unit 1)
+  (symbol (lib_id "Connector:Micro_SD_Card_Det2") (at 166.37 69.85 0) (unit 1)
     (in_bom yes) (on_board yes) (dnp no) (fields_autoplaced)
-    (property "Reference" "J1" (at 167.005 49.53 0)
-      (effects (font (size 1.27 1.27)))
-    )
-    (property "Value" "Molex_47219-2001" (at 167.005 52.07 0)
-      (effects (font (size 1.27 1.27)))
-    )
-    (property "Footprint" "Library:Molex_uSD-47219-2001" (at 195.58 59.69 0)
-      (effects (font (size 1.27 1.27)) hide)
-    )
-    (property "Datasheet" "http://katalog.we-online.de/em/datasheet/693072010801.pdf" (at 166.37 67.31 0)
-      (effects (font (size 1.27 1.27)) hide)
-    )
-    (pin "1")
+    (property "Reference" "J3" (at 167.005 49.53 0)
+      (effects (font (size 1.27 1.27)))
+    )
+    (property "Value" "Molex_1040310811" (at 167.005 52.07 0)
+      (effects (font (size 1.27 1.27)))
+    )
+    (property "Footprint" "" (at 218.44 52.07 0)
+      (effects (font (size 1.27 1.27)) hide)
+    )
+    (property "Datasheet" "https://www.hirose.com/en/product/document?clcode=&productname=&series=DM3&documenttype=Catalog&lang=en&documentid=D49662_en" (at 168.91 67.31 0)
+      (effects (font (size 1.27 1.27)) hide)
+    )
+    (pin "1")
+    (pin "10")
+    (pin "11")
     (pin "2")
     (pin "3")
@@
       (project "sdm24logger"
         (path "/89b3ea44-cadd-4bd5-8c60-f45fe49f0b09/755989b5-01b1-4d90-aab7-caeafb9cb82b"
-          (reference "J1") (unit 1)
-        )
-      )
+          (reference "J3") (unit 1)
+        )
+      )

Commit message: adding updates
Parts:
- R12: renamed from R4; value R_Small -> 2.7k
- R13: renamed from R3; value R_Small -> 2.7k
- renumbered J3 to J1, U7 to U6, U6 to U7
Changed lines of the file:
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@@
   (title_block
     (title "SDM-24 Data Logger")
-    (date "2023-07-30")
+    (date "2023-09-07")
     (rev "v1")
     (company "Sun Devil Motorsports")
@@
     (effects (font (size 1.27 1.27)) (justify left bottom))
   )
-  (label "CD" (at 101.6 58.42 180) (fields_autoplaced)
-    (effects (font (size 1.27 1.27)) (justify right bottom))
-  )
-  (label "CD" (at 135.89 81.28 0) (fields_autoplaced)
-    (effects (font (size 1.27 1.27)) (justify left bottom))
+  (hierarchical_label "CD" (shape input) (at 101.6 58.42 180) (fields_autoplaced)
+    (effects (font (size 1.27 1.27)) (justify right))
   )
   (hierarchical_label "DAT1" (shape input) (at 100.33 76.2 180) (fields_autoplaced)
@@
     (effects (font (size 1.27 1.27)) (justify right))
   )
+  (hierarchical_label "CD" (shape input) (at 135.89 81.28 180) (fields_autoplaced)
+    (effects (font (size 1.27 1.27)) (justify right))
+  )
   (symbol (lib_id "power:+3.3V") (at 134.62 109.22 0) (unit 1)
     (in_bom yes) (on_board yes) (dnp no) (fields_autoplaced)
-    (property "Reference" "#PWR014" (at 134.62 113.03 0)
+    (property "Reference" "#PWR030" (at 134.62 113.03 0)
       (effects (font (size 1.27 1.27)) hide)
     )
@@
       (project "sdm24logger"
         (path "/89b3ea44-cadd-4bd5-8c60-f45fe49f0b09/755989b5-01b1-4d90-aab7-caeafb9cb82b"
-          (reference "#PWR014") (unit 1)
+          (reference "#PWR030") (unit 1)
         )
       )
@@
   (symbol (lib_id "Device:R_Small") (at 115.57 116.84 0) (mirror y) (unit 1)
     (in_bom yes) (on_board yes) (dnp no)
-    (property "Reference" "R4" (at 113.03 116.205 0)
+    (property "Reference" "R12" (at 113.03 116.205 0)
       (effects (font (size 1.27 1.27)) (justify left))
     )
-    (property "Value" "R_Small" (at 113.03 118.745 0)
+    (property "Value" "2.7k" (at 113.03 118.745 0)
       (effects (font (size 1.27 1.27)) (justify left))
     )
@@
       (project "sdm24logger"
         (path "/89b3ea44-cadd-4bd5-8c60-f45fe49f0b09/755989b5-01b1-4d90-aab7-caeafb9cb82b"
-          (reference "R4") (unit 1)
+          (reference "R12") (unit 1)
         )
       )
@@
   (symbol (lib_id "lib:ST_M24128-XX") (at 133.35 110.49 0) (unit 1)
     (in_bom yes) (on_board yes) (dnp no)
-    (property "Reference" "U6" (at 127 106.68 0)
+    (property "Reference" "U7" (at 127 106.68 0)
       (effects (font (size 1.27 1.27)))
     )
@@
       (project "sdm24logger"
         (path "/89b3ea44-cadd-4bd5-8c60-f45fe49f0b09/755989b5-01b1-4d90-aab7-caeafb9cb82b"
-          (reference "U6") (unit 1)
+          (reference "U7") (unit 1)
         )
       )
@@
   (symbol (lib_id "power:GND") (at 140.97 91.44 0) (unit 1)
     (in_bom yes) (on_board yes) (dnp no)
-    (property "Reference" "#PWR029" (at 140.97 97.79 0)
+    (property "Reference" "#PWR032" (at 140.97 97.79 0)
       (effects (font (size 1.27 1.27)) hide)
     )
@@
       (project "sdm24logger"
         (path "/89b3ea44-cadd-4bd5-8c60-f45fe49f0b09/755989b5-01b1-4d90-aab7-caeafb9cb82b"
-          (reference "#PWR029") (unit 1)
+          (reference "#PWR032") (unit 1)
         )
       )
@@
   (symbol (lib_id "power:+3.3V") (at 138.43 46.99 0) (unit 1)
     (in_bom yes) (on_board yes) (dnp no) (fields_autoplaced)
-    (property "Reference" "#PWR028" (at 138.43 50.8 0)
+    (property "Reference" "#PWR031" (at 138.43 50.8 0)
       (effects (font (size 1.27 1.27)) hide)
     )
@@
       (project "sdm24logger"
         (path "/89b3ea44-cadd-4bd5-8c60-f45fe49f0b09/755989b5-01b1-4d90-aab7-caeafb9cb82b"
-          (reference "#PWR028") (unit 1)
+          (reference "#PWR031") (unit 1)
         )
       )
@@
   (symbol (lib_id "Connector:Micro_SD_Card_Det2") (at 166.37 69.85 0) (unit 1)
     (in_bom yes) (on_board yes) (dnp no) (fields_autoplaced)
-    (property "Reference" "J3" (at 167.005 49.53 0)
+    (property "Reference" "J1" (at 167.005 49.53 0)
       (effects (font (size 1.27 1.27)))
     )
@@
       (project "sdm24logger"
         (path "/89b3ea44-cadd-4bd5-8c60-f45fe49f0b09/755989b5-01b1-4d90-aab7-caeafb9cb82b"
-          (reference "J3") (unit 1)
+          (reference "J1") (unit 1)
         )
       )
@@
   (symbol (lib_id "lib:ST_EMIF06-MSD02N16") (at 120.65 52.07 0) (unit 1)
     (in_bom yes) (on_board yes) (dnp no)
-    (property "Reference" "U7" (at 119.38 46.99 0)
+    (property "Reference" "U6" (at 119.38 46.99 0)
       (effects (font (size 1.27 1.27)) (justify left))
     )
@@
       (project "sdm24logger"
         (path "/89b3ea44-cadd-4bd5-8c60-f45fe49f0b09/755989b5-01b1-4d90-aab7-caeafb9cb82b"
-          (reference "U7") (unit 1)
+          (reference "U6") (unit 1)
         )
       )
@@
   (symbol (lib_id "Device:R_Small") (at 148.59 116.84 0) (unit 1)
     (in_bom yes) (on_board yes) (dnp no) (fields_autoplaced)
-    (property "Reference" "R3" (at 151.13 116.205 0)
+    (property "Reference" "R13" (at 151.13 116.205 0)
       (effects (font (size 1.27 1.27)) (justify left))
     )
-    (property "Value" "R_Small" (at 151.13 118.745 0)
+    (property "Value" "2.7k" (at 151.13 118.745 0)
       (effects (font (size 1.27 1.27)) (justify left))
     )
@@
       (project "sdm24logger"
         (path "/89b3ea44-cadd-4bd5-8c60-f45fe49f0b09/755989b5-01b1-4d90-aab7-caeafb9cb82b"
-          (reference "R3") (unit 1)
+          (reference "R13") (unit 1)
         )
       )
@@
   (symbol (lib_id "power:GND") (at 132.08 138.43 0) (unit 1)
     (in_bom yes) (on_board yes) (dnp no)
-    (property "Reference" "#PWR030" (at 132.08 144.78 0)
+    (property "Reference" "#PWR029" (at 132.08 144.78 0)
       (effects (font (size 1.27 1.27)) hide)
     )
@@
       (project "sdm24logger"
         (path "/89b3ea44-cadd-4bd5-8c60-f45fe49f0b09/755989b5-01b1-4d90-aab7-caeafb9cb82b"
-          (reference "#PWR030") (unit 1)
-        )
-      )
+          (reference "#PWR029") (unit 1)
+        )
+      )
