File: drs/drs.kicad_pcb (KiCad board)
At the start: 2 copper layers, 68.5 x 53.5 mm, 2 parts, among them U1 SN65HVD230

Commit message: more progress on drs box
Parts:
- added C1: 100nF, Capacitor_SMD:C_0603_1608Metric, F.Cu at (148.1, 86.6)
- added C2: 100nF, Capacitor_SMD:C_0603_1608Metric, F.Cu at (146.0, 86.6)
- added JP1: CAN, Connector_PinHeader_2.54mm:PinHeader_1x02_P2.54mm_Vertical, F.Cu at (134.3, 86.4)
- added R1: 10k, Resistor_SMD:R_1206_3216Metric, F.Cu at (139.7, 91.0)
- added R3: 120, Resistor_SMD:R_0603_1608Metric, F.Cu at (134.3, 91.3)
- moved U1 11.1 mm to (140.7, 86.6)
Connections:
- A1 pad D11: unconnected-(A1-PadD11) -> /SERVO_RIGHT
- A1 pad D2: unconnected-(A1-PadD2) -> /USR_LED
- A1 pad D4: unconnected-(A1-PadD4) -> /CTX_5V
- A1 pad D5: unconnected-(A1-PadD5) -> /CRX_5V
- A1 pad D7: unconnected-(A1-PadD7) -> /BTN_INPUT
- A1 pad D9: unconnected-(A1-PadD9) -> /SERVO_LEFT
- U1 pad 6: unconnected-(U1-CANL-Pad6) -> /CANL
- U1 pad 7: unconnected-(U1-CANH-Pad7) -> /CANH
Routing:
- added copper zone on B.Cu, net GND
Other:
- outline, holes or cut-outs redrawn
- board text added: "BUTTON"
- board text added: "CAN"
- board text added: "LEFT"
- board text added: "M3"
- board text added: "POWER"
- board text added: "RIGHT"
- board text added: "SERVO SIGNAL"
- board text added: "Sun Devil Motorsports SDM-24 DRS Board"

Commit message: found shifter for drs
Parts:
- added C3: 100nF, Capacitor_SMD:C_0402_1005Metric, F.Cu at (155.3, 89.8)
- added C4: 100nF, Capacitor_SMD:C_0402_1005Metric, F.Cu at (155.4, 96.8)
- added D1: GREEN, LED_SMD:LED_1206_3216Metric, F.Cu at (154.0, 103.2)
- added D2: ESDCAN, Package_TO_SOT_SMD:SOT-323_SC-70, F.Cu at (131.4, 94.7)
- added D3: RED, LED_SMD:LED_1206_3216Metric, F.Cu at (175.6, 82.3)
- added J1: POWER, Connector_JST:JST_XH_B2B-XH-AM_1x02_P2.50mm_Vertical, F.Cu at (160.5, 114.0)
- added J2: BUTTON, Connector_JST:JST_XH_B2B-XH-AM_1x02_P2.50mm_Vertical, F.Cu at (160.3, 83.8)
- added J3: CAN, Connector_JST:JST_XH_B3B-XH-AM_1x03_P2.50mm_Vertical, F.Cu at (124.9, 95.7)
- added J4: SERVO, Connector_JST:JST_XH_B2B-XH-AM_1x02_P2.50mm_Vertical, F.Cu at (150.5, 78.5)
- added JP2: Shield, Connector_PinHeader_2.54mm:PinHeader_1x02_P2.54mm_Vertical, F.Cu at (131.4, 87.8)
- added R2: 220, Resistor_SMD:R_0805_2012Metric, F.Cu at (159.3, 75.8)
- added R4: 220, Resistor_SMD:R_0805_2012Metric, F.Cu at (175.7, 77.5)
- added R5: 220, Resistor_SMD:R_0805_2012Metric, F.Cu at (158.8, 103.2)
- added U2: TXU0202, Package_SO:VSSOP-8_2.3x2mm_P0.5mm, F.Cu at (155.1, 93.1)
- C1, C2: footprint Capacitor_SMD:C_0603_1608Metric -> Capacitor_SMD:C_0402_1005Metric
- moved R1 7.83 mm to (140.4, 98.8), turned to -90 degrees
- moved U1 7.05 mm to (142.9, 93.3)
- moved R3 7.05 mm to (136.5, 98.0)
- moved JP1 7.05 mm to (136.5, 93.1)
- moved C2 6.94 mm to (147.8, 93.3)
- moved C1 6.81 mm to (149.3, 93.3)
Other:
- board text added: "120Ω"
- board text added: "5V"
- board text added: "CANH"
- board text added: "CANL"
- board text added: "GND"
- board text added: "INPUT"
- board text added: "SHIELD"
- board text added: "USER"
- board text added: "VIN 6-24V"

Commit message: start routing on logger
Parts:
- added JP3: PULLDOWN, Connector_PinHeader_2.54mm:PinHeader_1x03_P2.54mm_Vertical, F.Cu at (154.3, 82.7)
- added R6: 10k, Resistor_SMD:R_0805_2012Metric, F.Cu at (159.4, 75.7)
- moved D1 11.6 mm to (152.6, 114.7), turned to -90 degrees
- moved R5 9.13 mm to (152.6, 109.9), turned to 90 degrees
- moved J4 5.70 mm to (144.8, 77.8), turned to 0 degrees
- moved R2 2.40 mm to (159.4, 78.2)
- moved J2 1.35 mm to (160.3, 85.2)
- moved R3 1.12 mm to (136.5, 96.9)
- moved A1 0.57 mm to (114.9, 122.3)
- moved R1 0.57 mm to (140.8, 98.4)
- moved U1 0.57 mm to (143.3, 92.9)
- moved C1 0.57 mm to (149.7, 92.9)
- moved C2 0.57 mm to (148.2, 92.9)
- moved C4 0.41 mm to (155.3, 96.4), turned to 0 degrees
- moved R4 0.08 mm to (175.6, 77.5), turned to 90 degrees
Connections:
- J4 pad 1: /SERVO_LEFT -> /SERVO_RIGHT
- J4 pad 2: /SERVO_RIGHT -> /SERVO_LEFT
- R2 pad 2: GND -> /STRONG_PULLDOWN
Routing:
- net +5V: track 0.00 -> 61.8 mm
- net +3.3V: track 0.00 -> 40.5 mm
- net /CRX_5V: track 0.00 -> 30.2 mm, vias 0 -> 1
- net /CTX_5V: track 0.00 -> 28.8 mm, vias 0 -> 2
- net /CANH: track 0.00 -> 19.9 mm
- net /CANL: track 0.00 -> 18.5 mm
- net /CRX_3V3: track 0.00 -> 17.9 mm, vias 0 -> 2
- net GND: track 0.00 -> 13.2 mm, vias 0 -> 5
- net /BTN_INPUT: track 0.00 -> 11.3 mm
- net /CTX_3V3: track 0.00 -> 10.3 mm, vias 0 -> 2
- net /SERVO_LEFT: track 0.00 -> 10.0 mm
- net /SERVO_RIGHT: track 0.00 -> 7.93 mm
- net /SHIELD: track 0.00 -> 7.71 mm
- net /STRONG_PULLDOWN: track 0.00 -> 7.42 mm
- net /USR_LED: track 0.00 -> 5.99 mm
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Other:
- board text added: "STRONG"
- board text added: "WEAK"

Commit message: drs board
Parts:
- removed JP3: PULLDOWN, Connector_PinHeader_2.54mm:PinHeader_1x03_P2.54mm_Vertical
- removed the R2 at (159.4, 78.2)
- added D4: GG040205170N2P, Diode_SMD:D_0402_1005Metric, F.Cu at (159.8, 78.3)
- added D5: GG040205170N2P, Diode_SMD:D_0402_1005Metric, F.Cu at (148.8, 74.2)
- added D6: GG040205170N2P, Diode_SMD:D_0402_1005Metric, F.Cu at (153.8, 74.2)
- added G***: LOGO, LOGO, F.Cu at (130.4, 107.6)
- added REF**: KiCad-Logo2_5mm_SilkScreen, Symbol:KiCad-Logo2_5mm_SilkScreen, F.Cu at (118.9, 78.8)
- R1: renamed from R6; footprint Resistor_SMD:R_0805_2012Metric -> Resistor_SMD:R_1206_3216Metric
- moved JP1 7.10 mm to (124.9, 85.0)
- moved J4 5.07 mm to (149.9, 78.2)
- moved R1 0.63 mm to (158.8, 75.9)
- renumbered D2 to D1, D1 to D2, J3 to J1, J1 to J2, J2 to J3, JP2 to JP1, JP1 to JP2, R3 to R2, R5 to R3, R1 to R4, R4 to R5
Connections:
- R1 pad 2: /WEAK_PULLDOWN -> GND
Routing:
- net /STRONG_PULLDOWN: track 7.42 -> 0.00 mm
- net GND: track 13.2 -> 19.8 mm, vias 5 -> 10
- net /WEAK_PULLDOWN: track 5.00 -> 0.00 mm
- net /SERVO_LEFT: track 10.0 -> 7.33 mm
- net /SHIELD: track 7.71 -> 5.74 mm
- net /SERVO_RIGHT: track 7.93 -> 7.06 mm
Other:
- board text added: "JLCJLCJLCJLC"
- board text added: "Sun Devil Motorsports SDM-24 DRS Board v1"
- board text added: "kanguwu"
- board text added: "{dblquote}Why are the engine scissors in the aero cabinet?{dblquote}"
- board text removed: "STRONG"
- board text removed: "Sun Devil Motorsports SDM-24 DRS Board"
- board text removed: "WEAK"

Commit message: fahb files
Changed lines of the file:
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@@
       (plot_on_all_layers_selection 0x0000000_00000000)
       (disableapertmacros false)
-      (usegerberextensions false)
-      (usegerberattributes true)
-      (usegerberadvancedattributes true)
-      (creategerberjobfile true)
+      (usegerberextensions true)
+      (usegerberattributes false)
+      (usegerberadvancedattributes false)
+      (creategerberjobfile false)
       (dashed_line_dash_ratio 12.000000)
       (dashed_line_gap_ratio 3.000000)
@@
       (psa4output false)
       (plotreference true)
-      (plotvalue true)
+      (plotvalue false)
       (plotinvisibletext false)
       (sketchpadsonfab false)
-      (subtractmaskfromsilk false)
+      (subtractmaskfromsilk true)
       (outputformat 1)
       (mirror false)
-      (drillshape 1)
+      (drillshape 0)
       (scaleselection 1)
-      (outputdirectory "")
+      (outputdirectory "fab/")
     )
   )
@@
       (stroke (width 0.1) (type solid)) (layer "F.Fab"))
     (pad "" np_thru_hole circle (at -1.6 2 90) (size 1.2 1.2) (drill 1.2) (layers "*.Cu" "*.Mask"))
-    (pad "1" thru_hole roundrect (at 0 0 90) (size 1.7 2) (drill 1) (layers "*.Cu" "*.Mask") (roundrect_rratio 0.147059)
+    (pad "1" thru_hole roundrect (at 0 0 90) (size 1.7 2) (drill 1) (layers "*.Cu" "*.Mask") (roundrect_rratio 0.1470588235)
       (net 40 "+5V") (pinfunction "Pin_1") (pintype "passive"))
     (pad "2" thru_hole oval (at 2.5 0 90) (size 1.7 2) (drill 1) (layers "*.Cu" "*.Mask")
@@
     (fp_line (start 1.6 0.8) (end -1.6 0.8)
       (stroke (width 0.1) (type solid)) (layer "F.Fab"))
-    (pad "1" smd roundrect (at -1.4625 0 180) (size 1.125 1.75) (layers "F.Cu" "F.Paste" "F.Mask") (roundrect_rratio 0.222222)
+    (pad "1" smd roundrect (at -1.4625 0 180) (size 1.125 1.75) (layers "F.Cu" "F.Paste" "F.Mask") (roundrect_rratio 0.2222222222)
       (net 17 "/BTN_INPUT") (pintype "passive"))
-    (pad "2" smd roundrect (at 1.4625 0 180) (size 1.125 1.75) (layers "F.Cu" "F.Paste" "F.Mask") (roundrect_rratio 0.222222)
+    (pad "2" smd roundrect (at 1.4625 0 180) (size 1.125 1.75) (layers "F.Cu" "F.Paste" "F.Mask") (roundrect_rratio 0.2222222222)
       (net 34 "GND") (pintype "passive"))
     (model "${KICAD6_3DMODEL_DIR}/Resistor_SMD.3dshapes/R_1206_3216Metric.wrl"
@@
     (fp_line (start 1 0.625) (end -1 0.625)
       (stroke (width 0.1) (type solid)) (layer "F.Fab"))
-    (pad "1" smd roundrect (at -0.9125 0 90) (size 1.025 1.4) (layers "F.Cu" "F.Paste" "F.Mask") (roundrect_rratio 0.243902)
+    (pad "1" smd roundrect (at -0.9125 0 90) (size 1.025 1.4) (layers "F.Cu" "F.Paste" "F.Mask") (roundrect_rratio 0.243902439)
       (net 44 "/PWR_LED") (pintype "passive"))
-    (pad "2" smd roundrect (at 0.9125 0 90) (size 1.025 1.4) (layers "F.Cu" "F.Paste" "F.Mask") (roundrect_rratio 0.243902)
+    (pad "2" smd roundrect (at 0.9125 0 90) (size 1.025 1.4) (layers "F.Cu" "F.Paste" "F.Mask") (roundrect_rratio 0.243902439)
       (net 34 "GND") (pintype "passive"))
     (model "${KICAD6_3DMODEL_DIR}/Resistor_SMD.3dshapes/R_0805_2012Metric.wrl"
@@
     (fp_line (start 1 0.625) (end -1 0.625)
       (stroke (width 0.1) (type solid)) (layer "F.Fab"))
-    (pad "1" smd roundrect (at -0.9125 0 90) (size 1.025 1.4) (layers "F.Cu" "F.Paste" "F.Mask") (roundrect_rratio 0.243902)
+    (pad "1" smd roundrect (at -0.9125 0 90) (size 1.025 1.4) (layers "F.Cu" "F.Paste" "F.Mask") (roundrect_rratio 0.243902439)
       (net 45 "/USR_LED_RSTR") (pintype "passive"))
-    (pad "2" smd roundrect (at 0.9125 0 90) (size 1.025 1.4) (layers "F.Cu" "F.Paste" "F.Mask") (roundrect_rratio 0.243902)
+    (pad "2" smd roundrect (at 0.9125 0 90) (size 1.025 1.4) (layers "F.Cu" "F.Paste" "F.Mask") (roundrect_rratio 0.243902439)
       (net 12 "/USR_LED") (pintype "passive"))
     (model "${KICAD6_3DMODEL_DIR}/Resistor_SMD.3dshapes/R_0805_2012Metric.wrl"
@@
     (fp_line (start 1.6 0.8) (end -1.6 0.8)
       (stroke (width 0.1) (type solid)) (layer "F.Fab"))
-    (pad "1" smd roundrect (at -1.4625 0 270) (size 1.125 1.75) (layers "F.Cu" "F.Paste" "F.Mask") (roundrect_rratio 0.222222)
+    (pad "1" smd roundrect (at -1.4625 0 270) (size 1.125 1.75) (layers "F.Cu" "F.Paste" "F.Mask") (roundrect_rratio 0.2222222222)
       (net 39 "/CAN_Rs") (pintype "passive"))
-    (pad "2" smd roundrect (at 1.4625 0 270) (size 1.125 1.75) (layers "F.Cu" "F.Paste" "F.Mask") (roundrect_rratio 0.222222)
+    (pad "2" smd roundrect (at 1.4625 0 270) (size 1.125 1.75) (layers "F.Cu" "F.Paste" "F.Mask") (roundrect_rratio 0.2222222222)
       (net 34 "GND") (pintype "passive"))
     (model "${KICAD6_3DMODEL_DIR}/Resistor_SMD.3dshapes/R_1206_3216Metric.wrl"
@@
       (stroke (width 0.1) (type solid)) (layer "F.Fab"))
     (pad "" np_thru_hole circle (at -1.6 2) (size 1.2 1.2) (drill 1.2) (layers "*.Cu" "*.Mask"))
-    (pad "1" thru_hole roundrect (at 0 0) (size 1.7 2) (drill 1) (layers "*.Cu" "*.Mask") (roundrect_rratio 0.147059)
+    (pad "1" thru_hole roundrect (at 0 0) (size 1.7 2) (drill 1) (layers "*.Cu" "*.Mask") (roundrect_rratio 0.1470588235)
       (net 21 "/SERVO_RIGHT") (pinfunction "Pin_1") (pintype "passive"))
     (pad "2" thru_hole oval (at 2.5 0) (size 1.7 2) (drill 1) (layers "*.Cu" "*.Mask")
@@
       (stroke (width 0.1) (type solid)) (layer "F.Fab"))
     (pad "" np_thru_hole circle (at -1.6 2 90) (size 1.2 1.2) (drill 1.2) (layers "*.Cu" "*.Mask"))
-    (pad "1" thru_hole roundrect (at 0 0 90) (size 1.7 1.95) (drill 0.95) (layers "*.Cu" "*.Mask") (roundrect_rratio 0.147059)
+    (pad "1" thru_hole roundrect (at 0 0 90) (size 1.7 1.95) (drill 0.95) (layers "*.Cu" "*.Mask") (roundrect_rratio 0.1470588235)
       (net 38 "/CANH") (pinfunction "Pin_1") (pintype "passive"))
     (pad "2" thru_hole oval (at 2.5 0 90) (size 1.7 1.95) (drill 0.95) (layers "*.Cu" "*.Mask")
@@
       (stroke (width 0.1) (type solid)) (layer "F.Fab"))
     (pad "" np_thru_hole circle (at -1.6 2 180) (size 1.2 1.2) (drill 1.2) (layers "*.Cu" "*.Mask"))
-    (pad "1" thru_hole roundrect (at 0 0 180) (size 1.7 2) (drill 1) (layers "*.Cu" "*.Mask") (roundrect_rratio 0.147059)
+    (pad "1" thru_hole roundrect (at 0 0 180) (size 1.7 2) (drill 1) (layers "*.Cu" "*.Mask") (roundrect_rratio 0.1470588235)
       (net 33 "VCC") (pinfunction "Pin_1") (pintype "passive"))
     (pad "2" thru_hole oval (at 2.5 0 180) (size 1.7 2) (drill 1) (layers "*.Cu" "*.Mask")
@@
     (effects (font (size 1 1) (thickness 0.15)) (justify left bottom))
   )
-  (gr_text "SHIELD" (at 124.9 80.3 90) (layer "F.SilkS" knockout)
+  (gr_text "SHIELD" (at 124.85 80.3 90) (layer "F.SilkS" knockout)
     (effects (font (size 1 1) (thickness 0.15)) (justify left bottom))
   )
