File: drs/drs.kicad_sch (KiCad schematic)
At the start: 17 parts, among them J1 POWER, J2 BUTTON, J3 CAN, U1 SN65HVD230

Commit message: more progress on drs box
Parts:
- C1, C2: footprint (none) -> Capacitor_SMD:C_0603_1608Metric
- D2: value D_TVS_Dual_AAC -> ESDCAN
- JP1: value Termination -> CAN; footprint (none) -> Connector_PinHeader_2.54mm:PinHeader_1x02_P2.54mm_Vertical
- R1: footprint (none) -> Resistor_SMD:R_1206_3216Metric
- R3: footprint (none) -> Resistor_SMD:R_0603_1608Metric
Connections:
- net GND: now also D2.3 (common)
- net USR_LED: now also A1.D2; no longer A1.D0 (D0/RX)
- net CANL: now reaches D2.1 (A1)
- net CANL: now also J3.2 (Pin_2), JP1.2 (B), U1.6 (CANL)
- net CANH: now reaches D2.2 (A2)
- net CANH: now also J3.1 (Pin_1), R3.1, U1.7 (CANH)
- net BUS_TERMINATION: now reaches R3.2
- net BUS_TERMINATION: now also JP1.1 (A)
- no-connect marks 12 -> 25
Other:
- note added: "TODO servo connectors"
- moved on the sheet: A1, C1, C2, D2, D3, J3, JP1, JP2, R1, R3, R4, U1

Commit message: drs work, wheel board m3
Parts:
- added J4: SERVO, symbol Connector:Conn_01x02_Pin
Connections:
- net SERVO_LEFT: now also J4.1 (Pin_1)
- net SERVO_RIGHT: now also J4.2 (Pin_2)
Other:
- note removed: "TODO servo connectors"
Changed lines of the file:
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@@
+    (stroke (width 0) (type default))
+  )
+  (wire (pts (xy 241.3 68.58) (xy 243.84 68.58))
     (stroke (width 0) (type default))
   )
@@
     (stroke (width 0) (type default))
   )
+  (wire (pts (xy 241.3 71.12) (xy 243.84 71.12))
+    (stroke (width 0) (type default))
+  )
   (wire (pts (xy 97.79 161.29) (xy 113.03 161.29))
     (stroke (width 0) (type default))
@@
   (wire (pts (xy 115.57 129.54) (xy 115.57 127))
     (stroke (width 0) (type default))
-  )
-  (text "TODO servo connectors" (at 97.79 85.09 0)
-    (effects (font (size 1.27 1.27)) (justify left bottom))
   )
   (text "TODO confirm value" (at 53.34 74.93 0)
@@
     (effects (font (size 1.27 1.27)) (justify left bottom))
   )
+  (label "SERVO_LEFT" (at 241.3 68.58 180) (fields_autoplaced)
+    (effects (font (size 1.27 1.27)) (justify right bottom))
+  )
   (label "CRX_3V3" (at 110.49 148.59 0) (fields_autoplaced)
     (effects (font (size 1.27 1.27)) (justify left bottom))
@@
   (label "CAN_Rs" (at 110.49 153.67 0) (fields_autoplaced)
     (effects (font (size 0.65 0.65)) (justify left bottom))
+  )
+  (label "SERVO_RIGHT" (at 241.3 71.12 180) (fields_autoplaced)
+    (effects (font (size 1.27 1.27)) (justify right bottom))
   )
   (label "SHIELD" (at 26.67 154.94 0) (fields_autoplaced)
@@
         )
       )
+    )
+  )
+  (symbol (lib_id "Connector:Conn_01x02_Pin") (at 248.92 68.58 0) (mirror y) (unit 1)
+    (in_bom yes) (on_board yes) (dnp no) (fields_autoplaced)
+    (property "Reference" "J4" (at 250.19 68.58 0)
+      (effects (font (size 1.27 1.27)) (justify right))
+    )
+    (property "Value" "SERVO" (at 250.19 71.12 0)
+      (effects (font (size 1.27 1.27)) (justify right))
+    )
+    (property "Footprint" "" (at 248.92 68.58 0)
+      (effects (font (size 1.27 1.27)) hide)
+    )
+    (property "Datasheet" "~" (at 248.92 68.58 0)
+      (effects (font (size 1.27 1.27)) hide)
+    )
+    (pin "1")
+    (pin "2")
+    (instances
+      (project "drs"
+        (path "/649c13a6-c815-4886-b904-75bc0e491aa4"
+          (reference "J4") (unit 1)
+        )
+      )

Commit message: found shifter for drs
Parts:
- added C3, C4: 100nF, Capacitor_SMD:C_0402_1005Metric, symbol Device:C_Small
- added U2: TXU0202, Package_SO:VSSOP-8_2.3x2mm_P0.5mm, symbol Library:TXU0202
- C1, C2: footprint Capacitor_SMD:C_0603_1608Metric -> Capacitor_SMD:C_0402_1005Metric
- D1, D3: footprint (none) -> LED_SMD:LED_1206_3216Metric
- D2: footprint (none) -> Package_TO_SOT_SMD:SOT-323_SC-70
- J1, J2, J4: footprint (none) -> Connector_JST:JST_XH_B2B-XH-AM_1x02_P2.50mm_Vertical
- J3: footprint (none) -> Connector_JST:JST_XH_B3B-XH-AM_1x03_P2.50mm_Vertical
- JP2: footprint (none) -> Connector_PinHeader_2.54mm:PinHeader_1x02_P2.54mm_Vertical
- R2, R4, R5: footprint (none) -> Resistor_SMD:R_0805_2012Metric
Connections:
- net +3.3V: now also C3.1, U2.3 (VCCA)
- net +5V: now also C4.1, U2.6 (OE), U2.7 (VCCB)
- net CRX_3V3: now also U2.5 (A1)
- net CRX_5V: now also U2.8 (B1Y)
- net CTX_3V3: now also U2.4 (A2Y)
- net CTX_5V: now also U2.1 (B2)
- net GND: now also C3.2, C4.2, U2.2 (GND)
Other:
- note removed: "TODO logic level shifter or switch to TJA1050"

Commit message: start routing on logger
Parts:
- added JP3: PULLDOWN, Connector_PinHeader_2.54mm:PinHeader_1x03_P2.54mm_Vertical, symbol Jumper:Jumper_3_Open
- added R6: 10k, Resistor_SMD:R_0805_2012Metric, symbol Device:R_Small
Connections:
- net BTN_INPUT: now also R6.1
- net GND: now also JP3.2 (C); no longer R2.2
- net SERVO_LEFT: now also J4.2 (Pin_2); no longer J4.1 (Pin_1)
- net SERVO_RIGHT: now also J4.1 (Pin_1); no longer J4.2 (Pin_2)
- new net STRONG_PULLDOWN: JP3.1 (A), R2.2
- new net WEAK_PULLDOWN: JP3.3 (B), R6.2
- no-connect marks 25 -> 27
Other:
- note added: "lol"

Commit message: drs board
Parts:
- removed JP3: PULLDOWN, Connector_PinHeader_2.54mm:PinHeader_1x03_P2.54mm_Vertical, symbol Jumper:Jumper_3_Open
- removed R2: 220, Resistor_SMD:R_0805_2012Metric, symbol Device:R_Small
- added D4, D5, D6: GG040205170N2P, Diode_SMD:D_0402_1005Metric, symbol Device:D_TVS
- R1: renamed from R6; footprint Resistor_SMD:R_0805_2012Metric -> Resistor_SMD:R_1206_3216Metric
- renumbered D2 to D1, D1 to D2, J3 to J1, J1 to J2, J2 to J3, JP2 to JP1, JP1 to JP2, R3 to R2, R5 to R3, R1 to R4, R4 to R5
Connections:
- net WEAK_PULLDOWN is gone; now on net GND: R1.2
- net BTN_INPUT: now also D4.2 (A2)
- net GND: now also D4.1 (A1), D5.1 (A1), D6.1 (A1)
- net SERVO_LEFT: now also D6.2 (A2)
- net SERVO_RIGHT: now also D5.2 (A2)
Other:
- note removed: "TODO confirm value"
- note removed: "lol"
- title: Aero Control Board -> DRS Control Board
- moved on the sheet: J3, R1
