File: lapbeacon/lapbeacon.kicad_pcb (KiCad board)
At the start: 2 copper layers, 32 x 44 mm, 32 parts, among them J1 USB, J2 BATTERY, J3 TC2030-NL, J4 UART, Q1 IRLML6346TRPBF, SW1 BIT_SEL, U1 STM32L031F6P7, U2 TPS3808DBV, U3 MIC37100-3.3

Commit message: over engineering yet again
Parts:
- removed the D1 at (135.2, 112.6)
- removed the R7 at (135.2, 114.6)
- added C11: 1uF, Capacitor_SMD:C_0603_1608Metric, F.Cu at (116.8, 107.1)
- added C13: 100nF, Capacitor_SMD:C_0402_1005Metric, F.Cu at (126.0, 98.0)
- added C3: 10uF, Capacitor_SMD:C_0805_2012Metric, F.Cu at (123.9, 109.4)
- added C4: 100nF, Capacitor_SMD:C_0402_1005Metric, F.Cu at (126.0, 102.0)
- added C9: 100nF, Capacitor_SMD:C_0402_1005Metric, F.Cu at (126.0, 100.0)
- added D2: RED, LED_SMD:LED_0603_1608Metric, F.Cu at (123.7, 112.2)
- added R5: 10k, Resistor_SMD:R_0402_1005Metric, F.Cu at (120.2, 110.9)
- added R6: 10k, Resistor_SMD:R_0402_1005Metric, F.Cu at (120.2, 112.9)
- added R8: 220, Resistor_SMD:R_0603_1608Metric, F.Cu at (116.8, 112.1)
- added U4: LMC555xMM, Package_SO:VSSOP-8_3.0x3.0mm_P0.65mm, F.Cu at (122.8, 105.6)
- added U5: MIC37100-3.3, Package_TO_SOT_SMD:SOT-223-3_TabPin2, F.Cu at (119.7, 99.2)
- added U6: 74AHC1G32, Package_TO_SOT_SMD:SOT-23-5, F.Cu at (112.2, 106.2)
- C1: value 100nF -> 1uF; footprint Capacitor_SMD:C_0402_1005Metric -> Capacitor_SMD:C_0603_1608Metric
- C2: value 10uF -> 100nF; footprint Capacitor_SMD:C_0805_2012Metric -> Capacitor_SMD:C_0402_1005Metric
- C8: value 1uF -> 50uF
- R3: footprint Resistor_SMD:R_0603_1608Metric -> Resistor_SMD:R_0402_1005Metric
- U3: value MIC37100-3.3 -> SN74LVC1G14DBV; footprint Package_TO_SOT_SMD:SOT-223-3_TabPin2 -> Package_TO_SOT_SMD:SOT-23-5
- moved U3 46.2 mm to (112.2, 101.8)
- moved TP1 41.0 mm to (111.1, 110.0)
- moved C8 38.0 mm to (116.8, 109.6), turned to 0 degrees
- moved U2 35.7 mm to (112.2, 97.3), turned to 0 degrees
- moved C1 32.7 mm to (116.8, 104.6)
- moved C2 31.0 mm to (126.0, 96.1)
- moved R3 26.8 mm to (120.2, 108.9), turned to 0 degrees
- moved R10 1.26 mm to (157.1, 124.0)
- moved Q1 0.81 mm to (161.0, 123.0), turned to 0 degrees
- moved R7 0.81 mm to (147.3, 125.3)
- moved R9 0.22 mm to (157.2, 126.1), turned to 180 degrees
- renumbered C6 to C10, C7 to C12, C3 to C5, C4 to C6, C5 to C7, D3 to D1, D2 to D3, R6 to R10, R8 to R11, R11 to R7, R5 to R9
Connections:
- C2 pad 1: +3.3V -> +BATT
- C8 pad 1: +BATT -> /TR
- U3 pad 1: +BATT -> unconnected-(U3-NC-Pad1)
- U3 pad 2: GND -> /~{RESET}
- U3 pad 3: +3.3V -> GND
Routing:
- net /BATT_IND: track 0.00 -> 5.54 mm
- net Net-(D1-K): track 0.00 -> 2.02 mm
- net Net-(Q1-D): track 3.27 -> 1.94 mm
- net GND: track 22.5 -> 23.8 mm, vias 8 -> 9
Other:
- board text removed: "+"
- board text removed: "-"

Commit message: things
Parts:
- added TP2: 3.3V, TestPoint:TestPoint_Pad_1.0x1.0mm, F.Cu at (161.8, 108.0)
- added TP3: GND, TestPoint:TestPoint_Pad_1.0x1.0mm, F.Cu at (161.9, 103.3)
- C8: value 50uF -> 20uF
- R11: value 25R / 250mW -> 24R / 250mW
- moved TP1 40.2 mm to (150.1, 100.3)
- moved C8 40.1 mm to (156.8, 109.0)
- moved U5 38.6 mm to (158.2, 97.5)
- moved C1 36.7 mm to (152.5, 96.2), turned to -90 degrees
- moved R5 35.7 mm to (155.6, 106.2), turned to 180 degrees
- moved R6 35.7 mm to (155.5, 107.5), turned to 180 degrees
- moved U2 34.9 mm to (147.1, 98.3), turned to 90 degrees
- moved C11 34.6 mm to (151.2, 103.4), turned to 180 degrees
- moved C3 32.8 mm to (156.0, 102.6)
- moved U3 31.6 mm to (143.6, 104.9)
- moved U6 31.2 mm to (143.3, 109.2)
- moved U4 28.2 mm to (150.9, 107.6)
- moved R3 26.6 mm to (144.6, 98.2), turned to -90 degrees
- moved C9 25.6 mm to (151.2, 104.9), turned to 180 degrees
- moved C13 22.5 mm to (146.0, 108.5), turned to -90 degrees
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Connections:
- net /BATT_IND renamed /USER_LED
- net Net-(D2-A) renamed /BATT_LED
Routing:
- net +BATT: track 0.00 -> 60.7 mm
- net +3.3V: track 38.9 -> 60.3 mm
- net GND: track 23.8 -> 45.2 mm, vias 9 -> 29
- net /~{RESET}: track 0.00 -> 16.3 mm
- net /Q: track 0.00 -> 11.6 mm
- net /TR: track 0.00 -> 9.57 mm
- net /BATT_LED: track 0.00 -> 8.41 mm
- net Net-(U4-R): track 0.00 -> 5.91 mm, vias 0 -> 2
- net Net-(U4-DIS): track 0.00 -> 3.75 mm
- net Net-(U2-~{MR}): track 0.00 -> 2.41 mm
- net /NRST: track 18.1 -> 15.9 mm, vias 2 -> 0
- net Net-(D2-K): track 0.00 -> 1.96 mm
- added copper zone on F.Cu, net +3.3V
- added copper zone on F.Cu, net +BATT
- added copper zone on F.Cu, net GND
Other:
- board text added: "3.3V"
- board text added: "BATT"
- board text added: "GND"
- board text added: "JLCJLCJLCJLC"
- board text added: "USER"
- board text added: "~{MR}"

Commit message: data logger 3.1
Other:
- board text removed: "JLCJLCJLCJLC"
Changed lines of the file:
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@@
-    (effects (font (size 1 1) (thickness 0.15)) (justify left bottom mirror))
-  )
-  (gr_text "JLCJLCJLCJLC" (at 162.1 99.7 90) (layer "B.SilkS")
     (effects (font (size 1 1) (thickness 0.15)) (justify left bottom mirror))
   )

Commit message: Fab files for pcbway
Parts:
- added G***: LOGO, LOGO, B.Cu at (147.9, 119.7)
Other:
- board text added: "WayWayWay"
