File: loadcelladapter/loadcelladapter.kicad_pcb (KiCad board)
At the start: 2 copper layers, 20 x 26 mm, 6 parts, among them J1 1734598-4, J2 JST-XH

Commit message: fahb files
Other:
- board text added: "M2.5"
- board text added: "TE Load Cell Cable Adapter"
- board text added: "systems starts with an s"
Changed lines of the file:
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@@
       (plot_on_all_layers_selection 0x0000000_00000000)
       (disableapertmacros false)
-      (usegerberextensions false)
-      (usegerberattributes true)
-      (usegerberadvancedattributes true)
-      (creategerberjobfile true)
+      (usegerberextensions true)
+      (usegerberattributes false)
+      (usegerberadvancedattributes false)
+      (creategerberjobfile false)
       (dashed_line_dash_ratio 12.000000)
       (dashed_line_gap_ratio 3.000000)
@@
       (psa4output false)
       (plotreference true)
-      (plotvalue true)
+      (plotvalue false)
       (plotinvisibletext false)
       (sketchpadsonfab false)
-      (subtractmaskfromsilk false)
+      (subtractmaskfromsilk true)
       (outputformat 1)
       (mirror false)
-      (drillshape 1)
+      (drillshape 0)
       (scaleselection 1)
       (outputdirectory "")
@@
     (property "ki_keywords" "connector")
     (attr through_hole)
-    (fp_text reference "J2" (at 3.75 4.525 90) (layer "F.SilkS")
+    (fp_text reference "J2" (at 11.6 2.6 90) (layer "F.SilkS")
         (effects (font (size 1 1) (thickness 0.15)))
     )
@@
       (stroke (width 0.1) (type solid)) (layer "F.Fab"))
     (pad "" np_thru_hole circle (at -1.6 2 270) (size 1.2 1.2) (drill 1.2) (layers "*.Cu" "*.Mask"))
-    (pad "1" thru_hole roundrect (at 0 0 270) (size 1.7 1.95) (drill 0.95) (layers "*.Cu" "*.Mask") (roundrect_rratio 0.147059)
+    (pad "1" thru_hole roundrect (at 0 0 270) (size 1.7 1.95) (drill 0.95) (layers "*.Cu" "*.Mask") (roundrect_rratio 0.1470588235)
       (net 1 "Net-(J1-Pin_1)") (pinfunction "Pin_1") (pintype "passive"))
     (pad "2" thru_hole oval (at 2.5 0 270) (size 1.7 1.95) (drill 0.95) (layers "*.Cu" "*.Mask")
@@
     (property "ki_keywords" "connector")
     (attr through_hole)
-    (fp_text reference "J1" (at -1.8416 3.0049 90 unlocked) (layer "F.SilkS")
+    (fp_text reference "J1" (at -6.8416 0.0049 90 unlocked) (layer "F.SilkS")
         (effects (font (size 1 1) (thickness 0.15)))
     )
@@
     (effects (font (size 1 1) (thickness 0.15)) (justify left bottom mirror))
   )
+  (gr_text "M2.5\n" (at 145.4 110.5 90) (layer "F.SilkS")
+    (effects (font (size 1 1) (thickness 0.15)) (justify left bottom))
+  )
+  (gr_text "TE Load Cell\nCable Adapter" (at 146.9 124.1 90) (layer "F.SilkS")
+    (effects (font (size 1 1) (thickness 0.15)) (justify left bottom))
+  )
+  (gr_text "systems starts with an s" (at 149.4 128.3 90) (layer "F.SilkS")
+    (effects (font (size 1 1) (thickness 0.15)) (justify left bottom))
+  )
   (segment (start 150.37 115) (end 147.7116 117.6584) (width 0.5) (layer "F.Cu") (net 1))

Commit message: data logger 3.1
Parts:
- removed H2, H3: M2.5, MountingHole:MountingHole_2.5mm
- H1, H4: footprint MountingHole:MountingHole_2.5mm -> MountingHole:MountingHole_3.2mm_M3
- moved H1 1.41 mm to (142.0, 110.0)
- moved H4 1.41 mm to (142.0, 128.0)
Other:
- board text added: "M3"
- board text removed: "M2.5"
Changed lines of the file:
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@@
   (net 3 "Net-(J1-Pin_3)")
   (net 4 "Net-(J1-Pin_4)")
-  (footprint "MountingHole:MountingHole_2.5mm" (layer "F.Cu")
-    (at 141 109)
-    (descr "Mounting Hole 2.5mm, no annular")
-    (tags "mounting hole 2.5mm no annular")
+  (footprint "MountingHole:MountingHole_3.2mm_M3" (layer "F.Cu")
+    (at 142 110)
+    (descr "Mounting Hole 3.2mm, no annular, M3")
+    (tags "mounting hole 3.2mm no annular m3")
     (property "Sheetfile" "loadcelladapter.kicad_sch")
     (property "Sheetname" "")
@@
     (property "ki_keywords" "mounting hole")
     (attr exclude_from_pos_files)
-    (fp_text reference "H1" (at 0 4) (layer "F.SilkS") hide
-        (effects (font (size 1 1) (thickness 0.15)))
-    )
-    (fp_text value "M2.5" (at 0 3.5) (layer "F.Fab")
+    (fp_text reference "H1" (at 0 -4.2) (layer "F.SilkS") hide
+        (effects (font (size 1 1) (thickness 0.15)))
+    )
+    (fp_text value "M2.5" (at 0 4.2) (layer "F.Fab")
         (effects (font (size 1 1) (thickness 0.15)))
     )
@@
         (effects (font (size 1 1) (thickness 0.15)))
     )
-    (fp_circle (center 0 0) (end 2.5 0)
+    (fp_circle (center 0 0) (end 3.2 0)
       (stroke (width 0.15) (type solid)) (fill none) (layer "Cmts.User"))
-    (fp_circle (center 0 0) (end 2.75 0)
+    (fp_circle (center 0 0) (end 3.45 0)
       (stroke (width 0.05) (type solid)) (fill none) (layer "F.CrtYd"))
-    (pad "" np_thru_hole circle (at 0 0) (size 2.5 2.5) (drill 2.5) (layers "*.Cu" "*.Mask"))
-  )
-  (footprint "MountingHole:MountingHole_2.5mm" (layer "F.Cu")
-    (at 155 109)
-    (descr "Mounting Hole 2.5mm, no annular")
-    (tags "mounting hole 2.5mm no annular")
-    (property "Sheetfile" "loadcelladapter.kicad_sch")
-    (property "Sheetname" "")
-    (property "ki_description" "Mounting Hole without connection")
-    (property "ki_keywords" "mounting hole")
-    (attr exclude_from_pos_files)
-    (fp_text reference "H2" (at 0 4) (layer "F.SilkS") hide
-        (effects (font (size 1 1) (thickness 0.15)))
-    )
-    (fp_text value "M2.5" (at 0 3.5) (layer "F.Fab")
-        (effects (font (size 1 1) (thickness 0.15)))
-    )
-    (fp_text user "${REFERENCE}" (at 0 0) (layer "F.Fab")
-        (effects (font (size 1 1) (thickness 0.15)))
-    )
-    (fp_circle (center 0 0) (end 2.5 0)
-      (stroke (width 0.15) (type solid)) (fill none) (layer "Cmts.User"))
-    (fp_circle (center 0 0) (end 2.75 0)
-      (stroke (width 0.05) (type solid)) (fill none) (layer "F.CrtYd"))
-    (pad "" np_thru_hole circle (at 0 0) (size 2.5 2.5) (drill 2.5) (layers "*.Cu" "*.Mask"))
+    (pad "" np_thru_hole circle (at 0 0) (size 3.2 3.2) (drill 3.2) (layers "*.Cu" "*.Mask"))
   )
   (footprint "Connector_JST:JST_XH_B4B-XH-AM_1x04_P2.50mm_Vertical" (layer "F.Cu")
@@
     )
   )
-  (footprint "MountingHole:MountingHole_2.5mm" (layer "F.Cu")
-    (at 141 129)
-    (descr "Mounting Hole 2.5mm, no annular")
-    (tags "mounting hole 2.5mm no annular")
+  (footprint "MountingHole:MountingHole_3.2mm_M3" (layer "F.Cu")
+    (at 142 128)
+    (descr "Mounting Hole 3.2mm, no annular, M3")
+    (tags "mounting hole 3.2mm no annular m3")
     (property "Sheetfile" "loadcelladapter.kicad_sch")
     (property "Sheetname" "")
@@
     (property "ki_keywords" "mounting hole")
     (attr exclude_from_pos_files)
-    (fp_text reference "H4" (at 0 -3.5) (layer "F.SilkS") hide
-        (effects (font (size 1 1) (thickness 0.15)))
-    )
-    (fp_text value "M2.5" (at 0 3.5) (layer "F.Fab")
+    (fp_text reference "H4" (at 5 0) (layer "F.SilkS") hide
+        (effects (font (size 1 1) (thickness 0.15)))
+    )
+    (fp_text value "M2.5" (at 0 4.2) (layer "F.Fab")
         (effects (font (size 1 1) (thickness 0.15)))
     )
@@
         (effects (font (size 1 1) (thickness 0.15)))
     )
-    (fp_circle (center 0 0) (end 2.5 0)
+    (fp_circle (center 0 0) (end 3.2 0)
       (stroke (width 0.15) (type solid)) (fill none) (layer "Cmts.User"))
-    (fp_circle (center 0 0) (end 2.75 0)
+    (fp_circle (center 0 0) (end 3.45 0)
       (stroke (width 0.05) (type solid)) (fill none) (layer "F.CrtYd"))
-    (pad "" np_thru_hole circle (at 0 0) (size 2.5 2.5) (drill 2.5) (layers "*.Cu" "*.Mask"))
-  )
-  (footprint "MountingHole:MountingHole_2.5mm" (layer "F.Cu")
-    (at 155 129)
-    (descr "Mounting Hole 2.5mm, no annular")
-    (tags "mounting hole 2.5mm no annular")
-    (property "Sheetfile" "loadcelladapter.kicad_sch")
-    (property "Sheetname" "")
-    (property "ki_description" "Mounting Hole without connection")
-    (property "ki_keywords" "mounting hole")
-    (attr exclude_from_pos_files)
-    (fp_text reference "H3" (at 0 -3.5) (layer "F.SilkS") hide
-        (effects (font (size 1 1) (thickness 0.15)))
-    )
-    (fp_text value "M2.5" (at 0 3.5) (layer "F.Fab")
-        (effects (font (size 1 1) (thickness 0.15)))
-    )
-    (fp_text user "${REFERENCE}" (at 0 0) (layer "F.Fab")
-        (effects (font (size 1 1) (thickness 0.15)))
-    )
-    (fp_circle (center 0 0) (end 2.5 0)
-      (stroke (width 0.15) (type solid)) (fill none) (layer "Cmts.User"))
-    (fp_circle (center 0 0) (end 2.75 0)
-      (stroke (width 0.05) (type solid)) (fill none) (layer "F.CrtYd"))
-    (pad "" np_thru_hole circle (at 0 0) (size 2.5 2.5) (drill 2.5) (layers "*.Cu" "*.Mask"))
+    (pad "" np_thru_hole circle (at 0 0) (size 3.2 3.2) (drill 3.2) (layers "*.Cu" "*.Mask"))
   )
   (gr_line (start 141 106) (end 155 106)
@@
     (effects (font (size 1 1) (thickness 0.15)) (justify left bottom mirror))
   )
-  (gr_text "M2.5\n" (at 145.4 110.5 90) (layer "F.SilkS")
+  (gr_text "M3" (at 146 111 90) (layer "F.SilkS")
     (effects (font (size 1 1) (thickness 0.15)) (justify left bottom))
   )

Commit message: Fab files for pcbway
Other:
- board text added: "WayWayWay"
- board text removed: "JLCJLCJLCJLC"
Changed lines of the file:
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@@
       (plot_on_all_layers_selection 0x0000000_00000000)
       (disableapertmacros false)
-      (usegerberextensions true)
+      (usegerberextensions false)
       (usegerberattributes false)
       (usegerberadvancedattributes false)
@@
       (drillshape 0)
       (scaleselection 1)
-      (outputdirectory "")
+      (outputdirectory "fab/")
     )
   )
@@
   (gr_arc (start 141 132) (mid 138.87868 131.12132) (end 138 129)
     (stroke (width 0.1) (type default)) (layer "Edge.Cuts"))
-  (gr_text "JLCJLCJLCJLC" (at 156 124 -90) (layer "B.SilkS")
-    (effects (font (size 1 1) (thickness 0.15)) (justify left bottom mirror))
-  )
   (gr_text "M3" (at 146 111 90) (layer "F.SilkS")
     (effects (font (size 1 1) (thickness 0.15)) (justify left bottom))
@@
     (effects (font (size 1 1) (thickness 0.15)) (justify left bottom))
   )
-  (gr_text "systems starts with an s" (at 149.4 128.3 90) (layer "F.SilkS")
-    (effects (font (size 1 1) (thickness 0.15)) (justify left bottom))
-  )
+  (gr_text "systems starts with an s" (at 149.3 126 90) (layer "F.SilkS")
+    (effects (font (size 1 1) (thickness 0.15)) (justify left bottom))
+  )
+  (gr_text "WayWayWay" (at 144.5 129.9) (layer "F.SilkS")
+    (effects (font (size 1 1) (thickness 0.15)) (justify left bottom))
+  )
