File: 2026/Logger/SDM26_Logger_3.0/SDM26LoggerV3.0.kicad_sch (KiCad schematic)
At the start: 97 parts, among them IC1 ESP32-S3-WROOM-1-N8R8, IC2 NEO-F9P-15B, IC3 MIC37100-3.3WS, IC5 TPS563211DRLR, IC6 CP2102N-A02-GQFN28, J1 USB_B, J2 USB_B_Micro, J3 1-776087-4, J4 Molex_1040310811, J5 USB_B_Micro, J6 1-776087-4, K1 IMB03IGR, Q1 SOT96P237X111-3N, Q2 SOT96P237X111-3N, U1 INA260, U11 ADC128S102, U2 TPS2116DRL, U3 ADR425BRZ, U4 SN65HVD230, U5 USBLC6-2SC6, U6 USBLC6-2SC6, U7 USBLC6-2SC6, U8 TPS2116, U9 ST_EMIF06-MSD02N16, Y2 ECX-.327-CDX-2096

Commit message: Beginning logger the loooong way (V3) and other misc changes
Parts:
- removed D10, D11, D12, D13, D6, D7, D8, D9: TVS, Diode_SMD:D_SOD-323, symbol Device:D_TVS
- added C1, C2, C3, C4, C5, C6, C7, C8: 33nF, Capacitor_SMD:C_0603_1608Metric, symbol Device:C_Small
- added D2, D3, D4, D5, D6, D7, D8, D9: MBR0540T1G, SOD3716X135N, symbol SDM_DIODES:MBR0540T1G
- added R1, R2, R23, R24, R3, R30, R31, R32, R33, R34, R4, R5: 100, Resistor_SMD:R_0603_1608Metric, symbol Device:R_Small
- renumbered D2 to D1
Connections:
- net +5V: now also J3.13 (Pin_13), J3.14 (Pin_14), J6.20 (Pin_20), J6.5 (Pin_5), J6.6 (Pin_6), J6.7 (Pin_7); no longer J3.10 (Pin_10), J3.3 (Pin_3), J3.9 (Pin_9), J6.22 (Pin_22), J6.23 (Pin_23)
- net +5VA: now also D2.1 (K), D3.1 (K), D4.1 (K), D5.1 (K), D6.1 (K), D7.1 (K), D8.1 (K), D9.1 (K)
- net ADC_CLK: now also R32.1; no longer U11.16 (SCLK)
- net ADC_CS: now also R31.1; no longer U11.1 (~{CS})
- net ADC_DIN: now also R33.2; no longer U11.14 (DIN)
- net ADC_DOUT: now also R34.1; no longer U11.15 (DOUT)
- net AIN0: now also J3.7 (Pin_7), R1.1; no longer J3.4 (Pin_4), U11.4 (IN0)
- net AIN1: now also J3.8 (Pin_8), R2.1; no longer J3.5 (Pin_5), U11.5 (IN1)
- net AIN2: now also J3.22 (Pin_22), R3.1; no longer J3.13 (Pin_13), U11.6 (IN2)
- net AIN3: now also J3.23 (Pin_23), R4.1; no longer J3.6 (Pin_6), U11.7 (IN3)
- net AIN4: now also J6.16 (Pin_16), R5.1; no longer J3.14 (Pin_14), U11.8 (IN4)
- net AIN5: now also J6.17 (Pin_17), R23.1; no longer J6.10 (Pin_10), U11.9 (IN5)
- net AIN6: now also J6.1 (Pin_1), R24.1; no longer J6.3 (Pin_3), U11.10 (IN6)
- net AIN7: now also J6.2 (Pin_2), R30.1; no longer J6.11 (Pin_11), U11.11 (IN7)
- net CAN+: now also J6.8 (Pin_8); no longer J3.23 (Pin_23)
- net CAN-: now also J6.23 (Pin_23); no longer J3.8 (Pin_8)
- net CAN_CTX: now also IC1.38 (IO2); no longer IC1.22 (IO14)
- net CAN_RTX: now also IC1.39 (IO1); no longer IC1.23 (IO21)
- net GND: now also J6.18 (Pin_18), J6.19 (Pin_19), J6.22 (Pin_22), J6.3 (Pin_3), J6.4 (Pin_4), C1.2, C2.2, C3.2, C4.2, C5.2, C6.2, C7.2, C8.2; no longer J6.5 (Pin_5), J6.6 (Pin_6), J6.7 (Pin_7), J6.8 (Pin_8)
- new net: C6.1, D7.2 (A), R23.2, U11.9 (IN5)
- new net: C1.1, D2.2 (A), R1.2, U11.4 (IN0)
- new net: C5.1, D6.2 (A), R5.2, U11.8 (IN4)
- new net: C4.1, D5.2 (A), R4.2, U11.7 (IN3)
- new net: C8.1, D9.2 (A), R30.2, U11.11 (IN7)
- new net: C3.1, D4.2 (A), R3.2, U11.6 (IN2)
- new net: C2.1, D3.2 (A), R2.2, U11.5 (IN1)
- new net: R31.2, U11.1 (~{CS})
- new net: C7.1, D8.2 (A), R24.2, U11.10 (IN6)
- new net: R33.1, U11.14 (DIN)
- new net: R34.2, U11.15 (DOUT)
- new net: R32.2, U11.16 (SCLK)
- no-connect marks 58 -> 55
Other:
- moved on the sheet: C41, C42, C43, C46, U11, Y2

Commit message: Logger V3.0 wiring complete needs silkscreen fixes
Parts:
- added C47, C48: 10uF, Capacitor_SMD:C_0603_1608Metric, symbol Device:C_Small
- added C49: 1uF, Capacitor_SMD:C_0603_1608Metric, symbol Device:C_Small
- added IC4: MIC37100-3.3WS, SOT230P700X180-4N, symbol VoltageRegulators:MIC37100-3.3WS
- added R35: 220, Resistor_SMD:R_0603_1608Metric, symbol Device:R_Small
- added R36: 100k, Resistor_SMD:R_0603_1608Metric, symbol Device:R_Small
- added R37, R38: 27, Resistor_SMD:R_0603_1608Metric, symbol Device:R_Small
- R20: value 10uF -> 10
- renumbered TP4 to TP3, TP3 to TP4
Connections:
- net +3.3V: no longer R19.2
- net +5V: now also J3.10 (Pin_10), J3.9 (Pin_9), LED1.1 (K); no longer J3.14 (Pin_14), J3.15 (Pin_15)
- net ADC_CLK: now also IC1.5 (IO5); no longer IC1.19 (IO11)
- net ADC_CS: now also IC1.4 (IO4); no longer IC1.18 (IO10)
- net ADC_DIN: now also IC1.7 (IO7); no longer IC1.21 (IO13)
- net ADC_DOUT: now also IC1.6 (IO6); no longer IC1.20 (IO12)
- net CAN_CTX: now also IC1.11 (IO18); no longer IC1.38 (IO2)
- net CAN_RTX: now also IC1.12 (IO8); no longer IC1.39 (IO1)
- net CAN_TERM: now also IC1.10 (IO17); no longer IC1.24 (IO47)
- net GND: now also C47.1, C48.2, IC4.2 (GND_1), IC4.4 (GND_2)
- net GPS_D+: now also R38.2; no longer U7.1 (I/O1)
- net GPS_D-: now also R37.1; no longer U7.3 (I/O2)
- net I2C1_SCL: now also IC1.24 (IO47); no longer IC1.17 (IO9)
- net I2C1_SDA: now also IC1.25 (IO48); no longer IC1.16 (IO46)
- net PPS_LED: now also R35.2; no longer IC2.3 (TIMEPULSE)
- net RF_IN: now also C49.2; no longer IC2.11 (RF_IN)
- net RTK_STAT: now also R19.2; no longer LED1.2 (A)
- net SD_CD: now also IC1.26 (IO45); no longer IC1.12 (IO8)
- net SD_CLK: now also IC1.19 (IO11); no longer IC1.6 (IO6)
- net SD_CMD: now also IC1.20 (IO12); no longer IC1.7 (IO7)
- net SD_DAT0: now also IC1.18 (IO10); no longer IC1.5 (IO5)
- net SD_DAT1: now also IC1.17 (IO9); no longer IC1.4 (IO4)
- net SD_DAT2: now also IC1.22 (IO14); no longer IC1.11 (IO18)
- net SD_DAT3: now also IC1.21 (IO13); no longer IC1.10 (IO17)
- net UART1_D+: now also IC1.16 (IO46); no longer IC1.14 (IO20)
- net UART1_D-: now also IC1.15 (IO3); no longer IC1.13 (IO19)
- net UART2_RX: now also IC1.14 (IO20); no longer IC1.25 (IO48)
- net UART2_TX: now also IC1.13 (IO19); no longer IC1.26 (IO45)
- net USER_LED: now also IC1.28 (IO35); no longer IC1.15 (IO3)
- net VUSB: now also C47.2, IC4.1 (IN); no longer IC2.7 (V_USB)
- net at R19.1: now also LED1.2 (A); no longer LED1.1 (K)
- new net: R38.1, U7.1 (I/O1)
- new net: R37.2, U7.3 (I/O2)
- new net: C49.1, IC2.11 (RF_IN)
- new net: IC2.3 (TIMEPULSE), R35.1
- new net GNSS_LDO: C48.1, IC4.3 (OUT), R36.1
- new net GNSS_USB_PWR: IC2.7 (V_USB), R36.2
- no-connect marks 55 -> 56
Other:
- moved on the sheet: R19, TP5
