File: 2026/TimingGates/SDM26_TimingGates_V1.1/SDM26_TimingGates_V1.1.kicad_sch (KiCad schematic)
At the start: 27 parts, among them IC1 MIC37100-3.3WS, IC2 ESP32-S3-WROOM-1U-N8R8, IC3 CP2102N-A02-GQFN28, IC4 DS3231SN#, J1 ESP_USB, J2 Conn_01x04_Socket, Q1 MMBT2222LT1G, Q2 MMBT2222LT1G, U1 USBLC6-2SC6

Commit message: Misc
Parts:
- Q1, Q2: symbol Simulation_SPICE:NPN -> SDM_TRANSISTOR:MMBT2222LT1G
Connections:
- net BOOT: now also IC2.27 (IO0), Q2.3 (C); no longer IC2.16 (IO46), Q2.1 (C)
- net CHIP_PU: now also Q1.3 (C); no longer Q1.1 (C)
- net at R2.1: now also Q2.1 (B); no longer Q2.2 (B)
- net at IC3.28 (DTR), R1.2: now also Q2.2 (E); no longer Q2.3 (E)
- net at R1.1: now also Q1.1 (B); no longer Q1.2 (B)
- net at IC3.24 (RTS), R2.2: now also Q1.2 (E); no longer Q1.3 (E)
Other:
- note added: "3.3v LDO"
- note added: "USB to UART Bridge"
- note removed: "ESP_PROG"
- note removed: "ESP_Programmer"
- moved on the sheet: C1, C2, C3, IC1, IC2, R4, R6
