File: 2026/Logger/SDM26_Logger_V4.0/SDM26LoggerV4.0.kicad_pcb (KiCad board)
At the start: 4 copper layers, 75 x 87 mm, 141 parts, among them IC1 ESP32-S3-WROOM-1-N8R8, IC2 CP2102N-A02-GQFN28, IC3 MIC37100-3.3WS, IC4 TPS563211DRLR, IC5 TLP175A_TPL,E, IC6 MIC37100-3.3WS, IC7 NEO-F9P-15B, IC8 TPS259250DRCR, J1 UART_USB, J2 ESP_USB, J3 GNSS_Debug, J4 Molex_1040310811, J5 1-776087-4, J6 1-776087-4, Q1 MMBT2222LT1G, Q2 MMBT2222LT1G, U1 INA260, U10 EMIF06-MSD02N16, U2 USBLC6-2SC6, U3 TPS2116DRL, U4 USBLC6-2SC6, U5 USBLC6-2SC6, U6 TPS2116, U7 SN65HVD230, U8 ADR425BRZ, U9 ADC128S102, Y1 ECX-.327-CDX-2096

Commit message: Logger 4.0 commit
Parts:
- Q1, Q2: footprint Transistors:SOT96P237X111-3N -> SDM_MiscFootprint:SOT96P237X111-3N
- moved R1 1.13 mm to (103.4, 89.8), turned to 180 degrees
- moved R2 1.00 mm to (103.4, 91.3), turned to 0 degrees
- moved Q2 0.20 mm to (102.3, 94.0)
- moved Q1 0.15 mm to (105.9, 94.0)
Connections:
- Q1 pad 1: /CHIP_PU -> Net-(Q1-B)
- Q1 pad 2: Net-(Q1-B) -> Net-(IC2-RTS)
- Q1 pad 3: Net-(IC2-RTS) -> /CHIP_PU
- Q2 pad 1: /GPIO0 -> Net-(Q2-B)
- Q2 pad 2: Net-(Q2-B) -> Net-(IC2-DTR)
- Q2 pad 3: Net-(IC2-DTR) -> /GPIO0
Routing:
- net Net-(IC2-DTR): track 0.64 -> 10.0 mm
- net Net-(IC2-RTS): track 1.26 -> 7.66 mm
- net Net-(Q1-B): track 0.00 -> 4.19 mm
- net Net-(Q2-B): track 0.00 -> 1.88 mm
- net /CHIP_PU: track 82.6 -> 83.9 mm
- net /GPIO0: track 50.5 -> 51.7 mm
- net /CAN_TERM: track 63.8 -> 63.1 mm
- net GND: track 145.6 -> 144.9 mm

Commit message: Computer Sync
Parts:
- added C48: 4.7uF, Capacitor_SMD:C_0603_1608Metric, F.Cu at (80.6, 107.3)
- added C49: 10uF, Capacitor_SMD:C_0603_1608Metric, F.Cu at (80.6, 109.8)
- added R45: 10k, Resistor_SMD:R_0603_1608Metric, F.Cu at (80.6, 112.3)
- added R46: 10k, Resistor_SMD:R_0603_1608Metric, F.Cu at (80.6, 114.8)

Commit message: Updates Before September Order
Parts:
- removed C3, C35: 1uF, Capacitor_SMD:C_0603_1608Metric
- added C50: 10uF, Capacitor_SMD:C_0603_1608Metric, F.Cu at (113.6, 155.4)
- added R47: 0, Resistor_SMD:R_0603_1608Metric, F.Cu at (125.9, 111.3)
- C1, C13, C18, C19, C2, C22, C23, C26, C28, C36: value 1uF -> 100nF
- C49: value 10uF -> 100uF
- U10: footprint uSDs:UQFN-17-3.5x1.2mm -> SDM_MiscFootprint:UQFN-17-3.5x1.2mm_copy
- moved R46 58.0 mm to (131.5, 142.5), turned to 180 degrees
- moved R45 56.4 mm to (131.4, 136.7)
- moved C49 23.2 mm to (103.6, 106.8), turned to 90 degrees
- moved C48 20.9 mm to (101.3, 104.9), turned to 180 degrees
- moved R13 5.96 mm to (107.6, 108.7), turned to -90 degrees
- moved C17 3.20 mm to (105.1, 106.0), turned to -90 degrees
- moved R11 2.30 mm to (107.4, 106.4)
- moved R12 2.30 mm to (107.4, 104.9)
- moved C36 2.19 mm to (110.9, 103.8)
- moved C2 1.50 mm to (123.6, 135.8)
- moved R30 1.50 mm to (110.9, 102.3)
- moved C1 0.76 mm to (112.1, 155.4), turned to -90 degrees
- turned C4 to -90 degrees
- turned C9 to 180 degrees
- turned R3 to -90 degrees
Connections:
- net Net-(IC8-ILIM) renamed /ILIM
- AE1 pad 1: /RF_IN -> /RF_UFL
- C4 pad 1: VBUS -> GND
- C4 pad 2: GND -> VBUS
- C9 pad 1: /5V_SMPS_OUT -> GND
- C9 pad 2: Net-(U3-MODE) -> /5V_SMPS_OUT
- IC7 pad 11: Net-(IC7-RF_IN) -> /RF_UFL
- L2 pad 1: /RF_IN -> /RF_UFL
- R3 pad 1: /ST -> /EFUSE IN
- R3 pad 2: /EFUSE IN -> /ST
- R5 pad 1: Net-(U3-MODE) -> /5V_SMPS_OUT
- U3 pad 3: Net-(U3-MODE) -> /5V_SMPS_OUT
- U3 pad 5: Net-(U3-MODE) -> /5V_SMPS_OUT
Routing:
- net Net-(U3-MODE): track 15.4 -> 0.00 mm, vias 2 -> 0
- net /5V_SMPS_OUT: track 62.7 -> 76.2 mm, vias 4 -> 5
- net +5V: track 231.8 -> 242.5 mm
- net /RF_UFL: track 0.00 -> 8.31 mm
- net GND: track 144.9 -> 151.3 mm, vias 192 -> 198
- net Net-(IC7-RF_IN): track 5.50 -> 0.00 mm
- net +3.3V: track 37.4 -> 42.1 mm, vias 11 -> 13
- net /RF_IN: track 4.12 -> 0.00 mm
- net Net-(IC2-VBUS): track 4.27 -> 7.42 mm
- net /ST: track 45.9 -> 43.3 mm
- net /RSTB: track 1.88 -> 4.23 mm
- net /EFUSE IN: track 4.31 -> 6.17 mm
- net /VCC_RF: track 9.29 -> 7.79 mm
- net /I2C1_SDA: track 42.9 -> 44.2 mm
- net VBUS: track 70.4 -> 69.2 mm
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Other:
- board text added: "SDM-26 DAQ Data Logger v4.0"
- board text removed: "SDM-26 DAQ Data Logger v3.3"

Commit message: September order final commit
Parts:
- C49: value 100uF -> 100nF
- R45, R46: value 10k -> 2.2k
Connections:
- IC1 pad 23: unconnected-(IC1-IO21-Pad23) -> /SD_CD
- IC1 pad 26: /SD_CD -> unconnected-(IC1-IO45-Pad26)
- IC7 pad 20: /UART2_TX -> /UART2_RX
- IC7 pad 21: /UART2_RX -> /UART2_TX
Routing:
- net /SD_CD: track 18.1 -> 11.1 mm
- net /UART2_TX: track 62.3 -> 63.4 mm
- net /UART2_RX: track 62.0 -> 60.9 mm
