File: 2026/IMU/SDM26_IMU_V1.0/SDM26_IMU_V1.0.kicad_pcb (KiCad board)
At the start: 4 copper layers, 52 x 41 mm, 52 parts, among them IC1 ESP32-S3-WROOM-1-N8R8, IC2 ISM330DHCXTR, IC3 MIC37100-3.3WS, IC4 CP2102N-A02-GQFN28, IC5 TLP175A_TPL,E, IC6 TPS2116DRLR, IC7 TPS259250DRCR, J1 Conn_01x04_Socket, J2 USB_B_Micro, Q1 MMBT2222LT1G, Q2 MMBT2222LT1G, U1 SN65HVD230, U2 USBLC6-2SC6

Commit message: Updates Before September Order
Parts:
- removed the C11 at (81.5, 67.5)
- removed the R18 at (82.5, 65.0)
- removed the R6 at (96.5, 66.0)
- added C12: 1uF, Capacitor_SMD:C_0603_1608Metric, F.Cu at (85.0, 79.0)
- added C2: 100nF, Capacitor_SMD:C_0603_1608Metric, F.Cu at (81.2, 44.0)
- added C3: 1uF, Capacitor_SMD:C_0603_1608Metric, F.Cu at (79.7, 50.7)
- added C5: 4.7uF, Capacitor_SMD:C_0603_1608Metric, F.Cu at (71.6, 71.5)
- added C6: 100uF, Capacitor_SMD:C_0603_1608Metric, F.Cu at (71.6, 73.0)
- added G***: LOGO, Library:wheelyboi, F.Cu at (107.9, 52.0)
- added G***: LOGO, Library:sdmlogo, F.Cu at (108.0, 59.3)
- added R1: 10k, Resistor_SMD:R_0603_1608Metric, F.Cu at (79.7, 49.2)
- added R20: 0, Resistor_SMD:R_0603_1608Metric, F.Cu at (83.6, 82.0)
- C1: value 100nF -> 10uF
- C4: renamed from C7; value 100nF -> 1uF
- C7: renamed from C5; value 100nF -> 1uF
- LED1: renamed from LED2; value 150060VS75000 -> 150060GS75000
- R18: renamed from R7; value 220 -> 68
- R8: renamed from R1; value 220 -> 5.05
- TP1: value TestPoint -> 5V_ST
- moved C11 7.64 mm to (77.0, 76.4)
- moved R9 5.63 mm to (76.9, 72.4), turned to -90 degrees
- moved C1 5.61 mm to (79.7, 44.0), turned to 90 degrees
- moved R8 3.29 mm to (99.5, 64.5)
- moved R13 3.26 mm to (69.3, 77.9), turned to -90 degrees
- moved TP1 2.94 mm to (79.1, 81.3)
- moved R17 2.20 mm to (81.3, 79.8), turned to -90 degrees
- moved R5 2.02 mm to (93.4, 67.7)
- moved R7 1.84 mm to (67.7, 66.1)
- moved LED1 1.82 mm to (102.0, 65.3)
- moved C9 1.66 mm to (78.3, 59.6), turned to 180 degrees
- moved R4 1.58 mm to (93.4, 64.7), turned to -90 degrees
- moved C10 1.52 mm to (78.3, 58.1), turned to 180 degrees
- moved R15 1.47 mm to (81.3, 76.8), turned to 90 degrees
- moved LED2 1.45 mm to (88.0, 80.8)
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- renumbered C3 to C10, C9 to C11, C4 to C13, C6 to C14, C10 to C15, C2 to C9, D2 to D1, IC4 to IC3, IC7 to IC4, IC3 to IC5, IC5 to IC7, LED1 to LED2, R12 to R10, R9 to R11, R13 to R12, R14 to R13, R17 to R14, R16 to R15, R2 to R16, R15 to R17, R3 to R19, R10 to R2, R11 to R3, R19 to R6, R20 to R7, R8 to R9, U2 to U1, U1 to U2
Connections:
- net Net-(IC7-ILIM) renamed /ILIM
- C1 pad 1: Net-(IC1-3V3) -> +3.3V
- C1 pad 2: +3.3V -> GND
- C13 pad 2: Net-(IC3-IN) -> +5V
- IC1 pad 13: /U0RXD -> unconnected-(IC1-IO19-Pad13)
- IC1 pad 14: /U0TXD -> unconnected-(IC1-IO20-Pad14)
- IC1 pad 2: Net-(IC1-3V3) -> +3.3V
- IC1 pad 36: unconnected-(IC1-RXD0-Pad36) -> /U0RXD
- IC1 pad 37: unconnected-(IC1-TXD0-Pad37) -> /U0TXD
- IC4 pad 3: +5V -> /EFUSE_IN
- IC4 pad 4: +5V -> /EFUSE_IN
- IC4 pad 5: +5V -> /EFUSE_IN
- IC4 pad 6: Net-(IC3-IN) -> +5V
- IC4 pad 7: Net-(IC3-IN) -> +5V
- IC4 pad 8: Net-(IC3-IN) -> +5V
- IC5 pad 1: Net-(IC3-IN) -> +5V
- IC6 pad 2: +5V -> /EFUSE_IN
- IC6 pad 7: +5V -> /EFUSE_IN
- LED1 pad 1: Net-(LED2-K) (its old number) -> GND
- LED1 pad 2: /USER_LED -> Net-(LED1-A)
- R15 pad 1: +5V -> /EFUSE_IN
- R17 pad 1: +5V -> /EFUSE_IN
- R4 pad 2: /I2C1_SDA -> /I2C1_SCL
- R5 pad 2: /I2C1_SCL -> /I2C1_SDA
- R8 pad 1: Net-(LED2-K) (its old number) -> /USER_LED
- R8 pad 2: GND -> Net-(LED1-A)
- R9 pad 2: VCC -> +5V
Routing:
- net /U0TXD: track 11.8 -> 34.6 mm, vias 0 -> 2
- net /U0RXD: track 13.1 -> 35.3 mm, vias 0 -> 2
- net +5V: track 15.1 -> 29.8 mm
- net +3.3V: track 20.0 -> 32.3 mm, vias 13 -> 11
- net /EFUSE_IN: track 0.00 -> 10.9 mm
- net Net-(IC3-IN): track 10.5 -> 0.00 mm
- net Net-(IC1-3V3): track 6.99 -> 0.00 mm
- net GND: track 65.1 -> 60.5 mm, vias 25 -> 34
- net Net-(IC3-RTS): track 19.5 -> 15.3 mm
- net VCC: track 34.2 -> 37.1 mm
- net Net-(IC6-PR1): track 6.40 -> 8.39 mm
- net VBUS: track 32.7 -> 30.8 mm
- net Net-(LED1-A): track 0.00 -> 1.80 mm
- net Net-(LED2-K) (its old number): track 1.78 -> 0.00 mm
- net /USER_LED: track 3.71 -> 2.60 mm
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- added copper zone on F.Cu, net +5V
- added copper zone on F.Cu, net /EFUSE_IN
Other:
- board text added: "+X"
- board text added: "+Y"
- board text added: "-Y"

Commit message: September order sync
Changed lines of the file:
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@@
 		(start 74.455 49.1)
 		(end 74.455 51.6)
-		(width 0.2)
+		(width 0.3)
 		(layer "F.Cu")
 		(net 4)
@@
 		(start 75.756 52.354032)
 		(end 75.756 53.035968)
-		(width 0.2)
+		(width 0.3)
 		(layer "F.Cu")
 		(net 4)
@@
 		(start 74.949 52.094)
 		(end 75.495968 52.094)
-		(width 0.2)
+		(width 0.3)
 		(layer "F.Cu")
 		(net 4)
@@
 		(start 74.826968 53.965)
 		(end 74.48 53.965)
-		(width 0.2)
+		(width 0.3)
 		(layer "F.Cu")
 		(net 4)
@@
 		(start 74.455 51.6)
 		(end 74.949 52.094)
-		(width 0.2)
+		(width 0.3)
 		(layer "F.Cu")
 		(net 4)
@@
 		(start 73.955 48.6)
 		(end 74.455 49.1)
-		(width 0.2)
+		(width 0.3)
 		(layer "F.Cu")
 		(net 4)
@@
 		(start 75.756 53.035968)
 		(end 74.826968 53.965)
-		(width 0.2)
+		(width 0.3)
 		(layer "F.Cu")
 		(net 4)
@@
 		(start 75.495968 52.094)
 		(end 75.756 52.354032)
-		(width 0.2)
+		(width 0.3)
 		(layer "F.Cu")
 		(net 4)
@@
 		(start 75.805 49.2)
 		(end 74.555 49.2)
-		(width 0.2)
+		(width 0.3)
 		(layer "F.Cu")
 		(net 4)
@@
 		(start 69.905 61.35)
 		(end 72.555 58.7)
-		(width 0.2)
+		(width 0.3)
 		(layer "F.Cu")
 		(net 5)
@@
 		(start 72.555 55.6)
 		(end 72.92 55.235)
-		(width 0.2)
+		(width 0.3)
 		(layer "F.Cu")
 		(net 5)
@@
 		(start 77.105 50.45)
 		(end 77.105 49.2)
-		(width 0.2)
+		(width 0.3)
 		(layer "F.Cu")
 		(net 5)
@@
 		(start 76.455 51.1)
 		(end 77.105 50.45)
-		(width 0.2)
+		(width 0.3)
 		(layer "F.Cu")
 		(net 5)
@@
 		(start 76.455 51.1)
 		(end 76.455 54.1)
-		(width 0.2)
+		(width 0.3)
 		(layer "F.Cu")
 		(net 5)
@@
 		(start 72.555 58.7)
 		(end 72.555 55.6)
-		(width 0.2)
+		(width 0.3)
 		(layer "F.Cu")
 		(net 5)
@@
 		(start 75.28 51.1)
 		(end 76.455 51.1)
-		(width 0.2)
+		(width 0.3)
 		(layer "F.Cu")
 		(net 5)
@@
 		(start 72.92 55.235)
 		(end 74.48 55.235)
-		(width 0.2)
+		(width 0.3)
 		(layer "F.Cu")
 		(net 5)
@@
 		(start 75.32 55.235)
 		(end 74.48 55.235)
-		(width 0.2)
+		(width 0.3)
 		(layer "F.Cu")
 		(net 5)
@@
 		(start 68.9 61.35)
 		(end 69.905 61.35)
-		(width 0.2)
+		(width 0.3)
 		(layer "F.Cu")
 		(net 5)
@@
 		(start 76.455 54.1)
 		(end 75.32 55.235)
-		(width 0.2)
+		(width 0.3)
 		(layer "F.Cu")
 		(net 5)
@@
 		(start 81.5 52)
 		(end 81.5 49)
-		(width 0.2)
+		(width 0.3)
 		(layer "F.Cu")
 		(net 44)
@@
 		(start 82.08 48.42)
 		(end 83.705 48.42)
-		(width 0.2)
+		(width 0.3)
 		(layer "F.Cu")
 		(net 44)
@@
 		(start 79.43 52.695)
 		(end 80.805 52.695)
-		(width 0.2)
+		(width 0.3)
 		(layer "F.Cu")
 		(net 44)
@@
 		(start 80.805 52.695)
 		(end 81.5 52)
-		(width 0.2)
+		(width 0.3)
 		(layer "F.Cu")
 		(net 44)
@@
 		(start 81.5 49)
 		(end 82.08 48.42)
-		(width 0.2)
+		(width 0.3)
 		(layer "F.Cu")
 		(net 44)
@@
 		(start 82.31 49.69)
 		(end 83.705 49.69)
-		(width 0.2)
+		(width 0.3)
 		(layer "F.Cu")
 		(net 46)
@@
 		(start 82 54.909999)
 		(end 82 50)
-		(width 0.2)
+		(width 0.3)
 		(layer "F.Cu")
 		(net 46)
@@
 		(start 80.404999 56.505)
 		(end 82 54.909999)
-		(width 0.2)
+		(width 0.3)
 		(layer "F.Cu")
 		(net 46)
@@
 		(start 79.43 56.505)
 		(end 80.404999 56.505)
-		(width 0.2)
+		(width 0.3)
 		(layer "F.Cu")
 		(net 46)
@@
 		(start 82 50)
 		(end 82.31 49.69)
-		(width 0.2)
+		(width 0.3)
 		(layer "F.Cu")
 		(net 46)
@@
 		(start 72.455 49.925)
 		(end 72.455 47.6)
-		(width 0.2)
+		(width 0.3)
 		(layer "F.Cu")
 		(net 95)
@@
 		(start 72.455 47.6)
 		(end 73.455 46.6)
-		(width 0.2)
+		(width 0.3)
 		(layer "F.Cu")
 		(net 95)
@@
 		(start 73.455 46.6)
 		(end 73.455 46.06)
-		(width 0.2)
+		(width 0.3)
 		(layer "F.Cu")
 		(net 95)
@@
 		(start 73.63 51.1)
 		(end 72.455 49.925)
-		(width 0.2)
+		(width 0.3)
 		(layer "F.Cu")
 		(net 95)

Commit message: September order final commit
Parts:
- C6: value 100uF -> 100nF
Connections:
- IC1 pad 24: unconnected-(IC1-IO47-Pad24) -> /USER_LED
- IC1 pad 26: /USER_LED -> unconnected-(IC1-IO45-Pad26)
- R9 pad 2: +5V -> VBUS
Routing:
- net +5V: track 29.8 -> 14.1 mm
- net VBUS: track 30.8 -> 42.9 mm
- net /USER_LED: track 2.60 -> 4.28 mm
- net VCC: track 37.1 -> 36.3 mm
Other:
- board text added: "SDM-26 DAQ IMU v1.0"

Commit message: Final Final update for September order
Parts:
- added G***: LOGO, LOGO, B.Cu at (86.4, 59.9)
- added G***: LOGO, LOGO, B.Cu at (92.3, 50.5)
Other:
- board text added: "First Board"
- board text added: "JLCJLCJLCJLC"
