File: 2026/IMU/SDM26_IMU_V1.0/SDM26_IMU_V1.0.kicad_pcb (KiCad board)
At the start: 4 copper layers, 52 x 41 mm, 60 parts, among them IC1 ESP32-S3-WROOM-1-N8R8, IC2 ISM330DHCXTR, IC3 CP2102N-A02-GQFN28, IC4 TPS259250DRCR, IC5 MIC37100-3.3WS, IC6 TPS2116DRLR, IC7 TLP175A_TPL,E, J1 Conn_01x04_Socket, J2 USB_B_Micro, Q1 MMBT2222LT1G, Q2 MMBT2222LT1G, U1 USBLC6-2SC6, U2 SN65HVD230

Commit message: Library maintenance
edited some 3dmodles to point to their footprints. edited symbols and footprints to link properly. edited footprint and symbol library names in all projects 2026-2027 to use the same library nick name "SDM" for both  symbol and footprint.
all users must delete their old lib and make a new one named SDM for symbol and footprint.
Parts:
- D1: footprint SDM_MiscFootprint:SOT65P210X110-3N -> SDM:SOT65P210X110-3N
- IC2: footprint SDM_MiscFootprint:LSM6DS3USTR -> SDM:LSM6DS3USTR
- IC3: footprint SDM_MiscFootprint:QFN50P500X500X80-29N-D -> SDM:QFN50P500X500X80-29N-D
- IC4: footprint SDM_MiscFootprint:SON50P300X300X100-11L-D -> SDM:SON50P300X300X100-11L-D
- IC7: footprint SDM_MiscFootprint:TLP266J -> SDM:TLP266J
- LED1, LED2: footprint SDM_MiscFootprint:LEDC1608X80N -> SDM:LEDC1608X80N
- Q1: footprint SDM_MiscFootprint:SOT96P237X111-3N -> SDM:SOT96P237X111-3N
Changed lines of the file:
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@@
 		)
 	)
-	(footprint "SDM_MiscFootprint:SON50P300X300X100-11L-D"
+	(footprint "SDM:SON50P300X300X100-11L-D"
 		(layer "F.Cu")
 		(at 83.955 76.6)
@@
 		)
 	)
-	(footprint "SDM_MiscFootprint:SOT96P237X111-3N"
+	(footprint "SDM:SOT96P237X111-3N"
 		(layer "F.Cu")
 		(at 85 66.55 90)
@@
 		)
 		(embedded_fonts no)
-		(model "${MISC_3D}/Transistors/MMBT2222LT1G.step"
+		(model "${SDM_MISC_3D}/MMBT2222LT1G.step"
 			(offset
 				(xyz 0 0 0)
@@
 		)
 	)
-	(footprint "SDM_MiscFootprint:LEDC1608X80N"
+	(footprint "SDM:LEDC1608X80N"
 		(layer "F.Cu")
 		(at 102 65.3 180)
@@
 		)
 	)
-	(footprint "SDM_MiscFootprint:LSM6DS3USTR"
+	(footprint "SDM:LSM6DS3USTR"
 		(layer "F.Cu")
 		(at 97.118 70.512)
@@
 		)
 	)
-	(footprint "SDM_MiscFootprint:TLP266J"
+	(footprint "SDM:TLP266J"
 		(layer "F.Cu")
 		(at 70.355 47.33)
@@
 		)
 	)
-	(footprint "SDM_MiscFootprint:SOT65P210X110-3N"
+	(footprint "SDM:SOT65P210X110-3N"
 		(layer "F.Cu")
 		(at 76.455 48.15 90)
@@
 		)
 		(embedded_fonts no)
-		(model "${MISC_3D}/Transistors/MMBT2222LT1G.step"
+		(model "${SDM_MISC_3D}/MMBT2222LT1G.step"
 			(offset
 				(xyz 0 0 0)
@@
 		)
 	)
-	(footprint "SDM_MiscFootprint:LEDC1608X80N"
+	(footprint "SDM:LEDC1608X80N"
 		(layer "F.Cu")
 		(at 87.95 80.8 180)
@@
 		)
 	)
-	(footprint "SDM_MiscFootprint:QFN50P500X500X80-29N-D"
+	(footprint "SDM:QFN50P500X500X80-29N-D"
 		(layer "F.Cu")
 		(at 75.305 67.6)
