File: 2026/TimingGates/SDM26_TimingGates_V2.0/SDM26_TimingGates_V2.0.kicad_pcb (KiCad board)
At the start: 4 copper layers, 48 x 35 mm, 29 parts, among them IC1 MIC37100-3.3WS, IC2 ESP32-S3-WROOM-1U-N8R8, IC3 CP2102N-A02-GQFN28, IC4 DS3231SN#, J1 ESP_USB, J2 Conn_01x04_Socket, Q1 MMBT2222LT1G, Q2 MMBT2222LT1G, U1 USBLC6-2SC6

Commit message: Timing Gates 2.0 Commit
Parts:
- removed the IC1 at (115.8, 131.6)
- added C7: 4.7uF, Capacitor_SMD:C_0603_1608Metric, F.Cu at (115.0, 128.1)
- added C8: 4.7uF, Capacitor_SMD:C_0603_1608Metric, F.Cu at (114.2, 124.3)
- added C9: 10uF, Capacitor_SMD:C_0603_1608Metric, F.Cu at (114.2, 125.8)
- added G***: LOGO, LOGO, B.Cu at (113.5, 123.8)
- added LED1: 150060RS75000, SDM_MiscFootprint:LEDC1608X80N, F.Cu at (106.8, 126.3)
- added LED2: 150060GS75000, SDM_MiscFootprint:LEDC1608X80N, F.Cu at (118.2, 134.0)
- added LED3: 150060GS75000, SDM_MiscFootprint:LEDC1608X80N, F.Cu at (113.3, 134.0)
- added R10: 10k, Resistor_SMD:R_0603_1608Metric, F.Cu at (125.8, 105.0)
- added R11: 68, Resistor_SMD:R_0603_1608Metric, F.Cu at (109.3, 127.1)
- added R12: 5.05, Resistor_SMD:R_0603_1608Metric, F.Cu at (115.8, 133.2)
- added R13: 5.05, Resistor_SMD:R_0603_1608Metric, F.Cu at (110.9, 133.2)
- C2: value 10uF -> 1uF
- C3, C4: value 100nF -> 1uF
- moved C2 18.5 mm to (124.0, 120.3), turned to 180 degrees
- moved R7 13.3 mm to (119.0, 131.0), turned to 0 degrees
- moved C1 6.44 mm to (116.5, 127.3)
- moved C5 6.43 mm to (119.0, 128.0), turned to 0 degrees
- moved R9 6.14 mm to (119.0, 129.5), turned to 0 degrees
- moved R8 1.90 mm to (119.0, 126.5), turned to 0 degrees
- moved G*** 0.82 mm to (112.7, 109.2)
- turned C3 to 90 degrees
- renumbered IC2 to IC1, IC3 to IC2, IC4 to IC3
Connections:
- C2 pad 1: GND -> /CHIP_PU
- C2 pad 2: +3.3V -> GND
- C3 pad 1: GND -> +3.3V
- C3 pad 2: +3.3V -> GND
- IC1 pad 13: unconnected-(IC2-IO19-Pad13) -> /USER_LED2
- IC1 pad 14: unconnected-(IC2-IO20-Pad14) -> /USER_LED1
- IC2 pad 7: +3.3V -> VBUS
Routing:
- net /USER_LED2: track 0.00 -> 29.3 mm, vias 0 -> 4
- net /USER_LED1: track 0.00 -> 27.7 mm, vias 0 -> 4
- net Net-(IC2-VBUS): track 10.3 -> 6.36 mm
- net GND: track 46.5 -> 49.5 mm, vias 33 -> 28
- net VBUS: track 50.4 -> 53.0 mm
- net +3.3V: track 12.6 -> 14.8 mm
- net Net-(LED2-A): track 0.00 -> 1.71 mm
- net Net-(LED1-A): track 0.00 -> 1.71 mm
- net Net-(LED3-A): track 0.00 -> 1.66 mm
- net Net-(H3-+): track 53.4 -> 53.9 mm
Other:
- board text added: "SDM-26 DAQ Timing Gates V2.0"

Commit message: Updates Before September Order
Parts:
- added C10: 10uF, Capacitor_SMD:C_0603_1608Metric, F.Cu at (125.8, 105.0)
- added R14: 10k, Resistor_SMD:R_0603_1608Metric, F.Cu at (137.3, 133.3)
- added R15: 10k, Resistor_SMD:R_0603_1608Metric, F.Cu at (143.3, 133.3)
- C1, C9: value 10uF -> 100uF
- C3: value 1uF -> 100nF
- LED2: value 150060GS75000 -> RED; footprint SDM_MiscFootprint:LEDC1608X80N -> SDM_MiscFootprint:SSFLXH100LID01
- R12: value 5.05 -> 220
- moved R13 13.4 mm to (114.2, 120.2), turned to 180 degrees
- moved R12 5.94 mm to (111.6, 129.0), turned to 0 degrees
- moved LED3 5.02 mm to (118.3, 133.6)
- moved LED2 3.92 mm to (114.3, 133.7), turned to 0 degrees
- moved R10 3.00 mm to (125.8, 108.0)
- moved R6 1.84 mm to (136.6, 130.9)
- moved R4 0.76 mm to (135.7, 128.6), turned to 180 degrees
- moved C6 0.40 mm to (140.3, 133.3)
Routing:
- net Net-(LED3-A): track 1.66 -> 15.8 mm, vias 0 -> 2
- net /USER_LED2: track 29.3 -> 15.6 mm
- net /INT: track 14.7 -> 18.1 mm
- net Net-(LED2-A): track 1.71 -> 4.96 mm
- net +3.3V: track 14.8 -> 17.7 mm, vias 7 -> 10
- net /32KHz: track 14.9 -> 17.1 mm
- net /I2C1_SCL: track 23.6 -> 22.0 mm
- net /USER_LED1: track 27.7 -> 26.5 mm

Commit message: September order final commit
Parts:
- C1, C9: value 100uF -> 100nF
- R4, R6: value 10k -> 2.2k
