File: 2026/Wheelboard/SDM26_Wheelboard_V2.0/SDM26_Wheelboard_V2.0.kicad_pcb (KiCad board)
At the start: 4 copper layers, 36 x 34 mm, 70 parts, among them IC1 ESP32-S3-WROOM-1-N8R8, IC2 TLP175A_TPL,E, IC3 MIC37100-3.3WS, IC4 TPS2116DRLR, IC5 MAX9924UAUB+, IC6 CP2102N-A02-GQFN28, IC7 TLP175A_TPL,E, IC8 MCP2518FDT-E_SL, J1 Conn_01x04_Socket, J2 Conn_01x04_Socket, J3 Conn_01x04_Socket, J4 Conn_01x04_Socket, J5 Conn_01x02_Socket, J6 Conn_01x02_Socket, J7 ESP_USB, Q1 SOT96P237X111-3N, Q2 SOT96P237X111-3N, U1 SN65HVD230, U2 USBLC6-2SC6, U3 SN65HVD230, Y1 ABM3B-20.000MHZ-10-1-U-T

Commit message: Finalizing Wheelboards
Parts:
- removed C15, C17, C6: 100nF, Capacitor_SMD:C_0603_1608Metric
- removed C18, C8: 1uF, Capacitor_SMD:C_0603_1608Metric
- removed C19: 15pF, Capacitor_SMD:C_0603_1608Metric
- removed IC7: TLP175A_TPL,E, SDM_MiscFootprint:TLP266J
- removed R10: 2.2k, Resistor_SMD:R_0603_1608Metric
- removed R21: 47.5k, Resistor_SMD:R_0603_1608Metric
- removed R3: 120, Resistor_SMD:R_0603_1608Metric
- removed R6: 68, Resistor_SMD:R_0603_1608Metric
- removed U3: SN65HVD230, Package_SO:SOIC-8_3.9x4.9mm_P1.27mm
- added C21: 100nF, Capacitor_SMD:C_0603_1608Metric, B.Cu at (152.9, 91.1)
- added C22: 1uF, Capacitor_SMD:C_0603_1608Metric, B.Cu at (155.8, 92.8)
- added C29: 15pF, Capacitor_SMD:C_0603_1608Metric, F.Cu at (142.8, 92.9)
- added C30: 15pF, Capacitor_SMD:C_0603_1608Metric, F.Cu at (142.1, 95.2)
- added IC9: MAX9924UAUB+, SDM_MiscFootprint:SOP50P490X110-10L, B.Cu at (158.2, 96.8)
- added R24: 22.1K, Resistor_SMD:R_0603_1608Metric, B.Cu at (158.1, 92.1)
- added R25: 1k, Resistor_SMD:R_0603_1608Metric, B.Cu at (154.6, 95.0)
- added R26: 47.5k, Resistor_SMD:R_0603_1608Metric, B.Cu at (155.8, 91.3)
- added R5: 10k, Resistor_SMD:R_0603_1608Metric, F.Cu at (161.9, 111.8)
- added R55: 1M, Resistor_SMD:R_0603_1608Metric, F.Cu at (149.1, 89.9)
- added U4: USBLC6-2SC6, Package_TO_SOT_SMD:SOT-23-6, B.Cu at (146.4, 87.9)
- C10, C11, C3, C4, C9, J2, J4, LED3, Q1, Q2, R7: moved to B.Cu
- C12: value 1nF -> 100nF
- C13: value 4.7uF -> 100nF; moved to F.Cu
- C14, J1, J3, J5: moved to F.Cu
- C16: value 100nF -> 1nF; moved to B.Cu
- C20: value 15pF -> 4.7uF; moved to B.Cu
- H1: value M3 -> M2; moved to F.Cu
- H2: value M3 -> M2
- IC1: value ESP32-S3-WROOM-1-N8R8 -> MCP2518FDT-H_QBB; footprint SDM_MiscFootprint:ESP32S3WROOM1N8R8 -> SDM_MiscFootprint:SON65P300X450X90-15L-D
- IC2: value TLP175A_TPL,E -> ESP32-S3-WROOM-1-N8R8; footprint SDM_MiscFootprint:TLP266J -> SDM_MiscFootprint:ESP32S3WROOM1N8R8
- IC3: value MIC37100-3.3WS -> TLP175A_TPL,E; footprint SDM_MiscFootprint:SOT230P700X180-4N -> SDM_MiscFootprint:TLP266J
- IC4: value TPS2116DRLR -> MIC37100-3.3WS; footprint SDM_MiscFootprint:SOTFL50P160X60-8L -> SDM_MiscFootprint:SOT230P700X180-4N; moved to B.Cu
- IC5: value MAX9924UAUB+ -> TPS2116DRLR; footprint SDM_MiscFootprint:SOP50P490X110-10L -> SDM_MiscFootprint:SOTFL50P160X60-8L
- IC6: value CP2102N-A02-GQFN28 -> TLP175A_TPL,E; footprint SDM_MiscFootprint:QFN50P500X500X80-29N-D -> SDM_MiscFootprint:TLP266J; moved to F.Cu
- IC8: value MCP2518FDT-E_SL -> CP2102N-A02-GQFN28; footprint SDM_MiscFootprint:SOIC127P600X175-14L -> SDM_MiscFootprint:QFN50P500X500X80-29N-D; moved to B.Cu
- J6: value Conn_01x02_Socket -> ESP_USB; footprint Connector_JST:JST_XH_S2B-XH-A_1x02_P2.50mm_Horizontal -> Connector_USB:USB_Micro-B_Molex-105017-0001
- J7: value ESP_USB -> Conn_01x02_Socket; footprint Connector_USB:USB_Micro-B_Molex-105017-0001 -> Connector_JST:JST_XH_S2B-XH-A_1x02_P2.50mm_Horizontal; moved to B.Cu
- R11, R4: value 10k -> 120
- R12, R15: value 10k -> 2.2k
- R13: value 1k -> 5.05; moved to B.Cu
- R16, R17: value 27 -> 10k; moved to B.Cu
- R18: value 22.1K -> 1k; moved to B.Cu
- R19: value 120 -> 10k; moved to B.Cu
- R20: value 1k -> 10k; moved to B.Cu
- R22: value 10k -> 27
- R23: value 1M -> 27
- R8: value 2.2k -> 68; moved to B.Cu
- R9: value 5.05 -> 10k
- U2: value USBLC6-2SC6 -> SN65HVD230; footprint Package_TO_SOT_SMD:SOT-23-6 -> Package_SO:SOIC-8_3.9x4.9mm_P1.27mm
- moved C7 107.6 mm to (160.4, 111.8), turned to 90 degrees
- moved IC8 105.3 mm to (150.8, 95.0), turned to -90 degrees
- moved C16 102.6 mm to (163.0, 98.8), turned to 180 degrees
- moved C9 102.3 mm to (162.4, 91.6), turned to 90 degrees
- moved R15 100.0 mm to (163.9, 112.5), turned to 90 degrees
- moved C10 98.7 mm to (159.7, 91.5), turned to 90 degrees
- moved R4 95.8 mm to (165.5, 89.4), turned to -90 degrees
- moved R11 93.5 mm to (165.5, 92.4), turned to 90 degrees
- moved C2 93.3 mm to (152.8, 82.0), turned to 180 degrees
- moved C3 92.4 mm to (152.8, 82.0), turned to 180 degrees
- moved R9 91.5 mm to (165.6, 82.6), turned to 90 degrees
- moved R19 91.5 mm to (163.0, 97.1), turned to 180 degrees
- moved Q1 85.3 mm to (145.9, 91.9), turned to 90 degrees
- moved C20 84.9 mm to (152.7, 89.7)
- moved R7 81.5 mm to (155.9, 82.0)
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Connections:
- C12 pad 1: Net-(IC5-IN+) -> +3.3V
- C12 pad 2: Net-(IC5-IN-) -> GND
- C14 pad 1: GND -> +3.3V
- C14 pad 2: +3.3V -> GND
- C16 pad 1: +3.3V -> Net-(IC9-IN+)
- C16 pad 2: GND -> Net-(IC9-IN-)
- C20 pad 1: Net-(IC8-OSC1) -> +3.3V
- IC1 pad 1: GND -> /CAN2_RTX
- IC1 pad 10: /CAN1_RTX -> /SPI_SCK
- IC1 pad 11: /CAN1_CTX -> /SPI_MOSI
- IC1 pad 12: /CAN2_TERM -> /SPI_MISO
- IC1 pad 14: /SPI_MISO -> +3.3V
- IC1 pad 15: unconnected-(IC1-IO3-Pad15) -> GND
- IC1 pad 2: +3.3V -> /CAN2_CTX
- IC1 pad 3: /CHIP_PU -> unconnected-(IC1-CLKO/SOF-Pad3)
- IC1 pad 4: /I2C1_SDA -> /CAN_2_INT
- IC1 pad 5: /I2C1_SCL -> Net-(IC1-OSC2)
- IC1 pad 6: /HE_OUTPUT -> Net-(IC1-OSC1)
- IC1 pad 7: unconnected-(IC1-IO7-Pad7) -> GND
- IC1 pad 8: unconnected-(IC1-IO15-Pad8) -> /CAN_2_INT1
- IC1 pad 9: /CAN1_TERM -> /CAN_2_INT0
- IC2 pad 1: /CAN1_TERM -> GND
- IC2 pad 3: GND -> /CHIP_PU
- IC2 pad 4: /CAN1- -> /I2C1_SDA
- IC2 pad 6: Net-(IC2-Pad6) -> /HE_OUTPUT
- IC3 pad 1: +5V -> /CAN1_TERM
- IC3 pad 3: +3.3V -> GND
- IC3 pad 4: GND -> /CAN1-
- IC4 pad 1: GND -> +5V
- IC4 pad 2: +5V -> GND
- IC4 pad 3: VCC -> +3.3V
- IC4 pad 4: Net-(IC4-PR1) -> GND
- IC5 pad 1: Net-(IC5-IN+) -> GND
- IC5 pad 2: Net-(IC5-IN-) -> +5V
- IC5 pad 3: unconnected-(IC5-N.C.-Pad3) -> VCC
- IC5 pad 4: GND -> Net-(IC5-PR1)
- IC5 pad 5: GND -> VCC
- IC5 pad 6: GND -> VBUS
- IC5 pad 7: /HE_OUTPUT -> +5V
- IC5 pad 8: unconnected-(IC5-EXT-Pad8) -> Net-(IC5-ST)
- IC6 pad 1: unconnected-(IC6-DCD-Pad1) -> /CAN2_TERM
- IC6 pad 4: /PROG_D+ -> /CAN2-
- IC6 pad 6: +3.3V -> Net-(IC6-Pad6)
- IC8 pad 1: /CAN2_CTX -> unconnected-(IC8-DCD-Pad1)
- IC8 pad 10: /SPI_SCK -> unconnected-(IC8-NC-Pad10)
- IC8 pad 11: /SPI_MOSI -> unconnected-(IC8-SUSPENDB-Pad11)
- IC8 pad 12: /SPI_MISO -> unconnected-(IC8-SUSPEND-Pad12)
- IC8 pad 13: /CAN2_CS -> unconnected-(IC8-CHREN-Pad13)
- IC8 pad 14: +3.3V -> unconnected-(IC8-CHR1-Pad14)
- IC8 pad 2: /CAN2_RTX -> unconnected-(IC8-RI/CLK-Pad2)
- IC8 pad 3: unconnected-(IC8-CLKO/SOF-Pad3) -> GND
- IC8 pad 4: /CAN_2_INT -> /PROG_D+
- IC8 pad 5: Net-(IC8-OSC2) -> /PROG_D-
- IC8 pad 6: Net-(IC8-OSC1) -> +3.3V
- IC8 pad 7: GND -> +3.3V
- IC8 pad 8: /CAN_2_INT1 -> Net-(IC8-VBUS)
- IC8 pad 9: /CAN_2_INT0 -> Net-(IC8-RSTB)
- J6 pad 1: /WSPD- -> VBUS
- J6 pad 2: /WSPD+ -> /USBM_D-
- J7 pad 1: VBUS -> /WSPD-
- J7 pad 2: /USBM_D- -> /WSPD+
- Q1 pad 3: Net-(IC6-RTS) -> Net-(IC8-RTS)
- Q2 pad 3: Net-(IC6-DTR) -> Net-(IC8-DTR)
- R1 pad 1: Net-(IC4-PR1) -> Net-(IC5-PR1)
- R11 pad 1: Net-(Q1-B) -> Net-(IC6-Pad6)
- R11 pad 2: Net-(IC6-DTR) -> /CAN2+
- R12 pad 1: /WSPD+ -> /I2C1_SCL
- R12 pad 2: Net-(IC5-IN+) -> +3.3V
- R13 pad 1: +3.3V -> /USER_LED
- R13 pad 2: /HE_OUTPUT -> Net-(LED2-A)
- R14 pad 1: /WSPD- -> GND
- R14 pad 2: Net-(IC5-IN-) -> Net-(U2-Rs)
- R15 pad 1: Net-(Q2-B) -> +3.3V
- R15 pad 2: Net-(IC6-RTS) -> /I2C1_SDA
- R16 pad 1: Net-(R16-Pad1) -> Net-(Q1-B)
- R16 pad 2: /PROG_D+ -> Net-(IC8-DTR)
- R17 pad 1: /PROG_D- -> /WSPD+
- R17 pad 2: Net-(R17-Pad2) -> Net-(IC9-IN+)
- R18 pad 1: Net-(IC6-VBUS) -> +3.3V
- R18 pad 2: VBUS -> /HE_OUTPUT
- R19 pad 1: Net-(IC7-Pad6) -> /WSPD-
- R19 pad 2: /CAN2+ -> Net-(IC9-IN-)
- R2 pad 2: Net-(IC4-PR1) -> Net-(IC5-PR1)
- R20 pad 1: Net-(IC6-RSTB) -> Net-(Q2-B)
- R20 pad 2: +3.3V -> Net-(IC8-RTS)
- R22 pad 1: GND -> Net-(R22-Pad1)
- R22 pad 2: Net-(U3-Rs) -> /PROG_D+
- R23 pad 1: Net-(IC8-OSC2) -> /PROG_D-
- R23 pad 2: Net-(IC8-OSC1) -> Net-(R23-Pad2)
- R4 pad 1: +3.3V -> Net-(IC3-Pad6)
- R4 pad 2: /CHIP_PU -> /CAN1+
- R7 pad 1: GND -> Net-(IC5-ST)
- R7 pad 2: Net-(U1-Rs) -> +5V
- R8 pad 1: /I2C1_SDA -> GND
- R8 pad 2: +3.3V -> Net-(LED1-K)
- R9 pad 1: /USER_LED -> GND
- R9 pad 2: Net-(LED2-A) -> Net-(U1-Rs)
- U2 pad 1: Net-(R16-Pad1) -> /CAN2_RTX
- U2 pad 3: Net-(R17-Pad2) -> +3.3V
- U2 pad 4: /USBM_D- -> /CAN2_CTX
- U2 pad 5: VBUS -> unconnected-(U2-Vref-Pad5)
- U2 pad 6: /USBM_D+ -> /CAN2-
- Y1 pad 1: Net-(IC8-OSC1) -> Net-(IC1-OSC1)
- Y1 pad 3: Net-(IC8-OSC2) -> Net-(IC1-OSC2)
Routing:
- net GND: track 4.87 -> 76.7 mm, vias 3 -> 35
- net /CHIP_PU: track 0.00 -> 49.4 mm, vias 0 -> 3
- net +3.3V: track 11.1 -> 40.1 mm, vias 4 -> 11
- net /CAN1+: track 0.00 -> 27.7 mm, vias 0 -> 1
- net /CAN1_TERM: track 0.00 -> 27.0 mm, vias 0 -> 2
- net /CAN1_CTX: track 0.00 -> 23.0 mm, vias 0 -> 2
- net /CAN1_RTX: track 0.00 -> 23.0 mm, vias 0 -> 2
- net /UOTXD: track 0.00 -> 21.2 mm, vias 0 -> 1
- net Net-(IC8-RTS): track 0.00 -> 21.0 mm, vias 0 -> 2
- net /UORXD: track 0.00 -> 20.6 mm, vias 0 -> 1
- net /CAN2+: track 0.00 -> 20.3 mm
- net /CAN2-: track 0.00 -> 20.0 mm, vias 0 -> 1
- net /HE_OUTPUT: track 0.00 -> 19.8 mm, vias 0 -> 1
- net /CAN1-: track 0.00 -> 19.3 mm
- net /USER_LED: track 0.00 -> 18.2 mm, vias 0 -> 1
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- added copper zone on In2.Cu, net VCC
- removed copper zone on B.Cu, net GND
Other:
- board size 36 x 34 mm -> 36 x 35.5 mm

Commit message: Misc (A lot and I don't wanna organize 😛)
Parts:
- added G***: LOGO, LOGO, B.Cu at (160.0, 111.0)
- added G***: LOGO, Library:sdmlogo, B.Cu at (149.4, 100.5)
- added G***: LOGO, Library:wheelyboi, B.Cu at (156.7, 100.6)
Routing:
- net /HE_OUTPUT: track 19.8 -> 21.4 mm
Other:
- board text added: "JLCJLCJLCJLC"
- board text added: "SDM26 DAQ Wheelboard V2.0"
- board text added: "You look lost baby girl"
