File: 2026/Wheelboard/SDM26_Wheelboard_V2.0/SDM26_Wheelboard_V2.0.kicad_pcb (KiCad board)
At the start: 4 copper layers, 36 x 35.5 mm, 72 parts, among them IC1 MCP2518FDT-H_QBB, IC2 ESP32-S3-WROOM-1-N8R8, IC3 TLP175A_TPL,E, IC4 MIC37100-3.3WS, IC5 TPS2116DRLR, IC6 TLP175A_TPL,E, IC8 CP2102N-A02-GQFN28, IC9 MAX9924UAUB+, J1 Conn_01x04_Socket, J2 Conn_01x04_Socket, J3 Conn_01x04_Socket, J4 Conn_01x04_Socket, J5 Conn_01x02_Socket, J6 ESP_USB, J7 Conn_01x02_Socket, Q1 SOT96P237X111-3N, Q2 SOT96P237X111-3N, U1 SN65HVD230, U2 SN65HVD230, U4 USBLC6-2SC6, Y1 ABM3B-20.000MHZ-10-1-U-T

Commit message: Library maintenance
edited some 3dmodles to point to their footprints. edited symbols and footprints to link properly. edited footprint and symbol library names in all projects 2026-2027 to use the same library nick name "SDM" for both  symbol and footprint.
all users must delete their old lib and make a new one named SDM for symbol and footprint.
Parts:
- D2: footprint SDM_MiscFootprint:SOT65P210X110-3N -> SDM:SOT65P210X110-3N
- IC1: footprint SDM_MiscFootprint:SON65P300X450X90-15L-D -> SDM:SON65P300X450X90-15L-D
- IC5: footprint SDM_MiscFootprint:SOTFL50P160X60-8L -> SDM:SOTFL50P160X60-8L
- IC8: footprint SDM_MiscFootprint:QFN50P500X500X80-29N-D -> SDM:QFN50P500X500X80-29N-D
- IC9: footprint SDM_MiscFootprint:SOP50P490X110-10L -> SDM:SOP50P490X110-10L
- LED1, LED2, LED3: footprint SDM_MiscFootprint:LEDC1608X80N -> SDM:LEDC1608X80N
- Y1: footprint SDM_MiscFootprint:ABM3B -> SDM:ABM3B
Changed lines of the file:
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@@
 		)
 	)
-	(footprint "SDM_MiscFootprint:LEDC1608X80N"
+	(footprint "SDM:LEDC1608X80N"
 		(layer "F.Cu")
 		(at 140.3 84.926)
@@
 		)
 	)
-	(footprint "SDM_MiscFootprint:SOT65P210X110-3N"
+	(footprint "SDM:SOT65P210X110-3N"
 		(layer "F.Cu")
 		(at 152.48 89.6)
@@
 		)
 	)
-	(footprint "SDM_MiscFootprint:SON65P300X450X90-15L-D"
+	(footprint "SDM:SON65P300X450X90-15L-D"
 		(layer "F.Cu")
 		(at 150.35 93.1 -90)
@@
 		)
 	)
-	(footprint "SDM_MiscFootprint:LEDC1608X80N"
+	(footprint "SDM:LEDC1608X80N"
 		(layer "F.Cu")
 		(at 140.3 83.026)
@@
 		)
 	)
-	(footprint "SDM_MiscFootprint:ABM3B"
+	(footprint "SDM:ABM3B"
 		(layer "F.Cu")
 		(at 145.6 92.9 90)
@@
 		)
 	)
-	(footprint "SDM_MiscFootprint:QFN50P500X500X80-29N-D"
+	(footprint "SDM:QFN50P500X500X80-29N-D"
 		(layer "B.Cu")
 		(at 150.8 94.95 -90)
@@
 		)
 	)
-	(footprint "SDM_MiscFootprint:SOP50P490X110-10L"
+	(footprint "SDM:SOP50P490X110-10L"
 		(layer "B.Cu")
 		(at 158.2 96.75 180)
@@
 		(embedded_fonts no)
 	)
-	(footprint "SDM_MiscFootprint:LEDC1608X80N"
+	(footprint "SDM:LEDC1608X80N"
 		(layer "B.Cu")
 		(at 161.65 94.2 180)
@@
 		)
 	)
-	(footprint "SDM_MiscFootprint:SOTFL50P160X60-8L"
+	(footprint "SDM:SOTFL50P160X60-8L"
 		(layer "B.Cu")
 		(at 155.7 83.925 180)
