File: 2027/SDM27_Logger_V1.0/connectors.kicad_sch (KiCad schematic)
At the start: 17 parts, among them IC2 CP2102N-A02-GQFN28, J3 USB_C_Receptacle_USB2.0_16P, Q1 MMBT2222LT1G, Q2 MMBT2222LT1G, U4 USBLC6-2SC6

Commit message: Logger updates
Parts:
- removed R15, R16: 5.1k, Resistor_SMD:R_0603_1608Metric, symbol Device:R_Small
- removed U4: USBLC6-2SC6, Package_TO_SOT_SMD:SOT-23-6, symbol Power_Protection:USBLC6-2SC6
- added C67, C68: 100nF, Capacitor_SMD:C_0603_1608Metric, symbol Device:C_Small
- added IC13: USB2512BT_M2, QFN50P600X600X100-37L-D, symbol SDM_USB:USB2512BT_M2
- added R27: 12k, Resistor_SMD:R_0603_1608Metric, symbol Device:R_Small
- added R29, R31: 27, Resistor_SMD:R_0603_1608Metric, symbol Device:R_Small
- added R32, R33: 100k, Resistor_SMD:R_0603_1608Metric, symbol Device:R_Small
- J3: value USB_C_Receptacle_USB2.0_16P -> USB_C; footprint SDM_MiscFootprint:USB_C_Receptacle_G-Switch_GT-USB-7010ASV -> SDM_MiscFootprint:USB_C_Receptacle_16P
Connections:
- net +3.3V: now also IC13.10 (VDDA33_2), IC13.15 (VDD33_1), IC13.23 (VDD33_2), IC13.29 (VDDA33_3), IC13.36 (VDDA33_4), IC13.5 (VDDA33_1)
- net GND: now also C67.2, C68.2, IC13.37 (GROUND_PAD_(VSS)), R27.2, R32.1
- net VBUS: no longer J3.A4 (VBUS), J3.A9 (VBUS), J3.B4 (VBUS), J3.B9 (VBUS)
- net C_CC2: now reaches J3.B5 (CC2)
- net C_CC1: now reaches J3.A5 (CC1)
- net C_SBU1: now reaches J3.A8 (SBU1)
- net C_SBU2: now reaches J3.B8 (SBU2)
- net USBM_D+ renamed C_USB+
- net USBM_D- renamed C_USB-
- new net: IC13.27 (VBUS_DET), R32.2, R33.1
- new net: C68.1, IC13.14 (CRFILT)
- new net: C67.1, IC13.34 (PLLFILT)
- new net: IC13.35 (RBIAS), R27.1
- new net USB_UP+: IC13.6 (NC_1), R29.1
- new net USB_UP-: IC13.7 (NC_2), R31.2
- new net USB_UP_D+: IC13.31 (USBDP_UP), R29.2
- new net USB_UP_D-: IC13.30 (USBDM_UP), R31.1
- new net VBUS HV: J3.A4 (VBUS), J3.A9 (VBUS), J3.B4 (VBUS), J3.B9 (VBUS)
- no-connect marks 18 -> 16
Other:
- moved on the sheet: C17, C48, C49, IC2, Q1, Q2, R1, R11, R12, R13, R2, R41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
