File: 2026/CAN_Splitter_Mini/4 Connector/SDM26_Splitter_Mini4_V1.0/SDM26_Splitter_Mini4_V1.0.kicad_sch (KiCad schematic)
At the start: 7 parts, among them J1 Conn_01x04_Socket, J2 Conn_01x04_Socket, J3 Conn_01x04_Socket

Commit message: Can Splitter and mini Can Splitter updates
Parts:
- added J4: Conn_01x04_Socket, SDM_MiscFootprint:JST_EH_S4B-EH_1x04_P2.50mm_Horizontal_1, symbol Connector:Conn_01x04_Socket
- J1, J2, J3: footprint Connector_JST:JST_EH_S4B-EH_1x04_P2.50mm_Horizontal -> SDM_MiscFootprint:JST_EH_S4B-EH_1x04_P2.50mm_Horizontal_1
- R1: value 220 -> 100
Connections:
- net +5V: now also J4.4 (Pin_4)
- net CANH: now also J4.2 (Pin_2)
- net CANL: now also J4.3 (Pin_3)
- net GND: now also J4.1 (Pin_1)
Changed lines of the file:
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@@
+	)
+	(junction
+		(at 64.77 82.55)
+		(diameter 0)
+		(color 0 0 0 0)
 	)
 	(junction
@@
 	)
 	(junction
+		(at 62.23 78.74)
+		(diameter 0)
+		(color 0 0 0 0)
+	)
+	(junction
 		(at 64.77 71.12)
 		(diameter 0)
@@
 	(wire
 		(pts
+			(xy 64.77 82.55) (xy 77.47 82.55)
+		)
+		(stroke
+			(width 0)
+			(type default)
+		)
+	)
+	(wire
+		(pts
 			(xy 64.77 59.69) (xy 64.77 71.12)
 		)
@@
 	(wire
 		(pts
+			(xy 77.47 90.17) (xy 62.23 90.17)
+		)
+		(stroke
+			(width 0)
+			(type default)
+		)
+	)
+	(wire
+		(pts
 			(xy 64.77 71.12) (xy 64.77 82.55)
 		)
@@
 	(wire
 		(pts
+			(xy 64.77 82.55) (xy 64.77 91.44)
+		)
+		(stroke
+			(width 0)
+			(type default)
+		)
+	)
+	(wire
+		(pts
+			(xy 71.12 85.09) (xy 77.47 85.09)
+		)
+		(stroke
+			(width 0)
+			(type default)
+		)
+	)
+	(wire
+		(pts
 			(xy 77.47 48.26) (xy 64.77 48.26)
 		)
@@
 	(wire
 		(pts
+			(xy 71.12 87.63) (xy 77.47 87.63)
+		)
+		(stroke
+			(width 0)
+			(type default)
+		)
+	)
+	(wire
+		(pts
 			(xy 71.12 73.66) (xy 77.47 73.66)
 		)
@@
 	(wire
 		(pts
-			(xy 77.47 78.74) (xy 62.23 78.74)
+			(xy 62.23 78.74) (xy 77.47 78.74)
 		)
 		(stroke
@@
 			(width 0)
 			(type default)
+		)
+	)
+	(wire
+		(pts
+			(xy 62.23 90.17) (xy 62.23 78.74)
+		)
+		(stroke
+			(width 0)
+			(type default)
+		)
+	)
+	(label "CANL"
+		(at 71.12 87.63 0)
+		(effects
+			(font
+				(size 1.27 1.27)
+			)
+			(justify left bottom)
 		)
 	)
@@
 		)
 	)
+	(label "CANH"
+		(at 71.12 85.09 0)
+		(effects
+			(font
+				(size 1.27 1.27)
+			)
+			(justify left bottom)
+		)
+	)
 	(label "CANL"
 		(at 71.12 64.77 0)
@@
 	(symbol
 		(lib_id "power:GND")
-		(at 64.77 82.55 0)
+		(at 64.77 91.44 0)
 		(unit 1)
 		(exclude_from_sim no)
@@
 		(fields_autoplaced yes)
 		(property "Reference" "#PWR02"
-			(at 64.77 88.9 0)
+			(at 64.77 97.79 0)
 			(effects
 				(font
@@
 		)
 		(property "Value" "GND"
-			(at 64.77 87.63 0)
+			(at 64.77 96.52 0)
 			(effects
 				(font
@@
 		)
 		(property "Footprint" ""
-			(at 64.77 82.55 0)
+			(at 64.77 91.44 0)
 			(effects
 				(font
@@
 		)
 		(property "Datasheet" ""
-			(at 64.77 82.55 0)
+			(at 64.77 91.44 0)
 			(effects
 				(font
@@
 		)
 		(property "Description" "Power symbol creates a global label with name \"GND\" , ground"
-			(at 64.77 82.55 0)
+			(at 64.77 91.44 0)
 			(effects
 				(font
@@
 		)
 		(instances
-			(project ""
+			(project "SDM26_Splitter_Mini4_V1.0"
 				(path "/6e35073e-5682-4b75-b4d2-cc1e866f2d05"
 					(reference "#PWR02")
+					(unit 1)
+				)
+			)
+		)
+	)
+	(symbol
+		(lib_id "Connector:Conn_01x04_Socket")
+		(at 82.55 85.09 0)
+		(unit 1)
+		(exclude_from_sim no)
+		(in_bom yes)
+		(on_board yes)
+		(dnp no)
+		(fields_autoplaced yes)
+		(property "Reference" "J4"
+			(at 83.82 85.0899 0)
+			(effects
+				(font
+					(size 1.27 1.27)
+				)
+				(justify left)
+			)
+		)
+		(property "Value" "Conn_01x04_Socket"
+			(at 83.82 87.6299 0)
+			(effects
+				(font
+					(size 1.27 1.27)
+				)
+				(justify left)
+			)
+		)
+		(property "Footprint" "SDM_MiscFootprint:JST_EH_S4B-EH_1x04_P2.50mm_Horizontal_1"
+			(at 82.55 85.09 0)
+			(effects
+				(font
+					(size 1.27 1.27)
+				)
+				(hide yes)
+			)
+		)
+		(property "Datasheet" "~"
+			(at 82.55 85.09 0)
+			(effects
+				(font
+					(size 1.27 1.27)
+				)
+				(hide yes)
+			)
+		)
+		(property "Description" "Generic connector, single row, 01x04, script generated"
+			(at 82.55 85.09 0)
+			(effects
+				(font
+					(size 1.27 1.27)
+				)
+				(hide yes)
+			)
+		)
+		(pin "2"
+		)
+		(pin "4"
+		)
+		(pin "3"
+		)
+		(pin "1"
+		)
+		(instances
+			(project "SDM26_Splitter_Mini4_V1.0"
+				(path "/6e35073e-5682-4b75-b4d2-cc1e866f2d05"
+					(reference "J4")
 					(unit 1)
 				)
@@
 			)
 		)
-		(property "Value" "220"
+		(property "Value" "100"
 			(at 92.71 38.1 90)
 			(effects
@@
 			)
 		)
-		(property "Footprint" "Connector_JST:JST_EH_S4B-EH_1x04_P2.50mm_Horizontal"
+		(property "Footprint" "SDM_MiscFootprint:JST_EH_S4B-EH_1x04_P2.50mm_Horizontal_1"
 			(at 82.55 73.66 0)
 			(effects
@@
 			)
 		)
-		(property "Footprint" "Connector_JST:JST_EH_S4B-EH_1x04_P2.50mm_Horizontal"
+		(property "Footprint" "SDM_MiscFootprint:JST_EH_S4B-EH_1x04_P2.50mm_Horizontal_1"
 			(at 82.55 62.23 0)
 			(effects
@@
 			)
 		)
-		(property "Footprint" "Connector_JST:JST_EH_S4B-EH_1x04_P2.50mm_Horizontal"
+		(property "Footprint" "SDM_MiscFootprint:JST_EH_S4B-EH_1x04_P2.50mm_Horizontal_1"
 			(at 82.55 50.8 0)
 			(effects
