File: 2026/CAN_Splitter_Mini/4 Connector/SDM26_Splitter_Mini4_V1.0/SDM26_Splitter_Mini4_V1.0.kicad_sch (KiCad schematic)
At the start: 8 parts, among them J1 Conn_01x04_Socket, J2 Conn_01x04_Socket, J3 Conn_01x04_Socket, J4 Conn_01x04_Socket

Commit message: Library maintenance
edited some 3dmodles to point to their footprints. edited symbols and footprints to link properly. edited footprint and symbol library names in all projects 2026-2027 to use the same library nick name "SDM" for both  symbol and footprint.
all users must delete their old lib and make a new one named SDM for symbol and footprint.
Parts:
- J1, J2, J3, J4: footprint SDM_MiscFootprint:JST_EH_S4B-EH_1x04_P2.50mm_Horizontal_1 -> SDM:JST_EH_S4B-EH_1x04_P2.50mm_Horizontal_1
- LED1: footprint SDM_MiscFootprint:LEDC1608X80N -> SDM:LEDC1608X80N
Changed lines of the file:
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@@
 			)
 		)
-		(property "Footprint" "SDM_MiscFootprint:JST_EH_S4B-EH_1x04_P2.50mm_Horizontal_1"
+		(property "Footprint" "SDM:JST_EH_S4B-EH_1x04_P2.50mm_Horizontal_1"
 			(at 82.55 85.09 0)
 			(effects
@@
 			)
 		)
-		(property "Footprint" "SDM_MiscFootprint:LEDC1608X80N"
+		(property "Footprint" "SDM:LEDC1608X80N"
 			(at 97.79 -53.01 0)
 			(effects
@@
 			)
 		)
-		(property "Footprint" "SDM_MiscFootprint:JST_EH_S4B-EH_1x04_P2.50mm_Horizontal_1"
+		(property "Footprint" "SDM:JST_EH_S4B-EH_1x04_P2.50mm_Horizontal_1"
 			(at 82.55 73.66 0)
 			(effects
@@
 			)
 		)
-		(property "Footprint" "SDM_MiscFootprint:JST_EH_S4B-EH_1x04_P2.50mm_Horizontal_1"
+		(property "Footprint" "SDM:JST_EH_S4B-EH_1x04_P2.50mm_Horizontal_1"
 			(at 82.55 62.23 0)
 			(effects
@@
 			)
 		)
-		(property "Footprint" "SDM_MiscFootprint:JST_EH_S4B-EH_1x04_P2.50mm_Horizontal_1"
+		(property "Footprint" "SDM:JST_EH_S4B-EH_1x04_P2.50mm_Horizontal_1"
 			(at 82.55 50.8 0)
 			(effects
