File: 2026/CAN_Splitter_Mini/4 Connector/SDM26_Splitter_Mini4_V1.0/SDM26_Splitter_Mini4_V1.0.kicad_pcb (KiCad board)
At the start: 2 copper layers, 20.3 x 32 mm, 8 parts, among them J1 Conn_01x04_Socket, J2 Conn_01x04_Socket, J3 Conn_01x04_Socket, J4 Conn_01x04_Socket

Commit message: Library maintenance
edited some 3dmodles to point to their footprints. edited symbols and footprints to link properly. edited footprint and symbol library names in all projects 2026-2027 to use the same library nick name "SDM" for both  symbol and footprint.
all users must delete their old lib and make a new one named SDM for symbol and footprint.
Parts:
- J1, J2, J3: footprint SDM_MiscFootprint:JST_EH_S4B-EH_1x04_P2.50mm_Horizontal_1 -> SDM:JST_EH_S4B-EH_1x04_P2.50mm_Horizontal_1
- LED1: footprint SDM_MiscFootprint:LEDC1608X80N -> SDM:LEDC1608X80N
Changed lines of the file:
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@@
 		(embedded_fonts no)
 	)
-	(footprint "SDM_MiscFootprint:JST_EH_S4B-EH_1x04_P2.50mm_Horizontal_1"
+	(footprint "SDM:JST_EH_S4B-EH_1x04_P2.50mm_Horizontal_1"
 		(layer "F.Cu")
 		(at 105.8 96.3 180)
@@
 		)
 		(embedded_fonts no)
-		(model "${KICAD9_3DMODEL_DIR}/Capacitor_SMD.3dshapes/C_0603_1608Metric.wrl"
+		(model "${SDM_MISC_3D}/KiCad-original/Capacitor_SMD.3dshapes/C_0603_1608Metric.wrl"
 			(offset
 				(xyz 0 0 0)
@@
 		)
 	)
-	(footprint "SDM_MiscFootprint:JST_EH_S4B-EH_1x04_P2.50mm_Horizontal_1"
+	(footprint "SDM:JST_EH_S4B-EH_1x04_P2.50mm_Horizontal_1"
 		(layer "F.Cu")
 		(at 102.5 91.25 90)
@@
 		(embedded_fonts no)
 	)
-	(footprint "SDM_MiscFootprint:LEDC1608X80N"
+	(footprint "SDM:LEDC1608X80N"
 		(layer "F.Cu")
 		(at 110.575 79.8 180)
@@
 		)
 	)
-	(footprint "SDM_MiscFootprint:JST_EH_S4B-EH_1x04_P2.50mm_Horizontal_1"
+	(footprint "SDM:JST_EH_S4B-EH_1x04_P2.50mm_Horizontal_1"
 		(layer "F.Cu")
 		(at 98.3 78.7)
