File: 2026/Telemetry/Telemetry.kicad_sch (KiCad schematic)
At the start: 46 parts, among them IC1 ESP32-S3-WROOM-1-N8R8, IC2 CP2102N-A02-GQFN28, IC3 TLP175A_TPL,E, IC4 TPS2116DRLR, IC5 MIC37100-3.3WS, J1 USB4730-GF-A, J2 Conn_01x04_Socket, Q1 MMBT2222LT1G, Q2 MMBT2222LT1G, U1 USBLC6-2SC6, U2 SN65HVD230

Commit message: Telemetry finalization
Parts:
- removed C4: 1uF, Capacitor_SMD:C_0603_1608Metric, symbol Device:C_Small
- removed LED1: GREEN, LED_SMD:LED_0603_1608Metric, symbol SDM_LED:SSF-LXH100LID-01
- removed R2: 220, Resistor_SMD:R_0603_1608Metric, symbol Device:R_Small
- removed TP1: ST_5V, TestPoint:TestPoint_Pad_1.5x1.5mm, symbol Connector:TestPoint
- added H1, H2: M2, MountingHole:MountingHole_2.2mm_M2, symbol Mechanical:MountingHole
- added LED3: 150060GS75000, SDM_MiscFootprint:LEDC1608X80N, symbol SDM_LED:150060GS75000
- IC1: footprint SDM_MiscFootprint:ESP32S3WROOM1N8R8 -> SDM_MiscFootprint:ESP32S3WROOM1UN8R8; symbol SDM_MICRO_CONTROLLER:ESP32-S3-WROOM-1-N8R8 -> SDM_MICRO_CONTROLLER:ESP32-S3-WROOM-1U-N8R8; Height 3.25 -> 3.35; Manufacturer_Part_Number ESP32-S3-WROOM-1-N8R8 -> ESP32-S3-WROOM-1U-N8R8; Mouser Part Number 356-EP32S3WROOM1N8R8 -> 356-ESP32S3WRM1UN8R8; Mouser Price/Stock https://www.mouser.co.uk/ProductDetail/Espressif-Systems/ESP32-S3-WROOM-1-N8R8?qs=7D1LtPJG0i3%2F28hKFavOpQ%3D%3D -> https://www.mouser.co.uk/ProductDetail/Espressif-Systems/ESP32-S3-WROOM-1U-N8R8?qs=Li%252BoUPsLEnvOglIa3CypaQ%3D%3D
- J1: footprint SDM_MiscFootprint:USB4730GFA -> SDM_MiscFootprint:USB_C_Receptacle_16P
- R15: value 10k -> 5.05
Connections:
- net CAN1+ is gone; now on net CAN+: J2.3 (Pin_3)
- net CAN1- is gone; now on net CAN-: J2.2 (Pin_2)
- net +5V: no longer R15.1
- net CAN_CTX: now also IC1.4 (IO4); no longer IC1.11 (IO18)
- net CAN_TERM: now also IC1.13 (IO19); no longer IC1.10 (IO17)
- net GND: now also LED3.1 (K)
- net USER_LED: now also IC1.25 (IO48), R15.2; no longer IC1.28 (IO35)
- net ST: no longer names the net of IC4.8 (ST)
- net ST: no longer R15.2
- new net: LED3.2 (A), R15.1
- no-connect marks 48 -> 49
Other:
- note added: "Power Management"
- note removed: "5v Efuse"
- note removed: "Max current calculation 12 * historic input current = 5 * output current + c c = losses due to heat, can essentialy be ignored 2025 max constant current = 400mA 12 * 0.4 = 5 * oc oc = 1.042A The lowest max rated current is TPS2116DRL @ 2.5A. Lowest Max rated current = LMC = 2.5A. Efuze Max current = EMC. Max constent current = MCC = 1.042. MCC < EMC <= LMC"
- note removed: "Power Protection"
- note removed: "TPS25925x Calculations TPS259250 = Latch on fault, TPS259251 = auto retry on fault Resitor @ ILIM pin calc = (ILIM (max current) - 0.7) / (3 * (10 ^ -5)) (LMC - 0.7) / (3 * (10 ^ -5)) = 60k Ohm Undervoltage Lockout Set = V_(UV) = ((R_1 + R_2) /R_2) * V_ENR (1.4 Given) Left open so default value of V_(UV) is 4.3V"
- note removed: "TPS563211DRLR has built in overcurrent protection @ 5.75A 12v side does not require additional overcurrent protection"
- moved on the sheet: C12, C13, C14, C8, C9, IC4, IC5, LED2, R13, R14, R17

Commit message: Added RF amplifier to telemetry board
Parts:
- added AE1, AE2: UFL, Connector_Coaxial:U.FL_Molex_MCRF_73412-0110_Vertical, symbol Device:Antenna_Shield
- added C15, C17, C21: 22pF, Capacitor_SMD:C_0603_1608Metric, symbol Device:C_Small
- added C16, C20, C4: 100nF, Capacitor_SMD:C_0603_1608Metric, symbol Device:C_Small
- added C18: 4.7uF, Capacitor_SMD:C_0603_1608Metric, symbol Device:C_Small
- added C19: 10uF, Capacitor_SMD:C_0603_1608Metric, symbol Device:C_Small
- added IC6: SE2576L-R, SDM_MiscFootprint:QFN50P300X300X90-17L-D, symbol SDM_RF_AMPLIFIER:SE2576L-R
- added R18: 0, Resistor_SMD:R_0603_1608Metric, symbol Device:R_Small
- added R19: 10k, Resistor_SMD:R_0603_1608Metric, symbol Device:R_Small
- R17: value 68 -> 100
Connections:
- net +3.3V: now also R18.1
- net +5V: now also C15.2, C16.2, C17.1, C18.2, C19.2, C20.2, C21.1, C4.1, IC6.13 (VCC2), IC6.15 (VCC1), IC6.4 (VCCO)
- net CAN_CTX: now also IC1.5 (IO5); no longer IC1.4 (IO4)
- net GND: now also AE1.2 (Shield), AE2.2 (Shield), C15.1, C16.1, C17.2, C18.1, C19.1, C20.1, C21.2, C4.2, IC6.12 (GND_5), IC6.16 (GND_6), IC6.17 (EP_(GND)), IC6.3 (GND_1), IC6.5 (GND_2), IC6.6 (GND_3), IC6.9 (GND_4), R19.1
- net USER_LED: now also IC1.4 (IO4); no longer IC1.25 (IO48)
- net AMP_DET: now reaches IC1.38 (IO2)
- net AMP_DET: now also IC6.7 (DET), R19.2
- net AMP_EN: now reaches IC1.39 (IO1)
- net AMP_EN: now also IC6.2 (EN), R18.2
- new net: AE2.1 (A), IC6.10 (RFOUT), IC6.11 (RF_OUT)
- new net: AE1.1 (A), IC6.1 (RF_IN)
- no-connect marks 49 -> 47
Other:
- note added: "100nF + 22 pF for high and very high freq filtering 4.7uF and 10uF for bulk, some mid - low freq filtering stage 2 needs more power hense larger bulk Place smaller value capacitors closer to the pin"
- note added: "Link to source"
- note added: "Power Net Names: Any voltage Like 3.3v or 5v comes from a regulator on board. VBUS comes from a USB connection VCC comes from the car/anywhere outside the board. GND/VSS = Ground"
- note added: "RF AMPLIFIER"
- note removed: "Power Net Names: Any voltage Like 3.3v or 5v comes from a regulator on board. VBUS comes from a USB connection VCC comes from the car/anywhere outside the board. GND/VDD = Ground"
- note removed: "Power Stuff"
- moved on the sheet: H1, H2
