File: 2026/Telemetry/SDM26_Telemetry_V1.0/SDM26_Telemetry_V1.0.kicad_sch (KiCad schematic)
At the start: 58 parts, among them IC1 ESP32-S3-WROOM-1-N8R8, IC2 CP2102N-A02-GQFN28, IC3 TLP175A_TPL,E, IC4 TPS2116DRLR, IC5 MIC37100-3.3WS, IC6 SE2576L-R, J1 USB4730-GF-A, J2 Conn_01x04_Socket, Q1 MMBT2222LT1G, Q2 MMBT2222LT1G, U1 USBLC6-2SC6, U2 SN65HVD230

Commit message: Renamed, added impedance matching documentation
Parts:
- added C22: 3.3nF, Capacitor_SMD:C_0603_1608Metric, symbol Device:C_Small
- AE1, AE2: footprint Connector_Coaxial:U.FL_Molex_MCRF_73412-0110_Vertical -> SDM_MiscFootprint:CONUFL001SMDT; symbol Device:Antenna_Shield -> SDM_CONNECTOR:CONUFL001-SMD-T; Height (none) -> 1.3; Manufacturer_Name (none) -> TE Connectivity; Manufacturer_Part_Number (none) -> CONUFL001-SMD-T; Mouser Part Number (none) -> N/A; Mouser Price/Stock (none) -> https://www.mouser.co.uk/ProductDetail/TE-Connectivity/CONU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
- C15: value 22pF -> 470nF
- C16, C20: value 100nF -> 470nF
- C17, C21: value 22pF -> 3.3nF
- C18: value 4.7uF -> 10uF
- C4: value 100nF -> 10uF
Connections:
- net +5V: now also C22.2; no longer C17.1
- net AMP_EN: now also C17.1
- net GND: now also AE1.3 (Shield), AE2.3 (Shield), C22.1
Other:
- note added: "470nF + 3.3nF for high and very high freq filtering 10uF for bulk, some mid - low freq filtering Place smaller value capacitors closer to the pin Also using SKY66312-11 Reference Design"
- note added: "CAN Connector"
- note added: "Link to SKY66312-11 Datasheet"
- note added: "Mounting Holes"
- note added: "USB-C"
- note removed: "100nF + 22 pF for high and very high freq filtering 4.7uF and 10uF for bulk, some mid - low freq filtering stage 2 needs more power hense larger bulk Place smaller value capacitors closer to the pin"
- moved on the sheet: C16, C20, H1, H2
