File: 2026/Telemetry/SDM26_Telemetry_V1.0/SDM26_Telemetry_V1.0.kicad_sch (KiCad schematic)
At the start: 59 parts, among them IC1 ESP32-S3-WROOM-1-N8R8, IC2 CP2102N-A02-GQFN28, IC3 TLP175A_TPL,E, IC4 TPS2116DRLR, IC5 MIC37100-3.3WS, IC6 SE2576L-R, J1 USB4730-GF-A, J2 Conn_01x04_Socket, Q1 MMBT2222LT1G, Q2 MMBT2222LT1G, U1 USBLC6-2SC6, U2 SN65HVD230

Commit message: Library maintenance
edited some 3dmodles to point to their footprints. edited symbols and footprints to link properly. edited footprint and symbol library names in all projects 2026-2027 to use the same library nick name "SDM" for both  symbol and footprint.
all users must delete their old lib and make a new one named SDM for symbol and footprint.
Parts:
- AE1, AE2: footprint SDM_MiscFootprint:CONUFL001SMDT -> SDM:CONUFL001SMDT; symbol SDM_CONNECTOR:CONUFL001-SMD-T -> SDM:CONUFL001-SMD-T
- D1: footprint SDM_MiscFootprint:SOT65P210X110-3N -> SDM:SOT65P210X110-3N; symbol SDM_ESD:ESDCAN03-2BWY -> SDM:ESDCAN03-2BWY
- IC1: footprint SDM_MiscFootprint:ESP32S3WROOM1UN8R8 -> SDM:ESP32S3WROOM1UN8R8; symbol SDM_MICRO_CONTROLLER:ESP32-S3-WROOM-1U-N8R8 -> SDM:ESP32-S3-WROOM-1U-N8R8
- IC2: footprint SDM_MiscFootprint:QFN50P500X500X80-29N-D -> SDM:QFN50P500X500X80-29N-D; symbol SDM_USBUART:CP2102N-A02-GQFN28 -> SDM:CP2102N-A02-GQFN28
- IC3: footprint SDM_MiscFootprint:TLP266J -> SDM:TLP266J
- IC4: footprint SDM_MiscFootprint:SOTFL50P160X60-8L -> SDM:SOTFL50P160X60-8L; symbol SDM_LOGIC:TPS2116DRLR -> SDM:TPS2116DRLR
- IC5: footprint SDM_MiscFootprint:SOT230P700X180-4N -> SDM:SOT230P700X180-4N; symbol SDM_VOLTAGE_REGULATORS:MIC37100-3.3WS -> SDM:MIC37100-3.3WS
- IC6: footprint SDM_MiscFootprint:QFN50P300X300X90-17L-D -> SDM:QFN50P300X300X90-17L-D; symbol SDM_RF_AMPLIFIER:SE2576L-R -> SDM:SE2576L-R
- J1: footprint SDM_MiscFootprint:USB_C_Receptacle_16P -> SDM:USB_C_Receptacle_16P
- LED2: footprint SDM_MiscFootprint:LEDC1608X80N -> SDM:LEDC1608X80N; symbol SDM_LED:150060RS75000 -> SDM:150060RS75000
- LED3: footprint SDM_MiscFootprint:LEDC1608X80N -> SDM:LEDC1608X80N; symbol SDM_LED:150060GS75000 -> SDM:150060GS75000
- Q1, Q2: footprint SDM_MiscFootprint:SOT96P237X111-3N -> SDM:SOT96P237X111-3N; symbol SDM_TRANSISTOR:MMBT2222LT1G -> SDM:MMBT2222LT1G
