File: 2026/Dash/Dash.kicad_sch (KiCad schematic)
At the start: 152 parts, among them IC1 ESP32-S3-WROOM-1-N8R8, IC10 TPS563211DRLR, IC2 CP2102N-A02-GQFN28, IC3 TLP175A_TPL,E, IC4 TPS2116DRLR, IC5 MIC37100-3.3WS, IC6 TLC5955RTQT, IC7 TLC5955RTQT, IC8 BT818Q-T, IC9 S25FL256LAGNFB010, J1 USB4730-GF-A, J2 Conn_01x40_Pin, J3 19428-0011, J4 Molex_1040310811, Q1 MMBT2222LT1G, Q2 MMBT2222LT1G, U1 USBLC6-2SC6, U10 EMIF06-MSD02N16, U2 SN65HVD230

Commit message: Hella dash edits
just cranked that shit out
Parts:
- removed C5: 4.7uF, Capacitor_SMD:C_0603_1608Metric, symbol Device:C_Small
- removed C6: 100nF, Capacitor_SMD:C_0603_1608Metric, symbol Device:C_Small
- removed C7: 1uF, Capacitor_SMD:C_0603_1608Metric, symbol Device:C_Small
- removed IC2: CP2102N-A02-GQFN28, SDM_MiscFootprint:QFN50P500X500X80-29N-D, symbol SDM_USBUART:CP2102N-A02-GQFN28
- removed Q1, Q2: MMBT2222LT1G, SDM_MiscFootprint:SOT96P237X111-3N, symbol SDM_TRANSISTOR:MMBT2222LT1G
- removed R17, R18, R19, R20, R21, R22, R23, R24, R25, R26, R27, R28, R29, R30, R32, R33, R35, R36, R37, R38, R39, R40, R41, R42, R43, R44, R45, R46, R47, R48, R49, R50, R52, R53: 33, Resistor_SMD:R_0603_1608Metric, symbol Device:R_Small
- removed R6: 47.5K, Resistor_SMD:R_0603_1608Metric, symbol Device:R_Small
- removed R7, R8: 10k, Resistor_SMD:R_0603_1608Metric, symbol Device:R_Small
- removed R9: 1k, Resistor_SMD:R_0603_1608Metric, symbol Device:R_Small
- R5: value 22.1K -> 10k
Connections:
- net +3.3V: now also IC6.33 (VCC), IC7.33 (VCC), LED10.1 (A), LED11.1 (A), LED12.1 (A), LED13.1 (A), LED14.1 (A), LED15.1 (A), LED16.1 (A), LED17.1 (A), LED18.1 (A), LED19.1 (A), LED2.1 (A), LED20.1 (A), LED21.1 (A), LED22.1 (A), LED23.1 (A), LED24.1 (A), LED25.1 (A), LED26.1 (A), LED27.1 (A), LED28.1 (A), LED29.1 (A), LED3.1 (A), LED30.1 (A), LED31.1 (A), LED32.1 (A), LED33.1 (A), LED4.1 (A), LED5.1 (A), LED6.1 (A), LED7.1 (A), LED8.1 (A), LED9.1 (A), R5.2
- net A10B: no longer IC6.26 (OUTB9)
- net A10G: no longer IC6.24 (OUTG9)
- net A10R: no longer IC6.25 (OUTR9)
- net A11B: no longer IC6.17 (OUTB10)
- net A11G: no longer IC6.15 (OUTG10)
- net A11R: no longer IC6.16 (OUTR10)
- net A12B: no longer IC6.11 (OUTB11)
- net A12G: no longer IC6.9 (OUTG11)
- net A12R: no longer IC6.10 (OUTR11)
- net A13B: no longer IC6.29 (OUTB12)
- net A13G: now also IC7.27 (OUTG12); no longer IC6.27 (OUTG12)
- net A13R: now also IC7.28 (OUTR12); no longer IC6.28 (OUTR12)
- net A14B: no longer IC6.23 (OUTB13)
- net A14G: no longer IC6.21 (OUTG13)
- net A14R: no longer IC6.22 (OUTR13)
- net A15B: no longer IC6.20 (OUTB14)
- net A15G: no longer IC6.18 (OUTG14)
- net A15R: no longer IC6.19 (OUTR14)
- net A16B: no longer IC6.14 (OUTB15)
- net A16G: no longer IC6.12 (OUTG15)
- net A16R: no longer IC6.13 (OUTR15)
- net A1B: no longer IC6.42 (OUTB0)
- net A1G: no longer IC6.44 (OUTG0)
- net A1R: no longer IC6.43 (OUTR0)
- net A2B: no longer IC6.48 (OUTB1)
- net A2G: no longer IC6.50 (OUTG1)
- net A2R: no longer IC6.49 (OUTR1)
- net A3B: no longer IC6.51 (OUTB2)
- net A3G: no longer IC6.53 (OUTG2)
- net A3R: no longer IC6.52 (OUTR2)
- net A4B: no longer IC6.1 (OUTB3)
- net A4G: no longer IC6.3 (OUTG3)
- net A4R: no longer IC6.2 (OUTR3)
- net A5B: no longer IC6.39 (OUTB4)
- net A5G: no longer IC6.41 (OUTG4)
- net A5R: no longer IC6.40 (OUTR4)
- net A6B: no longer IC6.45 (OUTB5)
- net A6G: no longer IC6.47 (OUTG5)
- net A6R: no longer IC6.46 (OUTR5)
- net A7B: no longer IC6.54 (OUTB6)
- net A7G: no longer IC6.56 (OUTG6)
- net A7R: no longer IC6.55 (OUTR6)
- net A8B: no longer IC6.4 (OUTB7)
- net A8G: no longer IC6.6 (OUTG7)
- net A8R: no longer IC6.5 (OUTR7)
- net A9B: no longer IC6.32 (OUTB8)
- net A9G: no longer IC6.30 (OUTG8)
- net A9R: no longer IC6.31 (OUTR8)
- net B0: now also IC8.47 (B0)
- net B1: now also IC8.46 (B1)
- net B10B: now also IC6.26 (OUTB9)
- net B10G: now also IC6.24 (OUTG9)
- net B10R: now also IC6.25 (OUTR9)
- net B11B: now also IC6.17 (OUTB10)
- net B11G: now also IC6.15 (OUTG10)
- net B11R: now also IC6.16 (OUTR10)
- net B12B: now also IC6.11 (OUTB11)
- net B12G: now also IC6.9 (OUTG11)
- net B12R: now also IC6.10 (OUTR11)
- net B13B: now also IC6.29 (OUTB12)
- net B13G: now also IC6.27 (OUTG12); no longer IC7.27 (OUTG12)
- net B13R: now also IC6.28 (OUTR12); no longer IC7.28 (OUTR12)
- net B14B: now also IC6.23 (OUTB13)
- net B14G: now also IC6.21 (OUTG13)
- net B14R: now also IC6.22 (OUTR13)
- net B15B: now also IC6.20 (OUTB14)
- net B15G: now also IC6.18 (OUTG14)
- net B16B: now also IC6.14 (OUTB15)
- net B16G: now also IC6.12 (OUTG15)
- net B16R: now also IC6.13 (OUTR15); no longer LED32.2 (R)
- net B1B: now also IC6.42 (OUTB0)
- net B1G: now also IC6.44 (OUTG0)
- net B1R: now also IC6.43 (OUTR0)
- net B2: now also IC8.45 (B2)
- net B2B: now also IC6.48 (OUTB1)
- net B2G: now also IC6.50 (OUTG1)
- net B2R: now also IC6.49 (OUTR1)
- net B3: now also IC8.44 (B3)
- net B3B: now also IC6.51 (OUTB2)
- net B3G: now also IC6.53 (OUTG2)
- net B3R: now also IC6.52 (OUTR2)
- net B4: now also IC8.43 (B4)
- net B4B: now also IC6.1 (OUTB3)
- net B4G: now also IC6.3 (OUTG3)
- net B4R: now also IC6.2 (OUTR3)
- net B5: now also IC8.42 (B5)
- net B5B: now also IC6.39 (OUTB4)
- net B5G: now also IC6.41 (OUTG4)
- net B5R: now also IC6.40 (OUTR4)
- net B6: now also IC8.41 (B6)
- net B6B: now also IC6.45 (OUTB5)
- net B6G: now also IC6.47 (OUTG5)
- net B6R: now also IC6.46 (OUTR5)
- net B7: now also IC8.40 (B7)
- net B7B: now also IC6.54 (OUTB6)
- net B7G: now also IC6.56 (OUTG6)
- net B7R: now also IC6.55 (OUTR6)
- net B8B: now also IC6.4 (OUTB7)
- net B8G: now also IC6.6 (OUTG7)
- net B8R: now also IC6.5 (OUTR7)
- net B9B: now also IC6.32 (OUTB8)
- net B9G: now also IC6.30 (OUTG8)
- net B9R: now also IC6.31 (OUTR8)
- net G0: now also IC8.56 (G0)
- net G1: now also IC8.55 (G1)
- net G2: now also IC8.54 (G2)
- net G3: now also IC8.53 (G3)
- net G4: now also IC8.52 (G4)
- net G5: now also IC8.51 (G5)
- net G6: now also IC8.50 (G6)
- net G7: now also IC8.49 (G7)
- net GND: now also IC6.35 (GND_2), IC6.57 (THERMAL_PAD), IC7.57 (THERMAL_PAD)
- net GPIO0: now also R5.1
- net LED_GSCLK: no longer IC1.14 (IO20)
- net LED_LAT: no longer IC1.13 (IO19)
- net PROG_D+: now also IC1.14 (IO20)
- net PROG_D-: now also IC1.13 (IO19)
- net R0: now also IC8.1 (R0)
- net R1: now also IC8.64 (R1)
- net R2: now also IC8.63 (R2)
- net R3: now also IC8.62 (R3)
- net R4: now also IC8.61 (R4)
- net R5: now also IC8.60 (R5)
- net R6: now also IC8.59 (R6)
- net R7: now also IC8.58 (R7)
- net SD_CD: no longer IC1.23 (IO21)
- net SPI_CLK: now also IC8.3 (SCK)
- net SPI_DATA0: now also IC8.4 (MISO)
- net SPI_DATA1: now also IC8.5 (MOSI)
- net SPI_DATA2: now also IC8.7 (GPIO0/IO2)
- net SPI_DATA3: now also IC8.8 (GPIO1/IO3)
- net VBUS: no longer R5.2
- net at IC9.3 (W_P#_/_IO_2): now also IC8.19 (SPIM_IO2)
- net at IC9.2 (SO/IO_1): now also IC8.18 (SPIM_MISO)
- net at IC9.5 (SI_/_IO_0): now also IC8.16 (SPIM_MOSI)
- net at IC9.6 (SCK): now also IC8.14 (SPIM_SCLK)
- net at IC9.7 (IO_3_/_RESET#): now also IC8.20 (SPIM_IO3)
- new net B15R: IC6.19 (OUTR14), LED32.2 (R)
- no-connect marks 40 -> 24
Other:
- moved on the sheet: C4
Changed lines of the file:
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@@
 (kicad_sch
-	(version 20250114)
+	(version 20260306)
 	(generator "eeschema")
-	(generator_version "9.0")
+	(generator_version "10.0")
 	(paper "User" 390 450)
