File: 2026/Dash/Dash.kicad_pcb (KiCad board)
At the start: 2 copper layers, 151 parts, among them IC1 ESP32-S3-WROOM-1-N8R8, IC10 TPS563211DRLR, IC2 CP2102N-A02-GQFN28, IC3 TLP175A_TPL,E, IC4 TPS2116DRLR, IC5 MIC37100-3.3WS, IC6 TLC5955RTQT, IC7 TLC5955RTQT, IC8 BT818Q-T, IC9 S25FL256LAGNFB010, J1 USB4730-GF-A, J2 Conn_01x40_Pin, J3 19428-0011, J4 Molex_1040310811, Q1 MMBT2222LT1G, Q2 MMBT2222LT1G, U1 USBLC6-2SC6, U2 SN65HVD230

Commit message: Dash PCB work
Parts:
- added U10: EMIF06-MSD02N16, SDM_MiscFootprint:UQFN-17-3.5x1.2mm, F.Cu at (134.8, 120.9)
- moved IC7 91.1 mm to (207.6, 72.8)
- moved J2 76.8 mm to (164.1, 95.8)
- moved J4 64.8 mm to (135.5, 128.5), turned to 180 degrees
- moved J3 62.4 mm to (162.0, 71.5)
- moved J1 60.7 mm to (117.3, 131.5)
- moved D2 54.1 mm to (96.8, 80.2)
- moved D4 54.1 mm to (96.8, 83.6)
- moved LED18 54.1 mm to (87.8, 80.1)
- moved LED19 54.1 mm to (87.8, 83.3)
- moved LED20 54.1 mm to (87.8, 86.6)
- moved LED21 54.1 mm to (87.8, 89.9)
- moved LED22 54.1 mm to (87.8, 93.1)
- moved LED23 54.1 mm to (87.8, 96.4)
- moved LED24 54.1 mm to (87.8, 99.7)
- moved LED25 54.1 mm to (87.8, 102.9)
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Routing:
- net /CHIP_PU: track 0.00 -> 46.7 mm, vias 0 -> 2
- net /U0RXD: track 0.00 -> 38.3 mm
- net /U0TXD: track 0.00 -> 37.8 mm
- net /GPIO0: track 0.00 -> 25.3 mm
- net VBUS: track 0.00 -> 18.7 mm
- net Net-(J4-DAT2): track 0.00 -> 13.8 mm
- net Net-(J4-DAT3/CD): track 0.00 -> 13.5 mm
- net Net-(J4-DAT1): track 0.00 -> 13.5 mm
- net Net-(J4-CMD): track 0.00 -> 13.2 mm
- net Net-(J4-DAT0): track 0.00 -> 13.2 mm
- net Net-(J4-CLK): track 0.00 -> 12.5 mm
- net /PROG_D+: track 0.00 -> 10.7 mm
- net /PROG_D-: track 0.00 -> 10.1 mm
- net Net-(IC2-RTS): track 0.00 -> 9.47 mm, vias 0 -> 2
- net Net-(IC2-DTR): track 0.00 -> 8.95 mm
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Other:
- board outline added: 130 x 81.2 mm
- copper layers 2 -> 4

Commit message: Dash
Parts:
- LED10, LED11, LED12, LED13, LED14, LED15, LED16, LED2, LED3, LED4, LED5, LED6, LED7, LED8, LED9: moved to B.Cu
- moved LED16 89.1 mm to (162.0, 57.0)
- moved LED15 84.0 mm to (158.0, 57.0)
- moved LED14 78.9 mm to (154.0, 57.0)
- moved LED13 73.9 mm to (150.0, 57.0)
- moved LED9 71.0 mm to (134.0, 57.0)
- moved LED12 68.9 mm to (146.0, 57.0)
- moved LED8 65.8 mm to (130.0, 57.0)
- moved LED11 63.9 mm to (142.0, 57.0)
- moved LED7 60.7 mm to (126.0, 57.0)
- moved LED10 58.9 mm to (138.0, 57.0)
- moved LED6 55.5 mm to (122.0, 57.0)
- moved LED5 50.4 mm to (118.0, 57.0)
- moved LED4 45.2 mm to (114.0, 57.0)
- moved LED3 40.0 mm to (110.0, 57.0)
- moved LED2 34.9 mm to (106.0, 57.0)
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Other:
- board size 130 x 81.2 mm -> 130 x 81 mm

Commit message: dash
Parts:
- J2, LED17, LED18, LED19, LED20, LED21, LED22, LED23, LED24, LED25, LED26, LED27, LED28, LED29, LED30, LED31, LED32, LED33, S1, S2, S3, S4: moved to B.Cu
- moved S2 164.8 mm to (228.5, 128.1), turned to -90 degrees
- moved S1 163.2 mm to (228.5, 117.0), turned to -90 degrees
- moved IC8 160.5 mm to (-22.5, 134.3)
- moved IC3 141.6 mm to (200.5, 87.5), turned to 90 degrees
- moved BLACK_TP1 140.9 mm to (-20.8, 178.2)
- moved C25 140.9 mm to (-23.2, 198.8)
- moved TP2 140.9 mm to (-21.2, 169.6)
- moved U2 137.7 mm to (194.5, 87.5), turned to 90 degrees
- moved R30 133.9 mm to (-66.2, 153.3), turned to 90 degrees
- moved D1 133.4 mm to (194.5, 82.0), turned to -90 degrees
- moved R33 132.5 mm to (-69.2, 153.3), turned to 90 degrees
- moved R32 132.5 mm to (-67.7, 153.3), turned to 90 degrees
- moved R19 132.2 mm to (-64.7, 158.2)
- moved R20 132.2 mm to (-64.7, 160.8)
- moved R21 132.2 mm to (-64.7, 163.3)
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Connections:
- LED16 pad 2: /A16R -> /A15R
- LED17 pad 4: /A7B -> /A16B
Routing:
- net /BTN2: track 0.00 -> 79.2 mm, vias 0 -> 1
- net /BTN1: track 0.00 -> 75.1 mm, vias 0 -> 1
- net /BTN3: track 0.00 -> 60.4 mm, vias 0 -> 1
- net /BTN4: track 0.00 -> 59.4 mm, vias 0 -> 1
- net /CAN-: track 0.00 -> 56.9 mm
- net /SD_CMD: track 0.00 -> 46.6 mm, vias 0 -> 2
- net /SPI_CLK: track 0.00 -> 44.7 mm, vias 0 -> 2
- net /CAN+: track 0.00 -> 44.0 mm
- net /SPI_DATA0: track 0.00 -> 44.0 mm, vias 0 -> 2
- net /SPI_DATA1: track 0.00 -> 43.4 mm, vias 0 -> 2
- net /A9G: track 0.00 -> 42.1 mm, vias 0 -> 1
- net /A9R: track 0.00 -> 41.8 mm, vias 0 -> 1
- net /A9B: track 0.00 -> 40.3 mm, vias 0 -> 1
- net /SPI_DATA2: track 0.00 -> 39.1 mm, vias 0 -> 2
- net /SPI_DATA3: track 0.00 -> 38.4 mm, vias 0 -> 2
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- added copper zone on In2.Cu, net +5V
- added copper zone on F.Cu, net GND
- added copper zone on In1.Cu, net GND
- added copper zone on In2.Cu, net VBUS
Other:
- outline, holes or cut-outs redrawn

Commit message: Hella dash edits
just cranked that shit out
Parts:
- removed C5: 4.7uF, Capacitor_SMD:C_0603_1608Metric
- removed C6: 100nF, Capacitor_SMD:C_0603_1608Metric
- removed C7: 1uF, Capacitor_SMD:C_0603_1608Metric
- removed IC2: CP2102N-A02-GQFN28, SDM_MiscFootprint:QFN50P500X500X80-29N-D
- removed Q1, Q2: MMBT2222LT1G, SDM_MiscFootprint:SOT96P237X111-3N
- removed R17, R18, R19, R20, R21, R22, R23, R24, R25, R26, R27, R28, R29, R30, R32, R33, R35, R36, R37, R38, R39, R40, R41, R42, R43, R44, R45, R46, R47, R48, R49, R50, R52, R53: 33, Resistor_SMD:R_0603_1608Metric
- removed R6: 47.5K, Resistor_SMD:R_0603_1608Metric
- removed R7, R8: 10k, Resistor_SMD:R_0603_1608Metric
- removed R9: 1k, Resistor_SMD:R_0603_1608Metric
- removed TP2: SMPS, TestPoint:TestPoint_Pad_1.5x1.5mm
- J2: moved to F.Cu
- R5: value 22.1K -> 10k
- moved C16 279.6 mm to (213.8, 102.0), turned to 135 degrees
- moved C15 278.6 mm to (216.5, 114.0), turned to 45 degrees
- moved C17 277.9 mm to (212.7, 103.1), turned to 135 degrees
- moved IC8 232.6 mm to (208.5, 107.4), turned to 135 degrees
- moved IC9 212.5 mm to (219.0, 107.4), turned to -90 degrees
- moved R15 209.2 mm to (188.5, 86.2)
- moved C25 202.9 mm to (152.3, 96.9), turned to 90 degrees
- moved C19 202.6 mm to (174.0, 100.0), turned to 180 degrees
- moved C20 202.5 mm to (174.0, 98.2), turned to 180 degrees
- moved C21 196.0 mm to (167.5, 100.0), turned to 90 degrees
- moved C10 194.6 mm to (220.1, 111.8)
- moved BLACK_TP1 186.2 mm to (150.5, 105.2)
- moved R58 174.3 mm to (224.5, 130.0), turned to 90 degrees
- moved R51 172.8 mm to (222.6, 107.5), turned to -90 degrees
- moved R57 172.3 mm to (224.0, 119.0), turned to 90 degrees
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Connections:
- IC1 pad 13: /LED_LAT -> /PROG_D-
- IC1 pad 14: /LED_GSCLK -> /PROG_D+
- IC1 pad 23: /SD_CD -> unconnected-(IC1-IO21-Pad23)
- IC6 pad 1: /A4B -> /B4B
- IC6 pad 10: /A12R -> /B12R
- IC6 pad 11: /A12B -> /B12B
- IC6 pad 12: /A16G -> /B16G
- IC6 pad 13: /A16R -> /B16R
- IC6 pad 14: /A16B -> /B16B
- IC6 pad 15: /A11G -> /B11G
- IC6 pad 16: /A11R -> /B11R
- IC6 pad 17: /A11B -> /B11B
- IC6 pad 18: /A15G -> /B15G
- IC6 pad 19: /A15R -> /B15R
- IC6 pad 2: /A4R -> /B4R
- IC6 pad 20: /A15B -> /B15B
- IC6 pad 21: /A14G -> /B14G
- IC6 pad 22: /A14R -> /B14R
- IC6 pad 23: /A14B -> /B14B
- IC6 pad 24: /A10G -> /B10G
- IC6 pad 25: /A10R -> /B10R
- IC6 pad 26: /A10B -> /B10B
- IC6 pad 27: /A13G -> /B13G
- IC6 pad 28: /A13R -> /B13R
- IC6 pad 29: /A13B -> /B13B
- IC6 pad 3: /A4G -> /B4G
- IC6 pad 30: /A9G -> /B9G
- IC6 pad 31: /A9R -> /B9R
- IC6 pad 32: /A9B -> /B9B
- IC6 pad 33: unconnected-(IC6-VCC-Pad33) -> +3.3V
- IC6 pad 35: unconnected-(IC6-GND_2-Pad35) -> GND
- IC6 pad 39: /A5B -> /B5B
- IC6 pad 4: /A8B -> /B8B
- IC6 pad 40: /A5R -> /B5R
- IC6 pad 41: /A5G -> /B5G
- IC6 pad 42: /A1B -> /B1B
- IC6 pad 43: /A1R -> /B1R
- IC6 pad 44: /A1G -> /B1G
- IC6 pad 45: /A6B -> /B6B
- IC6 pad 46: /A6R -> /B6R
- IC6 pad 47: /A6G -> /B6G
- IC6 pad 48: /A2B -> /B2B
- IC6 pad 49: /A2R -> /B2R
- IC6 pad 5: /A8R -> /B8R
- IC6 pad 50: /A2G -> /B2G
- IC6 pad 51: /A3B -> /B3B
- IC6 pad 52: /A3R -> /B3R
- IC6 pad 53: /A3G -> /B3G
- IC6 pad 54: /A7B -> /B7B
- IC6 pad 55: /A7R -> /B7R
- IC6 pad 56: /A7G -> /B7G
- IC6 pad 57: unconnected-(IC6-THERMAL_PAD-Pad57) -> GND
- IC6 pad 6: /A8G -> /B8G
- IC6 pad 9: /A12G -> /B12G
- IC7 pad 27: /B13G -> /A13G
- IC7 pad 28: /B13R -> /A13R
- IC7 pad 33: unconnected-(IC7-VCC-Pad33) -> +3.3V
- IC7 pad 57: unconnected-(IC7-THERMAL_PAD-Pad57) -> GND
- IC8 pad 1: Net-(IC8-R0) -> /R0
- IC8 pad 3: Net-(IC8-SCK) -> /SPI_CLK
- IC8 pad 4: Net-(IC8-MISO) -> /SPI_DATA0
- IC8 pad 40: Net-(IC8-B7) -> /B7
- IC8 pad 41: Net-(IC8-B6) -> /B6
- IC8 pad 42: Net-(IC8-B5) -> /B5
- IC8 pad 43: Net-(IC8-B4) -> /B4
- IC8 pad 44: Net-(IC8-B3) -> /B3
- IC8 pad 45: Net-(IC8-B2) -> /B2
- IC8 pad 46: Net-(IC8-B1) -> /B1
- IC8 pad 47: Net-(IC8-B0) -> /B0
- IC8 pad 49: Net-(IC8-G7) -> /G7
- IC8 pad 5: Net-(IC8-MOSI) -> /SPI_DATA1
- IC8 pad 50: Net-(IC8-G6) -> /G6
- IC8 pad 51: Net-(IC8-G5) -> /G5
- IC8 pad 52: Net-(IC8-G4) -> /G4
- IC8 pad 53: Net-(IC8-G3) -> /G3
- IC8 pad 54: Net-(IC8-G2) -> /G2
- IC8 pad 55: Net-(IC8-G1) -> /G1
- IC8 pad 56: Net-(IC8-G0) -> /G0
- IC8 pad 58: Net-(IC8-R7) -> /R7
- IC8 pad 59: Net-(IC8-R6) -> /R6
- IC8 pad 60: Net-(IC8-R5) -> /R5
- IC8 pad 61: Net-(IC8-R4) -> /R4
- IC8 pad 62: Net-(IC8-R3) -> /R3
- IC8 pad 63: Net-(IC8-R2) -> /R2
- IC8 pad 64: Net-(IC8-R1) -> /R1
- IC8 pad 7: Net-(IC8-GPIO0/IO2) -> /SPI_DATA2
- IC8 pad 8: Net-(IC8-GPIO1/IO3) -> /SPI_DATA3
- IC9 pad 2: Net-(IC9-SO/IO_1) -> Net-(IC8-SPIM_MISO)
- IC9 pad 3: Net-(IC9-W_P#_/_IO_2) -> Net-(IC8-SPIM_IO2)
- IC9 pad 5: Net-(IC9-SI_/_IO_0) -> Net-(IC8-SPIM_MOSI)
- IC9 pad 6: Net-(IC9-SCK) -> Net-(IC8-SPIM_SCLK)
- IC9 pad 7: Net-(IC9-IO_3_/_RESET#) -> Net-(IC8-SPIM_IO3)
- LED10 pad 1: unconnected-(LED10-A-Pad1) -> +3.3V
- LED11 pad 1: unconnected-(LED11-A-Pad1) -> +3.3V
- LED12 pad 1: unconnected-(LED12-A-Pad1) -> +3.3V
- LED13 pad 1: unconnected-(LED13-A-Pad1) -> +3.3V
- LED14 pad 1: unconnected-(LED14-A-Pad1) -> +3.3V
- LED15 pad 1: unconnected-(LED15-A-Pad1) -> +3.3V
- LED16 pad 1: unconnected-(LED16-A-Pad1) -> +3.3V
- LED17 pad 1: unconnected-(LED17-A-Pad1) -> +3.3V
- LED18 pad 1: unconnected-(LED18-A-Pad1) -> +3.3V
- LED19 pad 1: unconnected-(LED19-A-Pad1) -> +3.3V
- LED2 pad 1: unconnected-(LED2-A-Pad1) -> +3.3V
- LED20 pad 1: unconnected-(LED20-A-Pad1) -> +3.3V
- LED21 pad 1: unconnected-(LED21-A-Pad1) -> +3.3V
- LED22 pad 1: unconnected-(LED22-A-Pad1) -> +3.3V
- LED23 pad 1: unconnected-(LED23-A-Pad1) -> +3.3V
- LED24 pad 1: unconnected-(LED24-A-Pad1) -> +3.3V
- LED25 pad 1: unconnected-(LED25-A-Pad1) -> +3.3V
- LED26 pad 1: unconnected-(LED26-A-Pad1) -> +3.3V
- LED27 pad 1: unconnected-(LED27-A-Pad1) -> +3.3V
- LED28 pad 1: unconnected-(LED28-A-Pad1) -> +3.3V
- LED29 pad 1: unconnected-(LED29-A-Pad1) -> +3.3V
- LED3 pad 1: unconnected-(LED3-A-Pad1) -> +3.3V
- LED30 pad 1: unconnected-(LED30-A-Pad1) -> +3.3V
- LED31 pad 1: unconnected-(LED31-A-Pad1) -> +3.3V
- LED32 pad 1: unconnected-(LED32-A-Pad1) -> +3.3V
- LED32 pad 2: /B16R -> /B15R
- LED33 pad 1: unconnected-(LED33-A-Pad1) -> +3.3V
- LED4 pad 1: unconnected-(LED4-A-Pad1) -> +3.3V
- LED5 pad 1: unconnected-(LED5-A-Pad1) -> +3.3V
- LED6 pad 1: unconnected-(LED6-A-Pad1) -> +3.3V
- LED7 pad 1: unconnected-(LED7-A-Pad1) -> +3.3V
- LED8 pad 1: unconnected-(LED8-A-Pad1) -> +3.3V
- LED9 pad 1: unconnected-(LED9-A-Pad1) -> +3.3V
- R5 pad 1: Net-(IC2-VBUS) -> /GPIO0
- R5 pad 2: VBUS -> +3.3V
Routing:
- net /LED_SCLK: track 0.00 -> 169.1 mm, vias 0 -> 3
- net /SPI_DATA0: track 44.0 -> 141.0 mm, vias 2 -> 4
- net /Daisy Chain: track 0.00 -> 88.2 mm, vias 0 -> 2
- net /LED_GSCLK: track 0.00 -> 86.1 mm, vias 0 -> 2
- net /LED_DATA: track 0.00 -> 85.6 mm, vias 0 -> 2
- net /LED_LAT: track 0.00 -> 82.9 mm, vias 0 -> 2
- net /DISP_CS: track 0.00 -> 60.1 mm, vias 0 -> 2
- net /SPI_DATA3: track 38.4 -> 98.2 mm, vias 2 -> 4
- net Net-(R4-Pad2): track 1.68 -> 58.9 mm
- net GND: track 15.3 -> 72.4 mm, vias 17 -> 33
- net +BATT: track 0.00 -> 54.9 mm, vias 0 -> 2
- net /SPI_DATA2: track 39.1 -> 93.3 mm, vias 2 -> 4
- net Net-(R3-Pad1): track 2.06 -> 56.0 mm
- net /SPI_DATA1: track 43.4 -> 94.9 mm, vias 2 -> 4
- net /INT_N: track 0.00 -> 49.1 mm
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- added copper zone on In2.Cu, net +3.3V
- added copper zone on In2.Cu, net VCC
Other:
- outline, holes or cut-outs redrawn

Commit message: Dash check, Fernando
Parts:
- removed R13: 10k, Resistor_SMD:R_0603_1608Metric
- removed TP1: ST_5V, TestPoint:TestPoint_Pad_1.5x1.5mm
- added TP2: SMPS, TestPoint:TestPoint_Pad_1.5x1.5mm, F.Cu at (134.8, 106.1)
- moved C21 2.11 mm to (165.5, 100.7)
- moved L1 1.90 mm to (160.4, 96.4)
- moved PS1 1.90 mm to (166.6, 96.8)
- moved R31 1.90 mm to (169.6, 96.8)
- moved C22 1.85 mm to (167.3, 100.7)
- moved C19 1.76 mm to (172.7, 101.2)
- moved D2 1.64 mm to (167.4, 93.2)
- moved R34 1.60 mm to (169.1, 100.7)
- moved D4 1.59 mm to (172.2, 94.6)
- moved C20 1.52 mm to (172.7, 99.1)
- moved L2 1.28 mm to (134.0, 97.4)
- moved C8 1.16 mm to (119.1, 110.9)
- moved R56 0.98 mm to (144.5, 100.4)
- moved R11 0.56 mm to (116.4, 109.0)
- moved R3 0.19 mm to (164.9, 106.7)
Connections:
- IC4 pad 8: /ST -> unconnected-(IC4-ST-Pad8)
Routing:
- net /SPI_DATA0: track 141.0 -> 94.4 mm
- net GND: track 72.4 -> 111.0 mm, vias 33 -> 87
- net VBUS: track 19.3 -> 44.7 mm, vias 4 -> 5
- net +3.3V: track 36.0 -> 47.5 mm, vias 48 -> 53
- net VCC: track 34.9 -> 43.4 mm
- net /ST: track 5.31 -> 0.00 mm
- net VLED+: track 21.1 -> 24.2 mm
- net VLED-: track 18.2 -> 20.7 mm
- net /LED_LAT: track 82.9 -> 85.3 mm
- net +5V: track 17.9 -> 15.6 mm
- net /PWM0: track 39.2 -> 41.2 mm
- net /SPI_DATA3: track 98.2 -> 100.2 mm
- net /SMPS_SW: track 11.7 -> 13.0 mm
- net /LED_GSCLK: track 86.1 -> 87.1 mm
- net /SMPS_FB: track 5.73 -> 6.72 mm
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