File: 2026/Dash/Dash.kicad_pcb (KiCad board)
At the start: 4 copper layers, 130 x 81 mm, 106 parts, among them IC1 ESP32-S3-WROOM-1-N8R8, IC10 TPS563211DRLR, IC3 TLP175A_TPL,E, IC4 TPS2116DRLR, IC5 MIC37100-3.3WS, IC6 TLC5955RTQT, IC7 TLC5955RTQT, IC8 BT818Q-T, IC9 S25FL256LAGNFB010, J1 USB4730-GF-A, J2 Conn_01x40_Pin, J3 19428-0011, J4 Molex_1040310811, U1 USBLC6-2SC6, U10 EMIF06-MSD02N16, U2 SN65HVD230

Commit message: Library maintenance
edited some 3dmodles to point to their footprints. edited symbols and footprints to link properly. edited footprint and symbol library names in all projects 2026-2027 to use the same library nick name "SDM" for both  symbol and footprint.
all users must delete their old lib and make a new one named SDM for symbol and footprint.
Parts:
- BLACK_TP1: footprint SDM_MiscFootprint:5006 -> SDM:5006
- IC3: footprint SDM_MiscFootprint:TLP266J -> SDM:TLP266J
- IC4: footprint SDM_MiscFootprint:SOTFL50P160X60-8L -> SDM:SOTFL50P160X60-8L
- J1: footprint SDM_MiscFootprint:USB4730GFA -> SDM:USB4730GFA
- J3: footprint SDM_MiscFootprint:194280011 -> SDM:194280011
- LED1: footprint SDM_MiscFootprint:LEDC1608X80N -> SDM:LEDC1608X80N
- LED11, LED12, LED13, LED14, LED15, LED16, LED17, LED18, LED19, LED20, LED21, LED22, LED23, LED24, LED25, LED26, LED27, LED28, LED29, LED30, LED31, LED32, LED33, LED9: footprint SDM_MiscFootprint:PLCC4_CLMUD-FKC_CRW -> SDM:PLCC4_CLMUD-FKC_CRW
- PS1: footprint SDM_MiscFootprint:SOT65P210X110-5N -> SDM:SOT65P210X110-5N
- S1, S2, S3, S4: footprint SDM_MiscFootprint:KSS321GLFS -> SDM:KSS321GLFS
- U10: footprint SDM_MiscFootprint:UQFN-17-3.5x1.2mm -> SDM:UQFN-17-3.5x1.2mm
Changed lines of the file:
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@@
 		)
 	)
-	(footprint "SDM_MiscFootprint:LEDC1608X80N"
+	(footprint "SDM:LEDC1608X80N"
 		(layer "F.Cu")
 		(at 116 105.5 90)
@@
 		)
 	)
-	(footprint "SDM_MiscFootprint:UQFN-17-3.5x1.2mm"
+	(footprint "SDM:UQFN-17-3.5x1.2mm"
 		(layer "F.Cu")
 		(at 130.845 120.855 -90)
@@
 		)
 	)
-	(footprint "SDM_MiscFootprint:USB4730GFA"
+	(footprint "SDM:USB4730GFA"
 		(layer "F.Cu")
 		(at 114.135 131.455)
@@
 		)
 		(embedded_fonts no)
-		(model "BT818Q-T.stp"
+		(model "${SDM_MISC_3D}/BT818Q-T.stp"
 			(offset
 				(xyz 0 0 0)
@@
 		)
 	)
-	(footprint "SDM_MiscFootprint:SOT65P210X110-5N"
+	(footprint "SDM:SOT65P210X110-5N"
 		(layer "F.Cu")
 		(at 166.605 96.84)
@@
 		)
 	)
-	(footprint "SDM_MiscFootprint:TLP266J"
+	(footprint "SDM:TLP266J"
 		(layer "F.Cu")
 		(at 200.265001 87.5 90)
@@
 		)
 	)
-	(footprint "SDM_MiscFootprint:5006"
+	(footprint "SDM:5006"
 		(layer "F.Cu")
 		(at 150.5 105.25)
@@
 		)
 		(embedded_fonts no)
-		(model "${VICI_LIBRARIES}/ViciModels/BWVS006060454R7ML1.step"
+		(model "${SDM_MISC_3D}/BWVS006060454R7ML1.step"
 			(offset
 				(xyz 0 0 0)
@@
 		)
 	)
-	(footprint "SDM_MiscFootprint:194280011"
+	(footprint "SDM:194280011"
 		(layer "F.Cu")
 		(at 162 71.5)
@@
 		)
 		(embedded_fonts no)
-		(model "S25FL256LAGNFB010.stp"
+		(model "${SDM_MISC_3D}/S25FL256LAGNFB010.stp"
 			(offset
 				(xyz 0 0 0)
@@
 		)
 	)
-	(footprint "SDM_MiscFootprint:SOTFL50P160X60-8L"
+	(footprint "SDM:SOTFL50P160X60-8L"
 		(layer "F.Cu")
 		(at 120 106)
@@
 		)
 	)
-	(footprint "SDM_MiscFootprint:PLCC4_CLMUD-FKC_CRW"
+	(footprint "SDM:PLCC4_CLMUD-FKC_CRW"
 		(layer "B.Cu")
 		(at 102.25 72.75 -90)
@@
 		)
 	)
-	(footprint "SDM_MiscFootprint:PLCC4_CLMUD-FKC_CRW"
+	(footprint "SDM:PLCC4_CLMUD-FKC_CRW"
 		(layer "B.Cu")
 		(at 102.25 65.25 -90)
@@
 		)
 	)
-	(footprint "SDM_MiscFootprint:PLCC4_CLMUD-FKC_CRW"
+	(footprint "SDM:PLCC4_CLMUD-FKC_CRW"
 		(layer "B.Cu")
 		(at 191.2747 56.25 180)
@@
 		)
 	)
-	(footprint "SDM_MiscFootprint:KSS321GLFS"
+	(footprint "SDM:KSS321GLFS"
 		(layer "B.Cu")
 		(at 228.5 117 -90)
@@
 		)
 	)
-	(footprint "SDM_MiscFootprint:PLCC4_CLMUD-FKC_CRW"
+	(footprint "SDM:PLCC4_CLMUD-FKC_CRW"
 		(layer "B.Cu")
 		(at 146.25 56.25 180)
@@
 		)
 	)
-	(footprint "SDM_MiscFootprint:PLCC4_CLMUD-FKC_CRW"
+	(footprint "SDM:PLCC4_CLMUD-FKC_CRW"
 		(layer "B.Cu")
 		(at 102.25 102.7253 -90)
@@
 		)
 	)
-	(footprint "SDM_MiscFootprint:PLCC4_CLMUD-FKC_CRW"
+	(footprint "SDM:PLCC4_CLMUD-FKC_CRW"
 		(layer "B.Cu")
 		(at 131.25 56.25 180)
@@
 		)
 	)
-	(footprint "SDM_MiscFootprint:PLCC4_CLMUD-FKC_CRW"
+	(footprint "SDM:PLCC4_CLMUD-FKC_CRW"
 		(layer "B.Cu")
 		(at 213.75 56.25 180)
@@
 		)
 	)
-	(footprint "SDM_MiscFootprint:PLCC4_CLMUD-FKC_CRW"
+	(footprint "SDM:PLCC4_CLMUD-FKC_CRW"
 		(layer "B.Cu")
 		(at 161.25 56.25 180)
@@
 		)
 	)
-	(footprint "SDM_MiscFootprint:KSS321GLFS"
+	(footprint "SDM:KSS321GLFS"
 		(layer "B.Cu")
 		(at 101.5 117.25 90)
@@
 		)
 	)
-	(footprint "SDM_MiscFootprint:PLCC4_CLMUD-FKC_CRW"
+	(footprint "SDM:PLCC4_CLMUD-FKC_CRW"
 		(layer "B.Cu")
 		(at 102.25 110.25 -90)
@@
 		)
 	)
-	(footprint "SDM_MiscFootprint:PLCC4_CLMUD-FKC_CRW"
+	(footprint "SDM:PLCC4_CLMUD-FKC_CRW"
 		(layer "B.Cu")
 		(at 206.25 56.25 180)
@@
 		)
 	)
-	(footprint "SDM_MiscFootprint:PLCC4_CLMUD-FKC_CRW"
+	(footprint "SDM:PLCC4_CLMUD-FKC_CRW"
 		(layer "B.Cu")
 		(at 183.75 56.25 180)
@@
 		)
 	)
-	(footprint "SDM_MiscFootprint:PLCC4_CLMUD-FKC_CRW"
+	(footprint "SDM:PLCC4_CLMUD-FKC_CRW"
 		(layer "B.Cu")
 		(at 138.75 56.25 180)
@@
 		)
 	)
-	(footprint "SDM_MiscFootprint:PLCC4_CLMUD-FKC_CRW"
+	(footprint "SDM:PLCC4_CLMUD-FKC_CRW"
 		(layer "B.Cu")
 		(at 108.75 56.25 180)
@@
 		)
 	)
-	(footprint "SDM_MiscFootprint:PLCC4_CLMUD-FKC_CRW"
+	(footprint "SDM:PLCC4_CLMUD-FKC_CRW"
 		(layer "B.Cu")
 		(at 102.25 57.75 -90)
@@
 		)
 	)
-	(footprint "SDM_MiscFootprint:PLCC4_CLMUD-FKC_CRW"
+	(footprint "SDM:PLCC4_CLMUD-FKC_CRW"
 		(layer "B.Cu")
 		(at 102.25 80.2747 -90)
@@
 		)
 	)
-	(footprint "SDM_MiscFootprint:PLCC4_CLMUD-FKC_CRW"
+	(footprint "SDM:PLCC4_CLMUD-FKC_CRW"
 		(layer "B.Cu")
 		(at 176.25 56.25 180)
@@
 		)
 	)
-	(footprint "SDM_MiscFootprint:PLCC4_CLMUD-FKC_CRW"
+	(footprint "SDM:PLCC4_CLMUD-FKC_CRW"
 		(layer "B.Cu")
 		(at 102.25 95.25 -90)
@@
 		)
 	)
-	(footprint "SDM_MiscFootprint:PLCC4_CLMUD-FKC_CRW"
+	(footprint "SDM:PLCC4_CLMUD-FKC_CRW"
 		(layer "B.Cu")
 		(at 116.25 56.25 180)
@@
 		)
 	)
-	(footprint "SDM_MiscFootprint:PLCC4_CLMUD-FKC_CRW"
+	(footprint "SDM:PLCC4_CLMUD-FKC_CRW"
 		(layer "B.Cu")
 		(at 153.75 56.25 180)
@@
 		)
 	)
-	(footprint "SDM_MiscFootprint:PLCC4_CLMUD-FKC_CRW"
+	(footprint "SDM:PLCC4_CLMUD-FKC_CRW"
 		(layer "B.Cu")
 		(at 123.75 56.25 180)
@@
 		)
 	)
-	(footprint "SDM_MiscFootprint:PLCC4_CLMUD-FKC_CRW"
+	(footprint "SDM:PLCC4_CLMUD-FKC_CRW"
 		(layer "B.Cu")
 		(at 168.75 56.25 180)
@@
 		)
 	)
-	(footprint "SDM_MiscFootprint:PLCC4_CLMUD-FKC_CRW"
+	(footprint "SDM:PLCC4_CLMUD-FKC_CRW"
 		(layer "B.Cu")
 		(at 102.25 87.75 -90)
@@
 		)
 	)
-	(footprint "SDM_MiscFootprint:PLCC4_CLMUD-FKC_CRW"
+	(footprint "SDM:PLCC4_CLMUD-FKC_CRW"
 		(layer "B.Cu")
 		(at 198.75 56.25 180)
@@
 		)
 	)
-	(footprint "SDM_MiscFootprint:KSS321GLFS"
+	(footprint "SDM:KSS321GLFS"
 		(layer "B.Cu")
 		(at 228.5 128.125 -90)
@@
 		)
 	)
-	(footprint "SDM_MiscFootprint:KSS321GLFS"
+	(footprint "SDM:KSS321GLFS"
 		(layer "B.Cu")
 		(at 101.5 128.125 90)
@@
 		)
 	)
-	(footprint "SDM_MiscFootprint:PLCC4_CLMUD-FKC_CRW"
+	(footprint "SDM:PLCC4_CLMUD-FKC_CRW"
 		(layer "B.Cu")
 		(at 221.25 56.25 180)
