File: 2027/SDM27_WheelBoard/SDM27_WheelBoard_v1.0/SDM27_WheelBoard_v1.0.kicad_pcb (KiCad board)
At the start: 4 copper layers, 29.1 x 12.6 mm, 61 parts, among them IC1 NCP187AMT330TAG, IC8 TCAN3403DRBRQ1, IC9 MAX9924UAUB+, J1 5V, J10 WS+, J11 WS-, J12 CAN+, J13 CAN-, J2 GND, J3 CAN+, J4 CAN-, J5 5V, J6 GND, J7 SDA, J8 SCL, J9 GND, U1 ESP32-C5, Y1 Crystal_GND24

Commit message: wheel boards
Parts:
- removed C13: 1uF, Capacitor_SMD:C_0402_1005Metric
- removed C14: 10uF, Capacitor_SMD:C_0402_1005Metric
- removed IC9: MAX9924UAUB+, SDM:SOP50P490X110-10L
- removed J10: WS+, SDM:DoublePin1.00mm
- removed J11: WS-, SDM:DoublePin1.00mm
- removed J12, J3: CAN+, SDM:DoublePin1.00mm
- removed J13, J4: CAN-, SDM:DoublePin1.00mm
- removed J5: 5V, SDM:DoublePin1.00mm
- removed J6, J9: GND, SDM:DoublePin1.00mm
- removed J7: SDA, SDM:DoublePin1.00mm
- removed J8: SCL, SDM:DoublePin1.00mm
- removed LED3: 150060RS75000, SDM:LEDC1608X80N
- removed R16, R18: 1k, Resistor_SMD:R_0402_1005Metric
- removed R17, R19: 10k, Resistor_SMD:R_0402_1005Metric
- added C22: 0.1uF, Capacitor_SMD:C_0402_1005Metric, F.Cu at (124.6, 88.0)
- added C32: 1uF, Capacitor_SMD:C_0402_1005Metric, F.Cu at (130.3, 72.2)
- added C40: 100nF, Capacitor_SMD:C_0402_1005Metric, F.Cu at (130.3, 88.0)
- added C41: 100nF, Capacitor_SMD:C_0402_1005Metric, F.Cu at (133.2, 72.2)
- added C42: 22uF, Capacitor_SMD:C_0402_1005Metric, F.Cu at (133.2, 74.2)
- added C43: 10nF, Capacitor_SMD:C_0402_1005Metric, F.Cu at (133.2, 76.2)
- added C44: 10nF, Capacitor_SMD:C_0402_1005Metric, F.Cu at (133.2, 78.1)
- added C45: 22nF, Capacitor_SMD:C_0402_1005Metric, F.Cu at (133.2, 80.1)
- added C46: 10nF, Capacitor_SMD:C_0402_1005Metric, F.Cu at (133.2, 82.1)
- added C47: 1uF, Capacitor_SMD:C_0402_1005Metric, F.Cu at (133.2, 84.0)
- added IC2: TPS542951RSAR, SDM_Misc:QFN65P400X400X100-17N-D, F.Cu at (111.0, 93.4)
- added IC3: TPS2121RUXR, SDM:TPS2121RUXR, F.Cu at (118.0, 93.6)
- added IC4: MLX90614ESF-BAA-000-SP, SDM_Misc:MLX90614ESFBAA000SP, F.Cu at (136.0, 100.0)
- added IC5: SN74LVC1G17YZPR, SDM_Misc:BGA5C50P2X3_89X139X50, F.Cu at (125.3, 94.7)
- added L6: 2.2uH, Inductor_SMD:L_0402_1005Metric, F.Cu at (98.2, 82.2)
- added L7: 4.7uH, Inductor_SMD:L_0402_1005Metric, F.Cu at (98.2, 84.2)
- added R24: 18.2k, Resistor_SMD:R_0402_1005Metric, F.Cu at (101.1, 78.2)
- added R25: 5k, Resistor_SMD:R_0402_1005Metric, F.Cu at (101.1, 80.2)
- added R26: 63.4k, Resistor_SMD:R_0402_1005Metric, F.Cu at (101.1, 82.2)
- added R27: 5k, Resistor_SMD:R_0402_1005Metric, F.Cu at (101.1, 84.2)
- added R28: 10.2k, Resistor_SMD:R_0402_1005Metric, F.Cu at (101.1, 86.2)
- added R29: 5k, Resistor_SMD:R_0402_1005Metric, F.Cu at (104.0, 72.2)
- added R30: 23.7k, Resistor_SMD:R_0402_1005Metric, F.Cu at (104.0, 74.2)
- added R31: 5k, Resistor_SMD:R_0402_1005Metric, F.Cu at (104.0, 76.2)
- added R32: 100k, Resistor_SMD:R_0402_1005Metric, F.Cu at (104.0, 78.2)
- added R33: 73.2k, Resistor_SMD:R_0402_1005Metric, F.Cu at (104.0, 80.2)
- added R34: 22.1k, Resistor_SMD:R_0402_1005Metric, F.Cu at (104.0, 82.2)
- added R35: 100k, Resistor_SMD:R_0402_1005Metric, F.Cu at (104.0, 84.2)
- added R36: 18.0k, Resistor_SMD:R_0402_1005Metric, F.Cu at (104.0, 86.2)
- added R38: 23.7k, Resistor_SMD:R_0402_1005Metric, F.Cu at (106.9, 72.2)
- added R39: 5k, Resistor_SMD:R_0402_1005Metric, F.Cu at (106.9, 74.2)
- added R40: 5k, Resistor_SMD:R_0402_1005Metric, F.Cu at (106.9, 76.2)
- added R41: 23.7k, Resistor_SMD:R_0402_1005Metric, F.Cu at (106.9, 78.2)
- added R42: 10.2k, Resistor_SMD:R_0402_1005Metric, F.Cu at (106.9, 80.2)
- added R43: 5k, Resistor_SMD:R_0402_1005Metric, F.Cu at (106.9, 82.2)
- added R44: 5k, Resistor_SMD:R_0402_1005Metric, F.Cu at (106.9, 84.2)
- added R45: 100k, Resistor_SMD:R_0402_1005Metric, F.Cu at (106.9, 86.2)
- added R46: 100k, Resistor_SMD:R_0402_1005Metric, F.Cu at (109.8, 72.2)
- added R47: 10k, Resistor_SMD:R_0402_1005Metric, F.Cu at (109.8, 74.2)
- added R48: 4.7k, Resistor_SMD:R_0402_1005Metric, F.Cu at (109.8, 76.2)
- added R49: 27, Resistor_SMD:R_0402_1005Metric, F.Cu at (109.8, 78.2)
- added R50: 27, Resistor_SMD:R_0402_1005Metric, F.Cu at (109.8, 80.2)
- added U2: USBLC6-2SC6, Package_TO_SOT_SMD:SOT-23-6, F.Cu at (142.9, 74.5)
- C39: value 1nF -> 100nF
- IC1: value NCP187AMT330TAG -> TPS2121RUXR; footprint SDM:SON65P200X200X80-7N -> SDM_Misc:TPS2121RUXR
- J1: value 5V -> WEIPU SA12 7PIN; footprint SDM:DoublePin1.00mm -> SDM_Misc:SA12 7Pin; moved to B.Cu
- J2: value GND -> WEIPU SA6 5Pin; footprint SDM:DoublePin1.00mm -> Connector_JST:JST_PH_B5B-PH-SM4-TB_1x05-1MP_P2.00mm_Vertical
- moved J2 48.3 mm to (125.1, 65.8), turned to 0 degrees
- moved FL2 40.4 mm to (136.2, 67.1), turned to 0 degrees
- moved C36 39.9 mm to (130.3, 80.1)
- moved C10 39.9 mm to (124.6, 72.2), turned to 0 degrees
- moved C23 37.4 mm to (127.5, 72.2), turned to 0 degrees
- moved C24 35.3 mm to (127.5, 74.2), turned to 0 degrees
- moved C18 33.6 mm to (124.6, 80.1)
- moved C16 33.3 mm to (124.6, 76.2), turned to 0 degrees
- moved C34 33.1 mm to (130.3, 76.2), turned to 0 degrees
- moved C33 32.8 mm to (130.3, 74.2), turned to 0 degrees
- moved C25 32.5 mm to (127.5, 76.2), turned to 0 degrees
- moved C17 32.4 mm to (124.6, 78.1), turned to 0 degrees
- moved R21 31.3 mm to (101.1, 72.2), turned to 0 degrees
- moved C15 31.2 mm to (124.6, 74.2), turned to 0 degrees
- moved C26 30.3 mm to (127.5, 78.1), turned to 0 degrees
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Connections:
- IC1 pad 1: +5V -> VCC
- IC1 pad 2: Net-(IC1-EN) -> VBUS
- IC1 pad 3: GND -> Net-(IC1-CP2)
- IC1 pad 4: unconnected-(IC1-PG-Pad4) -> Net-(IC1-OV2)
- IC1 pad 5: +3.3V -> Net-(IC1-OV1)
- IC1 pad 6: +3.3V -> Net-(IC1-PR1)
- IC1 pad 7: GND -> +12V
- J1 pad 1: +5V -> /CAN+
- J2 pad 1: GND -> /SDA
- U1 pad 22: unconnected-(U1-GPIO13/USB_D-/SDIO_DATA3-Pad22) -> Net-(U1-GPIO13/USB_D-/SDIO_DATA3)
- U1 pad 23: unconnected-(U1-GPIO14/USB_D+/SDIO_DATA2-Pad23) -> Net-(U1-GPIO14/USB_D+/SDIO_DATA2)
- U1 pad 34: unconnected-(U1-GPIO24-Pad34) -> /WSP_PWM
Routing:
- net +3.3V: track 48.7 -> 0.00 mm, vias 7 -> 0
- net GND: track 49.4 -> 2.30 mm, vias 31 -> 0
- net VCC: track 0.00 -> 19.2 mm
- net /SCL: track 13.0 -> 0.00 mm, vias 2 -> 0
- net /HE_OUTPUT: track 10.1 -> 0.00 mm, vias 3 -> 0
- net /SDA: track 9.63 -> 0.00 mm
- net /CAN_CTX: track 8.02 -> 0.00 mm, vias 2 -> 0
- net +12V: track 0.00 -> 7.46 mm
- net Net-(IC2-SW1): track 6.75 -> 0.00 mm
- net /CAN_RTX: track 6.72 -> 0.00 mm, vias 2 -> 0
- net /GPIO0: track 6.65 -> 0.00 mm, vias 2 -> 0
- net Net-(U1-XTAL_P): track 6.61 -> 0.00 mm
- net Net-(U1-XTAL_N): track 4.97 -> 0.00 mm
- net Net-(U1-VDDA1): track 4.94 -> 0.00 mm
- net /CHIP_EN: track 4.81 -> 0.00 mm, vias 2 -> 0
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- removed copper zone on In2.Cu, net +3.3V
- removed copper zone on In1.Cu, net GND
Other:
- board size 29.1 x 12.6 mm -> 38 x 22 mm

Commit message: wheel board updates
Parts:
- J2: footprint Connector_JST:JST_PH_B5B-PH-SM4-TB_1x05-1MP_P2.00mm_Vertical -> Connector_JST:JST_SH_BM09B-SRSS-TB_1x09-1MP_P1.00mm_Vertical; moved to B.Cu
- moved C41 53.4 mm to (101.1, 114.9)
- moved C42 53.4 mm to (101.1, 116.9)
- moved C43 53.4 mm to (101.1, 118.8)
- moved C32 41.3 mm to (100.7, 101.0), turned to -90 degrees
- moved C39 40.4 mm to (103.3, 116.1)
- moved L6 37.9 mm to (98.3, 120.1)
- moved R34 36.5 mm to (97.6, 118.1)
- moved R33 36.5 mm to (97.6, 116.1)
- moved C10 32.9 mm to (117.4, 104.3), turned to -90 degrees
- moved R29 29.9 mm to (106.0, 102.1), turned to 180 degrees
- moved R30 28.9 mm to (103.8, 103.1), turned to 180 degrees
- moved C36 27.0 mm to (118.3, 104.3), turned to -90 degrees
- moved R31 27.0 mm to (106.0, 103.1), turned to 180 degrees
- moved J2 26.7 mm to (131.5, 91.7), turned to 180 degrees
- moved R32 21.0 mm to (100.7, 99.0), turned to -90 degrees
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Connections:
- D2 pad 1: /CAN+ -> /CAN-
- D2 pad 2: /CAN- -> /CAN+
- J1 pad 1: /CAN+ -> /CAN-
- J1 pad 2: /CAN- -> /CAN+
- J1 pad 3: /CAN+ -> /CAN-
- J1 pad 4: /CAN- -> /CAN+
- U1 pad 11: /CAN_RTX -> /CAN_CTX
- U1 pad 12: /CAN_CTX -> /CAN_RTX
Routing:
- net GND: track 2.30 -> 18.8 mm, vias 0 -> 3
- net /CAN_RTX: track 0.00 -> 6.23 mm
- net Net-(IC1-OV2): track 0.00 -> 4.86 mm
- net Net-(IC1-OV1): track 0.00 -> 4.02 mm, vias 0 -> 2
- net /CAN_CTX: track 0.00 -> 3.97 mm
- net Net-(IC1-CP2): track 0.00 -> 2.86 mm, vias 0 -> 2
- net Net-(IC1-PR1): track 0.00 -> 2.81 mm
- net +3.3V: track 0.00 -> 2.65 mm
- net VBUS: track 0.00 -> 2.45 mm
- net /CAN+: track 11.2 -> 13.5 mm
- net Net-(IC1-ILIM): track 0.00 -> 1.25 mm
- net Net-(IC1-SS): track 0.00 -> 1.25 mm
- net /CAN-: track 11.0 -> 11.6 mm

Commit message: part values update
Parts:
- moved R34 31.8 mm to (112.7, 90.2)
- moved R33 31.0 mm to (114.6, 90.2)
- moved C43 30.8 mm to (114.6, 91.2), turned to 180 degrees
- moved L6 30.4 mm to (114.6, 94.4)
- moved C41 29.3 mm to (117.6, 90.7)
- moved C42 29.1 mm to (116.8, 92.4)
- moved C39 23.6 mm to (114.6, 95.4)
- moved IC3 9.92 mm to (118.6, 83.6)
- turned IC2 to 90 degrees
Routing:
- net VCC: track 19.2 -> 8.87 mm
- net Net-(IC2-SW1): track 0.00 -> 2.53 mm
- net Net-(IC2-VBST1): track 0.00 -> 2.15 mm
- net +5V: track 1.35 -> 0.00 mm
- net GND: vias 3 -> 5
- added copper zone on In1.Cu, net GND

Commit message: board progrez 40%
its 4:30 am...
Parts:
- removed C18: 1uF, Capacitor_SMD:C_0402_1005Metric
- removed C23, C28: 0.1uF, Capacitor_SMD:C_0402_1005Metric
- removed C24: 2.6pF, Capacitor_SMD:C_0402_1005Metric
- removed C25: 3.0pF, Capacitor_SMD:C_0402_1005Metric
- removed C27: 10uF, Capacitor_SMD:C_0402_1005Metric
- removed L5: 2.0nH, Inductor_SMD:L_0402_1005Metric
- removed R20, R21: 4.7k, Resistor_SMD:R_0402_1005Metric
- removed R22, R23: 10k, Resistor_SMD:R_0402_1005Metric
- removed U1: ESP32-C5, Package_DFN_QFN:QFN-48-1EP_6x6mm_P0.4mm_EP4.6x4.6mm
- removed Y1: Crystal_GND24, Crystal:Crystal_SMD_2016-4Pin_2.0x1.6mm
- added C1: 12pF, Capacitor_SMD:C_0201_0603Metric, F.Cu at (123.0, 90.3)
- added C11: 3pF, Capacitor_SMD:C_0402_1005Metric, F.Cu at (91.0, 116.6)
- added C12: 0.1uF, Capacitor_SMD:C_0402_1005Metric, F.Cu at (91.0, 118.6)
- added C13: 2.6pF, Capacitor_SMD:C_0402_1005Metric, F.Cu at (93.9, 110.7)
- added C14: 10uF, Capacitor_SMD:C_0402_1005Metric, F.Cu at (93.9, 112.7)
- added C2: 12pF, Capacitor_SMD:C_0201_0603Metric, F.Cu at (126.2, 90.3)
- added C4: 0.1uF, Capacitor_SMD:C_0402_1005Metric, F.Cu at (91.0, 110.7)
- added C48: 1uF, Capacitor_SMD:C_0402_1005Metric, F.Cu at (113.5, 103.9)
- added C49: 100nF, Capacitor_SMD:C_0402_1005Metric, F.Cu at (114.2, 110.2)
- added C5: 0.1uF, Capacitor_SMD:C_0402_1005Metric, F.Cu at (91.0, 112.7)
- added C50: 22uF 10V, Capacitor_SMD:C_0805_2012Metric, F.Cu at (118.1, 101.1)
- added C51: 22uF 16V, Capacitor_SMD:C_0805_2012Metric, F.Cu at (106.2, 102.7)
- added C52: 10pF, Capacitor_SMD:C_0402_1005Metric, F.Cu at (115.4, 103.9)
- added C53: 10pF, Capacitor_SMD:C_0402_1005Metric, F.Cu at (108.9, 105.1)
- added C8: 0.1uF, Capacitor_SMD:C_0402_1005Metric, F.Cu at (91.0, 114.7)
- added IC6: ESP32-C5HF4, SDM_Misc:QFN40P600X600X90-49N-D, F.Cu at (124.0, 97.4)
- added L8: 2.0nH, Inductor_SMD:L_0402_1005Metric, F.Cu at (95.8, 117.9)
- added R37: 10k, Resistor_SMD:R_0402_1005Metric, F.Cu at (95.8, 119.9)
- added R51: 27, Resistor_SMD:R_0402_1005Metric, F.Cu at (95.8, 121.9)
- added R52: 10k, Resistor_SMD:R_0402_1005Metric, F.Cu at (95.8, 123.9)
- added REF**: MountingHole_2.2mm_M2, MountingHole:MountingHole_2.2mm_M2, F.Cu at (135.5, 91.5)
- added REF**: MountingHole_2.2mm_M2, MountingHole:MountingHole_2.2mm_M2, F.Cu at (135.5, 108.5)
- added Y2: CX1612DB48000D0FPJC1, Smart_Watch:CX1612DB48000D0FPJC1, F.Cu at (124.6, 90.1)
- C15: value 1uF -> 0.1uF
- C16: value 1uF -> 0.8pF
- C17: value 10pF -> 0.3pF
- C19: value 10uF -> 1uF
- C20: value 0.3pF -> 1uF
- C21: value 0.8pF -> 1uF
- C26: value 0.1uF -> 1uF
- C29: value 10pF -> 10uF
- C31: value 10nF -> 10uF
- C32, C47: value 1uF -> 1uF 10V 0603; footprint Capacitor_SMD:C_0402_1005Metric -> Capacitor_SMD:C_0603_1608Metric
- C41: value 100nF -> 10uF 25V; footprint Capacitor_SMD:C_0402_1005Metric -> Capacitor_SMD:C_0805_2012Metric
- C42: value 22uF -> 22uF 10V; footprint Capacitor_SMD:C_0402_1005Metric -> Capacitor_SMD:C_0805_2012Metric
- C44: value 10nF -> 10uF 25V; footprint Capacitor_SMD:C_0402_1005Metric -> Capacitor_SMD:C_0805_2012Metric
- C45: value 22nF -> 22uF 16V; footprint Capacitor_SMD:C_0402_1005Metric -> Capacitor_SMD:C_0805_2012Metric
- J2: moved to F.Cu
- L6: footprint Inductor_SMD:L_0402_1005Metric -> Inductor_SMD:L_1008_2520Metric
- L7: footprint Inductor_SMD:L_0402_1005Metric -> Inductor_SMD:L_1210_3225Metric
- R49: value 27 -> 10k
- moved C17 56.2 mm to (149.9, 128.3)
- moved C26 56.2 mm to (152.8, 128.3)
- moved C35 56.2 mm to (155.6, 128.3)
- moved C15 56.2 mm to (149.9, 124.3)
- moved C16 56.2 mm to (149.9, 126.3)
- moved C33 56.2 mm to (155.6, 124.3)
- moved C34 56.2 mm to (155.6, 126.3)
- moved R49 54.5 mm to (145.5, 119.4)
- moved R50 52.6 mm to (140.1, 123.2)
- moved FL2 50.8 mm to (125.2, 116.8)
- moved U2 44.2 mm to (130.4, 116.8)
- moved C19 42.0 mm to (110.4, 121.7)
- moved C20 42.0 mm to (110.4, 123.6)
- moved C21 42.0 mm to (110.4, 125.6)
- moved C22 42.0 mm to (110.4, 127.6)
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Connections:
- C17 pad 1: GND -> +3.3V
- C17 pad 2: Net-(C17-Pad2) -> GND
- C19 pad 1: GND -> Net-(IC6-VDDA5)
- C19 pad 2: +3.3V -> GND
- C20 pad 1: GND -> +3.3V
- C20 pad 2: +3.3V -> GND
- C21 pad 1: GND -> Net-(IC6-CHIP_PU)
- C21 pad 2: +3.3V -> GND
- C29 pad 1: GND -> +3.3V
- C29 pad 2: Net-(U1-XTAL_N) -> GND
- IC2 pad 11: GND -> Net-(IC2-VREG5)
- L1 pad 2: Net-(C17-Pad2) -> Net-(C1-Pad1)
- R49 pad 1: Net-(U1-GPIO14/USB_D+/SDIO_DATA2) -> +3.3V
- R49 pad 2: Net-(R49-Pad2) -> Net-(IC6-CHIP_PU)
- R50 pad 1: Net-(R50-Pad1) -> Net-(IC6-GPIO14)
- R50 pad 2: Net-(U1-GPIO13/USB_D-/SDIO_DATA3) -> Net-(R50-Pad2)
- U2 pad 1: Net-(R49-Pad2) -> Net-(R50-Pad2)
- U2 pad 3: Net-(R50-Pad1) -> Net-(R51-Pad1)
Routing:
- net GND: track 18.8 -> 54.8 mm, vias 5 -> 24
- net VCC: track 8.87 -> 31.0 mm, vias 0 -> 9
- net +5V PreMUX: track 0.00 -> 19.6 mm, vias 0 -> 3
- net +3.3V: track 2.65 -> 14.9 mm
- net VBUS: track 2.45 -> 12.5 mm, vias 0 -> 2
- net Net-(IC2-SW2): track 0.00 -> 7.53 mm
- net /CAN-: track 11.6 -> 18.4 mm
- net /CAN_RTX: track 6.23 -> 0.00 mm
- net Net-(IC2-VFB2): track 0.00 -> 5.21 mm
- net Net-(IC3-CP2): track 0.00 -> 4.42 mm, vias 0 -> 2
- net /CAN_CTX: track 3.97 -> 0.00 mm
- net Net-(IC3-PR1): track 0.00 -> 3.91 mm
- net Net-(IC2-VFB1): track 0.00 -> 3.25 mm
- net Net-(IC6-XTAL_N): track 0.00 -> 2.85 mm
- net /5V_EN: track 0.00 -> 2.77 mm
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Other:
- outline, holes or cut-outs redrawn

Commit message: WB 90% + added buttons
Parts:
- removed ANT1: ANT3216LL00R2400A, RF_Antenna:Johanson_2450AT18x100
- removed C30, C33: 1pF, Capacitor_SMD:C_0402_1005Metric
- removed C34, C35: 2.2pF, Capacitor_SMD:C_0402_1005Metric
- removed C37, C38: 1.2pF, Capacitor_SMD:C_0402_1005Metric
- removed FL2: LFD182G45DCHD277, SDM:LFD182G45DCHD277
- removed L2, L3, L4: 2.8nH, Inductor_SMD:L_0402_1005Metric
- removed the REF** at (135.5, 91.5)
- removed the REF** at (135.5, 108.5)
- added REF**: MountingHole_2.2mm_M2, MountingHole:MountingHole_2.2mm_M2, F.Cu at (133.5, 91.0)
- added REF**: MountingHole_2.2mm_M2, MountingHole:MountingHole_2.2mm_M2, F.Cu at (133.5, 109.0)
- added REF**: MountingHole_2.2mm_M2, MountingHole:MountingHole_2.2mm_M2, F.Cu at (116.4, 95.3)
- added S1: SKTHBAE010, SDM_Misc:SKTHBAE010, F.Cu at (129.1, 108.7)
- added S2: SKTHBAE010, SDM_Misc:SKTHBAE010, F.Cu at (122.9, 108.7)
- C1, C11, C12, C14, C15, C2, C20, C21, C22, C26, C29, C8, J2, L1, L8, R37, R49, R52, Y2: moved to B.Cu
- moved C26 50.0 mm to (120.5, 90.0), turned to 180 degrees
- moved C17 44.7 mm to (126.3, 90.2), turned to 90 degrees
- moved C12 42.9 mm to (127.5, 96.0)
- moved C16 42.5 mm to (127.3, 90.2), turned to 90 degrees
- moved R52 39.8 mm to (125.5, 97.4)
- moved C11 39.3 mm to (124.0, 95.3), turned to -90 degrees
- moved C31 39.2 mm to (125.4, 90.2), turned to 90 degrees
- moved C14 38.5 mm to (127.6, 94.2)
- moved C15 38.3 mm to (127.6, 93.2)
- moved R37 38.0 mm to (125.5, 96.3)
- moved L8 37.6 mm to (125.5, 94.9), turned to 180 degrees
- moved R49 37.5 mm to (119.8, 92.1), turned to -90 degrees
- moved C8 37.3 mm to (123.0, 95.3), turned to -90 degrees
- moved C13 37.3 mm to (127.8, 95.2)
- moved C22 36.4 mm to (130.4, 97.1), turned to 180 degrees
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Connections:
- IC6 pad 11: /CAN_RTX -> /CAN_CTX
- IC6 pad 12: /CAN_CTX -> /CAN_RTX
- IC6 pad 17: /SDA -> unconnected-(IC6-GPIO8-Pad17)
- IC6 pad 18: /SCL -> unconnected-(IC6-GPIO9-Pad18)
- IC6 pad 20: /WSP_PWM -> unconnected-(IC6-GPIO11-Pad20)
- IC6 pad 34: unconnected-(IC6-GPIO24-Pad34) -> /WSP_PWM
- IC6 pad 35: unconnected-(IC6-GPIO25-Pad35) -> /SCL
- IC6 pad 36: unconnected-(IC6-GPIO26-Pad36) -> /SDA
- J2 pad 6: (no net) -> GND
- J2 pad 7: (no net) -> /USB_D+
- J2 pad 8: (no net) -> VBUS
- J2 pad 9: (no net) -> /USB_D-
- J2 pad MP: (no net) -> GND
Routing:
- net +3.3V: track 14.9 -> 47.7 mm, vias 0 -> 16
- net GND: track 54.8 -> 87.6 mm, vias 24 -> 88
- net +5V: track 0.00 -> 30.3 mm, vias 0 -> 2
- net Net-(IC6-CHIP_PU): track 0.00 -> 27.5 mm, vias 0 -> 2
- net Net-(IC6-BOOT): track 0.00 -> 23.4 mm, vias 0 -> 1
- net /SDA: track 0.00 -> 16.7 mm, vias 0 -> 1
- net /SCL: track 0.00 -> 13.8 mm, vias 0 -> 1
- net /WSP_PWM: track 0.00 -> 7.84 mm
- net Net-(IC6-GPIO13): track 0.00 -> 6.61 mm
- net VBUS: track 12.5 -> 18.3 mm, vias 2 -> 3
- net /CAN_CTX: track 0.00 -> 5.67 mm
- net Net-(IC6-GPIO14): track 0.00 -> 5.01 mm
- net /USB_D+: track 0.00 -> 4.91 mm, vias 0 -> 1
- net /USB_D-: track 0.00 -> 4.91 mm, vias 0 -> 1
- net /CAN_RTX: track 0.00 -> 4.27 mm
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- added copper zone on In2.Cu, net +3.3V
- added copper zone on In2.Cu, net GND
Other:
- board size 38 x 22 mm -> 35.5 x 22 mm

Commit message: A few more WB edits before bed
Parts:
- moved IC4 2.50 mm to (130.3, 100.0)
Changed lines of the file:
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@@
 	(footprint "SDM_Misc:MLX90614ESFBAA000SP"
 		(layer "F.Cu")
-		(at 128.557897 101.792105 45)
+		(at 130.3 100 45)
 		(descr "MLX90614ESF-BAA-000-SP")
 		(tags "Integrated Circuit")
-		(property "Reference" "IC4"
-			(at 2.6 -6.1 45)
-			(layer "F.SilkS")
-			(effects
-				(font
-					(size 1.27 1.27)
-					(thickness 0.254)
-				)
-			)
-		)
 		(property "Value" "MLX90614ESF-BAA-000-SP"
 			(at 2.54 0 45)
@@
 			)
 		)
-		(sheetname "/")
-		(sheetfile "SDM27_WheelBoard_v1.0.kicad_sch")
-		(units
-			(unit
-				(name "A")
-				(pins "2" "1" "3" "4")
+		(property "Reference" "IC4"
+			(at 0.06 -6.1 45)
+			(layer "F.SilkS")
+			(effects
+				(font
+					(size 1.27 1.27)
+					(thickness 0.254)
+				)
 			)
 		)
+		(sheetname "/")
+		(sheetfile "SDM27_WheelBoard_v1.0.kicad_sch")
 		(attr through_hole)
 		(duplicate_pad_numbers_are_jumpers no)
 		(fp_line
-			(start -0.86 -4)
-			(end -1.46 -3.4)
+			(start -3.4 -4)
+			(end -4 -3.4)
 			(stroke
 				(width 0.1)
@@
 		)
 		(fp_line
-			(start -1.46 -3.4)
-			(end -0.860001 -2.799998)
+			(start -4 -3.4)
+			(end -3.400001 -2.799998)
 			(stroke
 				(width 0.1)
@@
 		)
 		(fp_line
-			(start -0.259999 -3.400001)
-			(end -0.86 -4)
+			(start -2.799999 -3.400001)
+			(end -3.4 -4)
 			(stroke
 				(width 0.1)
@@
 		)
 		(fp_line
-			(start -1.833 0.000001)
-			(end -1.833 0.000001)
+			(start -4.373 0.000001)
+			(end -4.373 0.000001)
 			(stroke
 				(width 0.1)
@@
 		)
 		(fp_line
-			(start 6.913 0)
-			(end 6.913 0)
+			(start 4.373 0)
+			(end 4.373 0)
 			(stroke
 				(width 0.1)
@@
 		)
 		(fp_arc
-			(start -1.833 0.000001)
-			(mid 2.54 -4.372997)
-			(end 6.913 0)
+			(start -4.373 0.000001)
+			(mid -0.000001 -4.372998)
+			(end 4.373 0)
 			(stroke
 				(width 0.1)
@@
 		)
 		(fp_arc
-			(start 6.913 0)
-			(mid 2.540002 4.373002)
-			(end -1.833 0.000001)
+			(start 4.373 0)
+			(mid 0.000001 4.373002)
+			(end -4.373 0.000001)
 			(stroke
 				(width 0.1)
@@
 		)
 		(fp_circle
-			(center 2.600001 0)
-			(end 2.600001 -5.400001)
+			(center 0.060001 0)
+			(end 0.060001 -5.400001)
 			(stroke
 				(width 0.05)
@@
 		)
 		(fp_line
-			(start -0.86 -4)
-			(end -0.259999 -3.400001)
+			(start -3.4 -4)
+			(end -2.799999 -3.400001)
 			(stroke
 				(width 0.2)
@@
 		)
 		(fp_line
-			(start -1.46 -3.4)
-			(end -0.86 -4)
+			(start -4 -3.4)
+			(end -3.4 -4)
 			(stroke
 				(width 0.2)
@@
 		)
 		(fp_line
-			(start -0.860001 -2.799998)
-			(end -1.46 -3.4)
+			(start -3.400001 -2.799998)
+			(end -4 -3.4)
 			(stroke
 				(width 0.2)
@@
 		)
 		(fp_line
-			(start -1.833 0.000001)
-			(end -1.833 0.000001)
+			(start -4.373 0.000001)
+			(end -4.373 0.000001)
 			(stroke
 				(width 0.2)
@@
 		)
 		(fp_line
-			(start 6.913 0)
-			(end 6.913 0)
+			(start 4.373 0)
+			(end 4.373 0)
 			(stroke
 				(width 0.2)
@@
 		)
 		(fp_arc
-			(start -1.833 0.000001)
-			(mid 2.54 -4.372997)
-			(end 6.913 0)
+			(start -4.373 0.000001)
+			(mid -0.000001 -4.372998)
+			(end 4.373 0)
 			(stroke
 				(width 0.2)
@@
 		)
 		(fp_arc
-			(start 6.913 0)
-			(mid 2.540002 4.373002)
-			(end -1.833 0.000001)
+			(start 4.373 0)
+			(mid 0.000001 4.373002)
+			(end -4.373 0.000001)
 			(stroke
 				(width 0.2)
@@
 		)
 		(pad "1" thru_hole circle
-			(at 0 0 45)
+			(at -2.54 0 45)
 			(size 1.2 1.2)
 			(drill 0.69)
@@
 		)
 		(pad "2" thru_hole circle
-			(at 2.54 2.54 45)
+			(at 0 2.54 45)
 			(size 1.2 1.2)
 			(drill 0.69)
@@
 		)
 		(pad "3" thru_hole circle
-			(at 5.080002 -0.000001 45)
+			(at 2.540002 -0.000001 45)
 			(size 1.2 1.2)
 			(drill 0.69)
@@
 		)
 		(pad "4" thru_hole circle
-			(at 2.54 -2.54 45)
+			(at 0 -2.54 45)
 			(size 1.2 1.2)
 			(drill 0.69)
@@
 		(layer "Edge.Cuts")
 	)
+	(dimension
+		(type orthogonal)
+		(layer "Edge.Cuts")
+		(pts
+			(xy 131 89) (xy 130.999999 111)
+		)
+		(height 8)
+		(orientation 1)
+		(format
+			(prefix "")
+			(suffix "")
+			(units 3)
+			(units_format 0)
+			(precision 4)
+			(suppress_zeroes yes)
+		)
+		(style
+			(thickness 0.05)
+			(arrow_length 1.27)
+			(text_position_mode 0)
+			(arrow_direction outward)
+			(extension_height 0.58642)
+			(extension_offset 0.5)
+			(keep_text_aligned yes)
+		)
+		(gr_text "22"
+			(at 137.85 100 90)
+			(layer "Edge.Cuts")
+			(effects
+				(font
+					(size 1 1)
+					(thickness 0.15)
+				)
+			)
+		)
+	)
+	(dimension
+		(type orthogonal)
+		(layer "Edge.Cuts")
+		(pts
+			(xy 135.5 94) (xy 100 100.4)
+		)
+		(height -6.5)
+		(orientation 0)
+		(format
+			(prefix "")
+			(suffix "")
+			(units 3)
+			(units_format 0)
+			(precision 4)
+			(suppress_zeroes yes)
+		)
+		(style
+			(thickness 0.05)
+			(arrow_length 1.27)
+			(text_position_mode 0)
+			(arrow_direction outward)
+			(extension_height 0.58642)
+			(extension_offset 0.5)
+			(keep_text_aligned yes)
+		)
+		(gr_text "35.5"
+			(at 117.75 86.35 0)
+			(layer "Edge.Cuts")
+			(effects
+				(font
+					(size 1 1)
+					(thickness 0.15)
+				)
+			)
+		)
+	)
+	(dimension
+		(type orthogonal)
+		(layer "Edge.Cuts")
+		(pts
+			(xy 135 109) (xy 132 109.049999)
+		)
+		(height -1.5)
+		(orientation 0)
+		(format
+			(prefix "")
+			(suffix "")
+			(units 3)
+			(units_format 0)
+			(precision 4)
+			(suppress_zeroes yes)
+		)
+		(style
+			(thickness 0.05)
+			(arrow_length 1.27)
+			(text_position_mode 0)
+			(arrow_direction outward)
+			(extension_height 0.58642)
+			(extension_offset 0.5)
+			(keep_text_aligned yes)
+		)
+		(gr_text "3"
+			(at 133.5 106.35 0)
+			(layer "Edge.Cuts")
+			(effects
+				(font
+					(size 1 1)
+					(thickness 0.15)
+				)
+			)
+		)
+	)
 	(segment
