File: 2027/SDM27_WheelBoard/SDM27_WheelBoard_v1.0/SDM27_WheelBoard_v1.0.kicad_pcb (KiCad board)
At the start: 4 copper layers, 35.5 x 22 mm, 87 parts, among them IC1 TPS2121RUXR, IC2 TPS542951RSAR, IC3 TPS2121RUXR, IC4 MLX90614ESF-BAA-000-SP, IC5 SN74LVC1G17YZPR, IC6 ESP32-C5HF4, IC8 TCAN3403DRBRQ1, J1 WEIPU SA12 7PIN, J2 WEIPU SA6 5Pin, U2 USBLC6-2SC6, Y2 CX1612DB48000D0FPJC1

Commit message: SDM27 WB - added USBC and UFL
Parts:
- removed the REF** at (133.5, 91.0)
- added C3: 2.2pF 25V NPO, Capacitor_SMD:C_0402_1005Metric, F.Cu at (131.0, 93.4)
- added C6: 2.2pF 25V NPO, Capacitor_SMD:C_0402_1005Metric, F.Cu at (130.6, 91.6)
- added J4: UFL, SDM_Misc:CONUFL001SMDT, F.Cu at (134.3, 91.7)
- added J5: USB4725-03-C-KIT, SDM_Misc:GCT_USB4730-GF-A_REVA, B.Cu at (135.2, 100.0)
- added L3: 2.8nH, Inductor_SMD:L_0402_1005Metric, F.Cu at (129.6, 92.9)
- added R53: 5.1k, Resistor_SMD:R_0402_1005Metric, F.Cu at (136.1, 102.9)
- added R54: 5.1k, Resistor_SMD:R_0402_1005Metric, F.Cu at (136.2, 97.1)
- C1, C2: footprint Capacitor_SMD:C_0201_0603Metric -> Capacitor_SMD:C_0402_1005Metric
- C22: moved to F.Cu
- J2: footprint Connector_JST:JST_SH_BM09B-SRSS-TB_1x09-1MP_P1.00mm_Vertical -> Connector_JST:JST_SH_BM05B-SRSS-TB_1x05-1MP_P1.00mm_Vertical
- moved C22 17.0 mm to (132.5, 114.0), turned to 0 degrees
- moved J2 2.04 mm to (128.2, 108.6)
- moved REF** 1.12 mm to (134.5, 108.5)
- moved C2 0.24 mm to (124.9, 91.8)
- moved C1 0.10 mm to (122.6, 92.1)
Connections:
- IC6 pad 42: /ANT2.4G -> /2.4ghz
- IC6 pad 48: /ANT5G -> unconnected-(IC6-ANT_5G-Pad48)
- J2 pad MP: GND -> (no net)
Routing:
- net VBUS: track 18.3 -> 64.7 mm, vias 3 -> 5
- net /USB_D+: track 4.91 -> 15.1 mm
- net /USB_D-: track 4.91 -> 13.7 mm
- net Net-(J5-CC2): track 0.00 -> 7.39 mm, vias 0 -> 1
- net Net-(J5-CC1): track 0.00 -> 7.31 mm, vias 0 -> 1
- net /2.4ghz: track 0.00 -> 5.24 mm
- net Net-(J4-A): track 0.00 -> 3.56 mm
- net GND: track 87.6 -> 90.5 mm, vias 88 -> 128
- net +3.3V: track 47.7 -> 46.2 mm
- net /SDA: track 16.7 -> 17.6 mm
- net +5V: track 30.3 -> 31.1 mm
- net VCC: vias 9 -> 8
Other:
- board size 35.5 x 22 mm -> 37 x 22 mm
