File: 2026/BSPD/SDM26_BSPD_V1.0/SDM26_BSPD_V1.0.kicad_pcb (KiCad board)
At the start: 4 copper layers, 90 x 40 mm, 84 parts, among them IC1 LM2901BIRTER, IC2 LM2901BIRTER, IC3 SN74HC08PWR, IC4 SN74HC32PWR, IC5 L7805ACD2T-TR, J1 776280-1, Q1 2N7002,215, U1 TPS2116DRL

Commit message: Library maintenance
edited some 3dmodles to point to their footprints. edited symbols and footprints to link properly. edited footprint and symbol library names in all projects 2026-2027 to use the same library nick name "SDM" for both  symbol and footprint.
all users must delete their old lib and make a new one named SDM for symbol and footprint.
Parts:
- BLACK_TP1: footprint SDM_MiscFootprint:5006 -> SDM:5006
- D1, D4, D6: footprint SDM_MiscFootprint:SODFL1608X70N -> SDM:SODFL1608X70N
- IC1, IC2: footprint SDM_MiscFootprint:QFN50P300X300X80-17N-D -> SDM:QFN50P300X300X80-17N-D
- IC3: footprint SDM_MiscFootprint:SOT65P212X110-5L -> SDM:SOT65P212X110-5L
- IC4: footprint SDM_MiscFootprint:SOP65P640X120-14L -> SDM:SOP65P640X120-14L
- IC5: footprint SDM_MiscFootprint:L7805ACD2TTR -> SDM:L7805ACD2TTR
- J1: footprint SDM_MiscFootprint:776280-1 -> SDM:776280-1
- LED1, LED2, LED3, LED4, LED5, LED6, LED7, LED8, LED9: footprint SDM_MiscFootprint:LEDC1608X80N -> SDM:LEDC1608X80N
- Q1: footprint SDM_MiscFootprint:SOT95P230X110-3N -> SDM:SOT95P230X110-3N
- RED_TP1, RED_TP2, RED_TP3, RED_TP4, RED_TP5, RED_TP6: footprint SDM_MiscFootprint:5005 -> SDM:5005
- VR1, VR2, VR3, VR4, VR5, VR6: footprint SDM_MiscFootprint:3386P1103TLF -> SDM:3386P1103TLF
- WHITE_TP1, WHITE_TP2: footprint SDM_MiscFootprint:5007 -> SDM:5007
Changed lines of the file:
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@@
 		)
 	)
-	(footprint "SDM_MiscFootprint:776280-1"
+	(footprint "SDM:776280-1"
 		(layer "F.Cu")
 		(at 97.9 120 -90)
@@
 		)
 	)
-	(footprint "SDM_MiscFootprint:5005"
+	(footprint "SDM:5005"
 		(layer "F.Cu")
 		(at 169 116)
@@
 		(embedded_fonts no)
 	)
-	(footprint "SDM_MiscFootprint:LEDC1608X80N"
+	(footprint "SDM:LEDC1608X80N"
 		(layer "F.Cu")
 		(at 140.6 138.5)
@@
 		)
 	)
-	(footprint "SDM_MiscFootprint:5005"
+	(footprint "SDM:5005"
 		(layer "F.Cu")
 		(at 165 116)
@@
 		)
 	)
-	(footprint "SDM_MiscFootprint:3386P1103TLF"
+	(footprint "SDM:3386P1103TLF"
 		(layer "F.Cu")
 		(at 119 106 180)
@@
 		)
 	)
-	(footprint "SDM_MiscFootprint:QFN50P300X300X80-17N-D"
+	(footprint "SDM:QFN50P300X300X80-17N-D"
 		(layer "F.Cu")
 		(at 149.35 117.9 180)
@@
 		)
 	)
-	(footprint "SDM_MiscFootprint:LEDC1608X80N"
+	(footprint "SDM:LEDC1608X80N"
 		(layer "F.Cu")
 		(at 181 137.7)
@@
 		)
 	)
-	(footprint "SDM_MiscFootprint:5006"
+	(footprint "SDM:5006"
 		(layer "F.Cu")
 		(at 165 129)
@@
 		)
 	)
-	(footprint "SDM_MiscFootprint:SOP65P640X120-14L"
+	(footprint "SDM:SOP65P640X120-14L"
 		(layer "F.Cu")
 		(at 140.938 121.55 180)
@@
 		)
 	)
-	(footprint "SDM_MiscFootprint:LEDC1608X80N"
+	(footprint "SDM:LEDC1608X80N"
 		(layer "F.Cu")
 		(at 144.9 138.5 180)
@@
 		)
 	)
-	(footprint "SDM_MiscFootprint:SODFL1608X70N"
+	(footprint "SDM:SODFL1608X70N"
 		(layer "F.Cu")
 		(at 143.711436 126.670883 90)
@@
 		)
 	)
-	(footprint "SDM_MiscFootprint:5007"
+	(footprint "SDM:5007"
 		(layer "F.Cu")
 		(at 181 129)
@@
 		)
 	)
-	(footprint "SDM_MiscFootprint:LEDC1608X80N"
+	(footprint "SDM:LEDC1608X80N"
 		(layer "F.Cu")
 		(at 136.425 138.5)
@@
 		)
 	)
-	(footprint "SDM_MiscFootprint:SODFL1608X70N"
+	(footprint "SDM:SODFL1608X70N"
 		(layer "F.Cu")
 		(at 132.95 116.5)
@@
 		)
 	)
-	(footprint "SDM_MiscFootprint:LEDC1608X80N"
+	(footprint "SDM:LEDC1608X80N"
 		(layer "F.Cu")
 		(at 173 137.7)
@@
 		)
 	)
-	(footprint "SDM_MiscFootprint:5005"
+	(footprint "SDM:5005"
 		(layer "F.Cu")
 		(at 181 116)
@@
 		)
 	)
-	(footprint "SDM_MiscFootprint:LEDC1608X80N"
+	(footprint "SDM:LEDC1608X80N"
 		(layer "F.Cu")
 		(at 177 137.7)
@@
 		)
 	)
-	(footprint "SDM_MiscFootprint:QFN50P300X300X80-17N-D"
+	(footprint "SDM:QFN50P300X300X80-17N-D"
 		(layer "F.Cu")
 		(at 123.55 116.05 180)
@@
 		)
 	)
-	(footprint "SDM_MiscFootprint:3386P1103TLF"
+	(footprint "SDM:3386P1103TLF"
 		(layer "F.Cu")
 		(at 180.5 106 180)
@@
 		)
 	)
-	(footprint "SDM_MiscFootprint:L7805ACD2TTR"
+	(footprint "SDM:L7805ACD2TTR"
 		(layer "F.Cu")
 		(at 124.818 132.4 90)
@@
 		)
 	)
-	(footprint "SDM_MiscFootprint:LEDC1608X80N"
+	(footprint "SDM:LEDC1608X80N"
 		(layer "F.Cu")
 		(at 169 137.7)
@@
 		)
 	)
-	(footprint "SDM_MiscFootprint:SOT95P230X110-3N"
+	(footprint "SDM:SOT95P230X110-3N"
 		(layer "F.Cu")
 		(at 145.7 130.95)
@@
 		)
 	)
-	(footprint "SDM_MiscFootprint:3386P1103TLF"
+	(footprint "SDM:3386P1103TLF"
 		(layer "F.Cu")
 		(at 131.3 106 180)
@@
 		)
 	)
-	(footprint "SDM_MiscFootprint:SOT65P212X110-5L"
+	(footprint "SDM:SOT65P212X110-5L"
 		(layer "F.Cu")
 		(at 134.1 120.15)
@@
 		)
 	)
-	(footprint "SDM_MiscFootprint:3386P1103TLF"
+	(footprint "SDM:3386P1103TLF"
 		(layer "F.Cu")
 		(at 143.62 106 180)
@@
 		)
 	)
-	(footprint "SDM_MiscFootprint:SODFL1608X70N"
+	(footprint "SDM:SODFL1608X70N"
 		(layer "F.Cu")
 		(at 141.8 116.5)
@@
 		)
 	)
-	(footprint "SDM_MiscFootprint:LEDC1608X80N"
+	(footprint "SDM:LEDC1608X80N"
 		(layer "F.Cu")
 		(at 165 137.7)
@@
 		)
 	)
-	(footprint "SDM_MiscFootprint:LEDC1608X80N"
+	(footprint "SDM:LEDC1608X80N"
 		(layer "F.Cu")
 		(at 185 137.7)
@@
 		)
 	)
-	(footprint "SDM_MiscFootprint:5007"
+	(footprint "SDM:5007"
 		(layer "F.Cu")
 		(at 185 129)
@@
 		)
 	)
-	(footprint "SDM_MiscFootprint:5005"
+	(footprint "SDM:5005"
 		(layer "F.Cu")
 		(at 185 116)
@@
 		)
 	)
-	(footprint "SDM_MiscFootprint:3386P1103TLF"
+	(footprint "SDM:3386P1103TLF"
 		(layer "F.Cu")
 		(at 155.9 106 180)
@@
 		)
 	)
-	(footprint "SDM_MiscFootprint:3386P1103TLF"
+	(footprint "SDM:3386P1103TLF"
 		(layer "F.Cu")
 		(at 168.2 106 180)
@@
 		)
 	)
-	(footprint "SDM_MiscFootprint:5005"
+	(footprint "SDM:5005"
 		(layer "F.Cu")
 		(at 173 116)
@@
 		)
 	)
-	(footprint "SDM_MiscFootprint:5005"
+	(footprint "SDM:5005"
 		(layer "F.Cu")
 		(at 177 116)
