File: 2026/BSPD_Test_Bench/SDM26_BSPD_Test_Bench_V1.0/SDM26_BSPD_Test_Bench_V1.0.kicad_sch (KiCad schematic)
At the start: 10 parts, among them J1 SM04B-ULHK-1TA1-ETB_HF_, U1 SPX2920U-5.0_TO220

Commit message: Library maintenance
edited some 3dmodles to point to their footprints. edited symbols and footprints to link properly. edited footprint and symbol library names in all projects 2026-2027 to use the same library nick name "SDM" for both  symbol and footprint.
all users must delete their old lib and make a new one named SDM for symbol and footprint.
Parts:
- J1: footprint Library:SM04BULHK1TA1ETBHF -> SDM:SM04BULHK1TA1ETBHF; symbol SDM_CONNECTOR:SM04B-ULHK-1TA1-ETB_HF_ -> SDM:SM04B-ULHK-1TA1-ETB_HF_
Changed lines of the file:
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@@
 	)
 	(symbol
-		(lib_id "SDM_CONNECTOR:SM04B-ULHK-1TA1-ETB_HF_")
+		(lib_id "SDM:SM04B-ULHK-1TA1-ETB_HF_")
 		(at 66.04 64.77 0)
 		(unit 1)
@@
 			)
 		)
-		(property "Footprint" "Library:SM04BULHK1TA1ETBHF"
+		(property "Footprint" "SDM:SM04BULHK1TA1ETBHF"
 			(at 85.09 159.69 0)
 			(effects
