File: 2026/IMU/SDM26_IMU_V1.1/SDM26_IMU_V1.1.kicad_pcb (KiCad board)
At the start: 4 copper layers, 52 x 41 mm, 65 parts, among them IC1 ESP32-S3-WROOM-1-N8R8, IC2 TLP175A_TPL,E, IC3 ISM330DHCXTR, IC4 TPS2116DRLR, IC5 MIC37100-3.3WS, IC6 CP2102N-A02-GQFN28, IC7 IIS2MDCTR, J1 USB_B_Micro, J2 Conn_01x04_Socket, Q1 MMBT2222LT1G, Q2 MMBT2222LT1G, U1 SN65HVD230, U2 USBLC6-2SC6

Commit message: Library maintenance
edited some 3dmodles to point to their footprints. edited symbols and footprints to link properly. edited footprint and symbol library names in all projects 2026-2027 to use the same library nick name "SDM" for both  symbol and footprint.
all users must delete their old lib and make a new one named SDM for symbol and footprint.
Parts:
- D1: footprint SDM_MiscFootprint:SOT65P210X110-3N -> SDM:SOT65P210X110-3N
- IC2: footprint SDM_MiscFootprint:TLP266J -> SDM:TLP266J
- IC3: footprint SDM_MiscFootprint:LSM6DS3USTR -> SDM:LSM6DS3USTR
- IC6: footprint SDM_MiscFootprint:QFN50P500X500X80-29N-D -> SDM:QFN50P500X500X80-29N-D
- IC7: footprint SDM_MiscFootprint:IIS2MDCTR -> SDM:IIS2MDCTR
- LED1, LED2: footprint SDM_MiscFootprint:LEDC1608X80N -> SDM:LEDC1608X80N
- Q1: footprint SDM_MiscFootprint:SOT96P237X111-3N -> SDM:SOT96P237X111-3N
Changed lines of the file:
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@@
 		)
 	)
-	(footprint "SDM_MiscFootprint:SOT96P237X111-3N"
+	(footprint "SDM:SOT96P237X111-3N"
 		(layer "F.Cu")
 		(at 81.835 66.43 90)
@@
 		)
 	)
-	(footprint "SDM_MiscFootprint:LEDC1608X80N"
+	(footprint "SDM:LEDC1608X80N"
 		(layer "F.Cu")
 		(at 94.44 63.89)
@@
 		)
 	)
-	(footprint "SDM_MiscFootprint:LSM6DS3USTR"
+	(footprint "SDM:LSM6DS3USTR"
 		(layer "F.Cu")
 		(at 93.938 70.597)
@@
 		)
 	)
-	(footprint "SDM_MiscFootprint:IIS2MDCTR"
+	(footprint "SDM:IIS2MDCTR"
 		(layer "F.Cu")
 		(at 96.81 77.71)
@@
 		)
 	)
-	(footprint "SDM_MiscFootprint:TLP266J"
+	(footprint "SDM:TLP266J"
 		(layer "F.Cu")
 		(at 70.355 47.33)
@@
 		)
 	)
-	(footprint "SDM_MiscFootprint:SOT65P210X110-3N"
+	(footprint "SDM:SOT65P210X110-3N"
 		(layer "F.Cu")
 		(at 76.455 48.15 90)
@@
 		)
 	)
-	(footprint "SDM_MiscFootprint:LEDC1608X80N"
+	(footprint "SDM:LEDC1608X80N"
 		(layer "F.Cu")
 		(at 85.045 81.69 180)
@@
 		)
 	)
-	(footprint "SDM_MiscFootprint:QFN50P500X500X80-29N-D"
+	(footprint "SDM:QFN50P500X500X80-29N-D"
 		(layer "F.Cu")
 		(at 75.305 67.6)
