File: 2026/Logger/SDM26_Logger_V1.0/SDM26Logger.kicad_sch (KiCad schematic)
At the start: 95 parts, among them IC1 ESP32-S3-WROOM-1-N8R8, IC2 NEO-F9P-15B, IC3 MIC37100-3.3WS, IC5 TPS563211DRLR, IC6 CP2102N-A02-GQFN28, J1 USB_B, J2 USB_B_Micro, J3 1-776087-4, J4 Molex_1040310811, J5 USB_B_Micro, Q1 SOT96P237X111-3N, Q2 SOT96P237X111-3N, U1 INA260, U11 ADC128S102, U2 TPS2116DRL, U3 ADR425BRZ, U4 SN65HVD230, U5 USBLC6-2SC6, U6 USBLC6-2SC6, U7 USBLC6-2SC6, U8 TPS2116, U9 ST_EMIF06-MSD02N16, Y2 ECX-.327-CDX-2096

Commit message: Library maintenance
edited some 3dmodles to point to their footprints. edited symbols and footprints to link properly. edited footprint and symbol library names in all projects 2026-2027 to use the same library nick name "SDM" for both  symbol and footprint.
all users must delete their old lib and make a new one named SDM for symbol and footprint.
Parts:
- IC2: footprint NEOF9P15B -> SDM:NEOF9P15B; symbol GNSS:NEO-F9P-15B -> SDM:NEO-F9P-15B
- IC3: footprint SOT230P700X180-4N -> SDM:SOT230P700X180-4N; symbol VoltageRegulators:MIC37100-3.3WS -> SDM:MIC37100-3.3WS
- IC5: footprint SOTFL50P160X60-8N -> SDM:SOTFL50P160X60-8N; symbol VoltageRegulators:TPS563211DRLR -> SDM:TPS563211DRLR
- IC6: footprint QFN50P500X500X80-29N-D -> SDM:QFN50P500X500X80-29N-D; symbol USBUART:CP2102N-A02-GQFN28 -> SDM:CP2102N-A02-GQFN28
- J1: footprint USBs:67068-7041 -> SDM:67068-7041
- J3: footprint Connectors:CONN23_776087_TEC -> SDM:CONN23_776087_TEC
- LED2, LED3: footprint SSFLXH100LID01 -> SDM:SSFLXH100LID01; symbol LEDs:SSF-LXH100LID-01 -> SDM:SSF-LXH100LID-01
- Q1, Q2: footprint Transistors:SOT96P237X111-3N -> SDM:SOT96P237X111-3N
- U11: symbol lib:TI_ADC128S102 -> SDM:TI_ADC128S102
- U8: footprint VoltageRegulators:SOT-5X3 -> SDM:SOT-5X3
Changed lines of the file:
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@@
 	)
 	(symbol
-		(lib_id "VoltageRegulators:TPS563211DRLR")
+		(lib_id "SDM:TPS563211DRLR")
 		(at 265.43 77.47 0)
 		(unit 1)
@@
 			)
 		)
-		(property "Footprint" "SOTFL50P160X60-8N"
+		(property "Footprint" "SDM:SOTFL50P160X60-8N"
 			(at 292.1 172.39 0)
 			(effects
@@
 	)
 	(symbol
-		(lib_id "VoltageRegulators:MIC37100-3.3WS")
+		(lib_id "SDM:MIC37100-3.3WS")
 		(at 383.54 69.85 270)
 		(unit 1)
@@
 			)
 		)
-		(property "Footprint" "SOT230P700X180-4N"
+		(property "Footprint" "SDM:SOT230P700X180-4N"
 			(at 288.62 96.52 0)
 			(effects
@@
 	)
 	(symbol
-		(lib_id "USBUART:CP2102N-A02-GQFN28")
+		(lib_id "SDM:CP2102N-A02-GQFN28")
 		(at 190.5 60.96 0)
 		(unit 1)
@@
 			)
 		)
-		(property "Footprint" "QFN50P500X500X80-29N-D"
+		(property "Footprint" "SDM:QFN50P500X500X80-29N-D"
 			(at 229.87 145.72 0)
 			(effects
@@
 	)
 	(symbol
-		(lib_id "lib:TI_ADC128S102")
+		(lib_id "SDM:TI_ADC128S102")
 		(at 233.68 161.29 0)
 		(unit 1)
@@
 			)
 		)
-		(property "Footprint" "VoltageRegulators:SOT-5X3"
+		(property "Footprint" "SDM:SOT-5X3"
 			(at 374.65 111.76 0)
 			(effects
@@
 	)
 	(symbol
-		(lib_id "LEDs:SSF-LXH100LID-01")
+		(lib_id "SDM:SSF-LXH100LID-01")
 		(at 375.92 59.69 90)
 		(unit 1)
@@
 			)
 		)
-		(property "Footprint" "SSFLXH100LID01"
+		(property "Footprint" "SDM:SSFLXH100LID01"
 			(at 469.57 46.99 0)
 			(effects
@@
 	)
 	(symbol
-		(lib_id "GNSS:NEO-F9P-15B")
+		(lib_id "SDM:NEO-F9P-15B")
 		(at 306.07 170.18 0)
 		(unit 1)
@@
 			)
 		)
-		(property "Footprint" "NEOF9P15B"
+		(property "Footprint" "SDM:NEOF9P15B"
 			(at 350.52 265.1 0)
 			(effects
@@
 			)
 		)
-		(property "Footprint" "Connectors:CONN23_776087_TEC"
+		(property "Footprint" "SDM:CONN23_776087_TEC"
 			(at 133.35 179.07 0)
 			(effects
@@
 			)
 		)
-		(property "Footprint" "Transistors:SOT96P237X111-3N"
+		(property "Footprint" "SDM:SOT96P237X111-3N"
 			(at 294.64 38.1 0)
 			(effects
@@
 	)
 	(symbol
-		(lib_id "LEDs:SSF-LXH100LID-01")
+		(lib_id "SDM:SSF-LXH100LID-01")
 		(at 393.7 193.04 180)
 		(unit 1)
@@
 			)
 		)
-		(property "Footprint" "SSFLXH100LID01"
+		(property "Footprint" "SDM:SSFLXH100LID01"
 			(at 381 99.39 0)
 			(effects
@@
 			)
 		)
-		(property "Footprint" "USBs:67068-7041"
+		(property "Footprint" "SDM:67068-7041"
 			(at 140.97 38.1 0)
 			(effects
@@
 			)
 		)
-		(property "Footprint" "Transistors:SOT96P237X111-3N"
+		(property "Footprint" "SDM:SOT96P237X111-3N"
 			(at 294.64 21.59 0)
 			(effects
