File: 2026/Logger/SDM26_Logger_V2.0/SDM26LoggerV2.kicad_pcb (KiCad board)
At the start: 4 copper layers, 101 x 60 mm, 98 parts, among them IC1 ESP32-S3-WROOM-1-N8R8, IC2 NEO-F9P-15B, IC3 MIC37100-3.3WS, IC5 TPS563211DRLR, IC6 CP2102N-A02-GQFN28, J1 USB_B, J2 USB_B_Micro, J3 1-776087-4, J4 Molex_1040310811, J5 USB_B_Micro, J6 1-776087-4, K1 IMB03IGR, Q1 SOT96P237X111-3N, Q2 SOT96P237X111-3N, U1 INA260, U11 ADC128S102, U2 TPS2116DRL, U3 ADR425BRZ, U4 SN65HVD230, U5 USBLC6-2SC6, U6 USBLC6-2SC6, U7 USBLC6-2SC6, U8 TPS2116, U9 ST_EMIF06-MSD02N16, Y2 ECX-.327-CDX-2096

Commit message: Library maintenance
edited some 3dmodles to point to their footprints. edited symbols and footprints to link properly. edited footprint and symbol library names in all projects 2026-2027 to use the same library nick name "SDM" for both  symbol and footprint.
all users must delete their old lib and make a new one named SDM for symbol and footprint.
Parts:
- D2: footprint Diodes:SOT65P210X110-3N -> SDM:SOT65P210X110-3N
- IC2: footprint GNSS:NEOF9P15B -> SDM:NEOF9P15B
- IC5: footprint VoltageRegulators:SOTFL50P160X60-8N -> SDM:SOTFL50P160X60-8N
- J1: footprint USBs:67068-7041 -> SDM:67068-7041
- K1: footprint Relays:IMB03IGR -> SDM:IMB03IGR
- Q1, Q2: footprint Transistors:SOT96P237X111-3N -> SDM:SOT96P237X111-3N
- U8: footprint VoltageRegulators:SOT-5X3 -> SDM:SOT-5X3
- Y2: footprint Crystals:ECX327CDX2096 -> SDM:ECX327CDX2096
