File: 2026/Logger/SDM26_Logger_V3.3/SDM26LoggerV3.3.kicad_sch (KiCad schematic)
At the start: 134 parts, among them IC1 ESP32-S3-WROOM-1-N8R8, IC2 CP2102N-A02-GQFN28, IC3 MIC37100-3.3WS, IC4 TPS563211DRLR, IC5 TLP175A_TPL,E, IC6 MIC37100-3.3WS, IC7 NEO-F9P-15B, IC8 TPS259250DRCR, J1 UART_USB, J2 ESP_USB, J3 GNSS_Debug, J4 Molex_1040310811, J5 1-776087-4, J6 1-776087-4, Q1 MMBT2222LT1G, Q2 MMBT2222LT1G, U1 INA260, U10 EMIF06-MSD02N16, U2 USBLC6-2SC6, U3 TPS2116DRL, U4 USBLC6-2SC6, U5 USBLC6-2SC6, U6 TPS2116, U7 SN65HVD230, U8 ADR425BRZ, U9 ADC128S102, Y1 ECX-.327-CDX-2096

Commit message: Library maintenance
edited some 3dmodles to point to their footprints. edited symbols and footprints to link properly. edited footprint and symbol library names in all projects 2026-2027 to use the same library nick name "SDM" for both  symbol and footprint.
all users must delete their old lib and make a new one named SDM for symbol and footprint.
Parts:
- D1: footprint SDM_MiscFootprint:SOT65P210X110-3N -> SDM:SOT65P210X110-3N; symbol SDM_ESD:ESDCAN03-2BWY -> SDM:ESDCAN03-2BWY
- D2, D3, D4, D5, D6, D7, D8, D9: footprint SDM_MiscFootprint:SOD3716X135N -> SDM:SOD3716X135N; symbol SDM_DIODES:MBR0540T1G -> SDM:MBR0540T1G
- IC1: footprint SDM_MiscFootprint:ESP32S3WROOM1N8R8 -> SDM:ESP32S3WROOM1N8R8
- IC2: footprint SDM_MiscFootprint:QFN50P500X500X80-29N-D -> SDM:QFN50P500X500X80-29N-D; symbol SDM_USBUART:CP2102N-A02-GQFN28 -> SDM:CP2102N-A02-GQFN28
- IC3, IC6: footprint SDM_MiscFootprint:SOT230P700X180-4N -> SDM:SOT230P700X180-4N; symbol SDM_VOLTAGE_REGULATORS:MIC37100-3.3WS -> SDM:MIC37100-3.3WS
- IC4: footprint SDM_MiscFootprint:SOTFL50P160X60-8N -> SDM:SOTFL50P160X60-8N; symbol SDM_VOLTAGE_REGULATORS:TPS563211DRLR -> SDM:TPS563211DRLR
- IC5: footprint SDM_MiscFootprint:TLP266J -> SDM:TLP266J
- IC7: footprint SDM_MiscFootprint:NEOF9P15B -> SDM:NEOF9P15B; symbol SDM_GNSS:NEO-F9P-15B -> SDM:NEO-F9P-15B
- IC8: footprint SDM_MiscFootprint:SON50P300X300X100-11L-D -> SDM:SON50P300X300X100-11L-D
- J1: footprint SDM_MiscFootprint:67068-7041 -> SDM:67068-7041
- J5, J6: footprint SDM_MiscFootprint:CONN23_776087_TEC -> SDM:CONN23_776087_TEC
- LED1, LED2, LED3, LED4: footprint SDM_MiscFootprint:SSFLXH100LID01 -> SDM:SSFLXH100LID01; symbol SDM_LED:SSF-LXH100LID-01 -> SDM:SSF-LXH100LID-01
- U6: footprint SDM_MiscFootprint:SOT-5X3 -> SDM:SOT-5X3
- U9: symbol SDM_ADC:TI_ADC128S102 -> SDM:TI_ADC128S102
- Y1: footprint SDM_MiscFootprint:ECX327CDX2096 -> SDM:ECX327CDX2096
