File: 2026/NondimensionalTractionControl/SDM26_NondimensionalTractionControl_V1.1/NondimensionalTractionControl_V1.1.kicad_pcb (KiCad board)
At the start: 4 copper layers, 70 x 35 mm, 63 parts, among them IC1 STM32H743VIT6, IC2 74LVC1G17SE-7, IC3 TLP175A_TPL,E, IC4 SN65HVD230QDR, IC5 TPS259250DRCR, IC6 MIC37100-3.3WS, IC7 TPS2116DRLR, J1 104031-0811, J2 Conn_ARM_SWD_TagConnect_TC203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, J3 USB_B_Micro, J4 SM04B-ULHK-1TA1-ETB_HF_, J5 SM04B-ULHK-1TA1-ETB_HF_, J6 SM04B-ULHK-1TA1-ETB_HF_, U1 USBLC6-2SC6, Y1 ABM3B-8.000MHZ-10-1-U-T

Commit message: Library maintenance
edited some 3dmodles to point to their footprints. edited symbols and footprints to link properly. edited footprint and symbol library names in all projects 2026-2027 to use the same library nick name "SDM" for both  symbol and footprint.
all users must delete their old lib and make a new one named SDM for symbol and footprint.
Parts:
- IC1: footprint SDM_MiscFootprint:QFP50P1600X1600X160-100L -> SDM:QFP50P1600X1600X160-100L
- IC3: footprint SDM_MiscFootprint:TLP266J -> SDM:TLP266J
- IC4: footprint SDM_MiscFootprint:SOIC127P600X175-8L -> SDM:SOIC127P600X175-8L
- IC5: footprint SDM_MiscFootprint:SON50P300X300X100-11L-D -> SDM:SON50P300X300X100-11L-D
- IC7: footprint SDM_MiscFootprint:SOTFL50P160X60-8L -> SDM:SOTFL50P160X60-8L
- J1: footprint SDM_MiscFootprint:1040310811 -> SDM:1040310811
- J4, J5: footprint SDM_MiscFootprint:SM04BULHK1TA1ETBHF -> SDM:SM04BULHK1TA1ETBHF
- LED1, LED2, LED3: footprint SDM_MiscFootprint:LEDC1608X80N -> SDM:LEDC1608X80N
Changed lines of the file:
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@@
 		)
 	)
-	(footprint "SDM_MiscFootprint:SM04BULHK1TA1ETBHF"
+	(footprint "SDM:SM04BULHK1TA1ETBHF"
 		(layer "F.Cu")
 		(at 104.4 130.5 90)
@@
 		)
 	)
-	(footprint "SDM_MiscFootprint:SOIC127P600X175-8L"
+	(footprint "SDM:SOIC127P600X175-8L"
 		(layer "F.Cu")
 		(at 144.2 144)
@@
 		)
 	)
-	(footprint "SDM_MiscFootprint:1040310811"
+	(footprint "SDM:1040310811"
 		(layer "F.Cu")
 		(at 163.644 122.655 90)
@@
 		)
 	)
-	(footprint "SDM_MiscFootprint:SOTFL50P160X60-8L"
+	(footprint "SDM:SOTFL50P160X60-8L"
 		(layer "F.Cu")
 		(at 155.25 136.2695 90)
@@
 		(embedded_fonts no)
 	)
-	(footprint "SDM_MiscFootprint:LEDC1608X80N"
+	(footprint "SDM:LEDC1608X80N"
 		(layer "F.Cu")
 		(at 151.7 116.575)
@@
 		)
 	)
-	(footprint "SDM_MiscFootprint:LEDC1608X80N"
+	(footprint "SDM:LEDC1608X80N"
 		(layer "F.Cu")
 		(at 101.5 117.2 90)
@@
 		)
 	)
-	(footprint "SDM_MiscFootprint:SM04BULHK1TA1ETBHF"
+	(footprint "SDM:SM04BULHK1TA1ETBHF"
 		(layer "F.Cu")
 		(at 104.4 144.2 90)
@@
 		)
 	)
-	(footprint "SDM_MiscFootprint:TLP266J"
+	(footprint "SDM:TLP266J"
 		(layer "F.Cu")
 		(at 152.15 143.9)
@@
 		)
 	)
-	(footprint "SDM_MiscFootprint:SON50P300X300X100-11L-D"
+	(footprint "SDM:SON50P300X300X100-11L-D"
 		(layer "F.Cu")
 		(at 155.249 139.6 180)
@@
 		)
 	)
-	(footprint "SDM_MiscFootprint:QFP50P1600X1600X160-100L"
+	(footprint "SDM:QFP50P1600X1600X160-100L"
 		(layer "F.Cu")
 		(at 129.1 139.9)
@@
 		)
 	)
-	(footprint "SDM_MiscFootprint:LEDC1608X80N"
+	(footprint "SDM:LEDC1608X80N"
 		(layer "F.Cu")
 		(at 155.2 116.6)
