File: 2026/NondimensionalTractionControl/SDM26_NondimensionalTractionControl_V1.1/NondimensionalTractionControl_V1.1.kicad_sch (KiCad schematic)
At the start: 61 parts, among them IC1 STM32H743VIT6, IC2 74LVC1G17SE-7, IC3 TLP175A_TPL,E, IC4 SN65HVD230QDR, IC5 TPS259250DRCR, IC6 MIC37100-3.3WS, IC7 TPS2116DRLR, J1 104031-0811, J2 Conn_ARM_SWD_TagConnect_TC203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, J3 USB_B_Micro, J4 SM04B-ULHK-1TA1-ETB_HF_, J5 SM04B-ULHK-1TA1-ETB_HF_, J6 SM04B-ULHK-1TA1-ETB_HF_, U1 USBLC6-2SC6, Y1 ABM3B-8.000MHZ-10-1-U-T

Commit message: Library maintenance
edited some 3dmodles to point to their footprints. edited symbols and footprints to link properly. edited footprint and symbol library names in all projects 2026-2027 to use the same library nick name "SDM" for both  symbol and footprint.
all users must delete their old lib and make a new one named SDM for symbol and footprint.
Parts:
- D1: footprint SDM_MiscFootprint:SOT65P210X110-3N -> SDM:SOT65P210X110-3N; symbol SDM_ESD:ESDCAN03-2BWY -> SDM:ESDCAN03-2BWY
- FL1: footprint SDM_MiscFootprint:EMIF06MSD02N16 -> SDM:EMIF06MSD02N16
- IC1: footprint SDM_MiscFootprint:QFP50P1600X1600X160-100L -> SDM:QFP50P1600X1600X160-100L; symbol SDM_MICRO_CONTROLLER:STM32H743VIT6 -> SDM:STM32H743VIT6
- IC2: footprint SDM_MiscFootprint:SOT65P210X110-5L -> SDM:SOT65P210X110-5L; symbol SDM_LOGIC:74LVC1G17SE-7 -> SDM:74LVC1G17SE-7
- IC3: footprint SDM_MiscFootprint:TLP266J -> SDM:TLP266J
- IC4: footprint SDM_MiscFootprint:SOIC127P600X175-8L -> SDM:SOIC127P600X175-8L; symbol SDM_CAN:SN65HVD230QDR -> SDM:SN65HVD230QDR
- IC5: footprint SDM_MiscFootprint:SON50P300X300X100-11L-D -> SDM:SON50P300X300X100-11L-D; symbol SDM_EFUSE:TPS259250DRCR -> SDM:TPS259250DRCR
- IC6: footprint SDM_MiscFootprint:SOT230P700X180-4N -> SDM:SOT230P700X180-4N; symbol SDM_VOLTAGE_REGULATORS:MIC37100-3.3WS -> SDM:MIC37100-3.3WS
- IC7: footprint SDM_MiscFootprint:SOTFL50P160X60-8L -> SDM:SOTFL50P160X60-8L; symbol SDM_LOGIC:TPS2116DRLR -> SDM:TPS2116DRLR
- J1: footprint SDM_MiscFootprint:1040310811 -> SDM:1040310811
- J2: footprint SDM_MiscFootprint:Tag-Connect_TC2030-IDC-NL_2x03_P1.27mm_Vertical -> SDM:Tag-Connect_TC2030-IDC-NL_2x03_P1.27mm_Vertical; symbol SDM_JTAG:Conn_ARM_SWD_TagConnect_TC2030-NL -> SDM:Conn_ARM_SWD_TagConnect_TC2030-NL
- J4, J5, J6: footprint SDM_MiscFootprint:SM04BULHK1TA1ETBHF -> SDM:SM04BULHK1TA1ETBHF; symbol SDM_CONNECTOR:SM04B-ULHK-1TA1-ETB_HF_ -> SDM:SM04B-ULHK-1TA1-ETB_HF_
- LED1: footprint SDM_MiscFootprint:LEDC1608X80N -> SDM:LEDC1608X80N; symbol SDM_LED:150060GS75000 -> SDM:150060GS75000
- LED2, LED3: footprint SDM_MiscFootprint:LEDC1608X80N -> SDM:LEDC1608X80N; symbol SDM_LED:150060RS75000 -> SDM:150060RS75000
- Y1: footprint SDM_MiscFootprint:ABM3B -> SDM:ABM3B
