File: 2026/PitotBoard/PitotBoard.kicad_pcb (KiCad board)
At the start: 2 copper layers, 20.8 x 15.7 mm, 6 parts, among them J1 Conn_01x04_Socket, U1 4525DO-DS5AI001DP

Commit message: Library maintenance
edited some 3dmodles to point to their footprints. edited symbols and footprints to link properly. edited footprint and symbol library names in all projects 2026-2027 to use the same library nick name "SDM" for both  symbol and footprint.
all users must delete their old lib and make a new one named SDM for symbol and footprint.
Parts:
- U1: footprint SDM_MiscFootprint:4525DO-DS...P -> SDM:4525DO-DS...P
Changed lines of the file:
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@@
 	(net 7 "unconnected-(U1-NC_2-Pad7)")
 	(net 8 "+3.3V")
-	(footprint "SDM_MiscFootprint:4525DO-DS...P"
+	(footprint "SDM:4525DO-DS...P"
 		(layer "F.Cu")
 		(at 100.7 105.8)
@@
 		)
 		(embedded_fonts no)
-		(model "${SDM_MISC3D}/4525DO-DS5AI001DP.step"
+		(model "${SDM_MISC_3D}/4525DO-DS5AI001DP.step"
 			(offset
 				(xyz -0.1800000044 -1.950000018 5.380000034)
