File: 2026/SteeringWheel/SDM26_SteeringWheel_V1.1/SDM26_SteeringWheel_V1.1.kicad_pcb (KiCad board)
At the start: 4 copper layers, 182.9 x 134 mm, 97 parts, among them IC1 ESP32-S3-WROOM-1-N8R8, IC3 CP2102N-A02-GQFN28, IC4 TLP175A_TPL,E, IC5 MIC37100-3.3WS, IC6 TPS2116DRLR, IC9 SN74AHC1G125DBVR, J1 Conn_01x02, J2 Conn_01x02, J3 ESP_USB, J4 Conn_01x04_Socket, J5 Conn_01x04_Socket, J6 Conn_01x02_Pin, J7 Molex_1040310811, J8 Conn_01x04_Socket, Q1 MMBT2222LT1G, Q2 MMBT2222LT1G, U1 USBLC6-2SC6, U10 EMIF06-MSD02N16, U2 SN65HVD230

Commit message: Library maintenance
edited some 3dmodles to point to their footprints. edited symbols and footprints to link properly. edited footprint and symbol library names in all projects 2026-2027 to use the same library nick name "SDM" for both  symbol and footprint.
all users must delete their old lib and make a new one named SDM for symbol and footprint.
Parts:
- D1: footprint SDM_MiscFootprint:SOT65P210X110-3N -> SDM:SOT65P210X110-3N
- IC1: footprint SDM_MiscFootprint:ESP32S3WROOM1N8R8 -> SDM:ESP32S3WROOM1N8R8
- IC3: footprint SDM_MiscFootprint:QFN50P500X500X80-29N-D -> SDM:QFN50P500X500X80-29N-D
- IC4: footprint SDM_MiscFootprint:TLP266J -> SDM:TLP266J
- IC9: footprint SDM_MiscFootprint:SOT95P280X145-5L -> SDM:SOT95P280X145-5L
- J7: footprint SDM_MiscFootprint:microSD_HC_Molex_104031-0811 -> SDM:microSD_HC_Molex_104031-0811
- LED1, LED2: footprint SDM_MiscFootprint:LEDC1608X80N -> SDM:LEDC1608X80N
- Q2: footprint SDM_MiscFootprint:SOT96P237X111-3N -> SDM:SOT96P237X111-3N
- S1, S2: footprint SDM_MiscFootprint:MHPS2285V -> SDM:MHPS2285V
- U10: footprint SDM_MiscFootprint:UQFN-17-3.5x1.2mm -> SDM:UQFN-17-3.5x1.2mm
- VR4, VR5: footprint SDM_MiscFootprint:P091N2QC20BR10K -> SDM:P091N2QC20BR10K
Changed lines of the file:
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@@
 		)
 	)
-	(footprint "SDM_MiscFootprint:ESP32S3WROOM1N8R8"
+	(footprint "SDM:ESP32S3WROOM1N8R8"
 		(layer "F.Cu")
 		(at 185.75 51.9)
@@
 		)
 	)
-	(footprint "SDM_MiscFootprint:TLP266J"
+	(footprint "SDM:TLP266J"
 		(layer "F.Cu")
 		(at 169.75 170.0998 90)
@@
 		(embedded_fonts no)
 	)
-	(footprint "SDM_MiscFootprint:microSD_HC_Molex_104031-0811"
+	(footprint "SDM:microSD_HC_Molex_104031-0811"
 		(layer "F.Cu")
 		(at 108.2 50.7)
@@
 		)
 	)
-	(footprint "SDM_MiscFootprint:UQFN-17-3.5x1.2mm"
+	(footprint "SDM:UQFN-17-3.5x1.2mm"
 		(layer "F.Cu")
 		(at 108.9 58.3 90)
@@
 		(embedded_fonts no)
 	)
-	(footprint "SDM_MiscFootprint:SOT96P237X111-3N"
+	(footprint "SDM:SOT96P237X111-3N"
 		(layer "F.Cu")
 		(at 124.502 155.0999)
@@
 		)
 	)
-	(footprint "SDM_MiscFootprint:LEDC1608X80N"
+	(footprint "SDM:LEDC1608X80N"
 		(layer "F.Cu")
 		(at 155.1 82.6 90)
@@
 		)
 	)
-	(footprint "SDM_MiscFootprint:MHPS2285V"
+	(footprint "SDM:MHPS2285V"
 		(layer "F.Cu")
 		(at 211.47 53)
@@
 		)
 	)
-	(footprint "SDM_MiscFootprint:LEDC1608X80N"
+	(footprint "SDM:LEDC1608X80N"
 		(layer "F.Cu")
 		(at 131.35 138.1249 180)
@@
 		)
 	)
-	(footprint "SDM_MiscFootprint:P091N2QC20BR10K"
+	(footprint "SDM:P091N2QC20BR10K"
 		(layer "F.Cu")
 		(at 128.1 79.25 180)
@@
 		)
 	)
-	(footprint "SDM_MiscFootprint:MHPS2285V"
+	(footprint "SDM:MHPS2285V"
 		(layer "F.Cu")
 		(at 74.31 53)
@@
 		)
 	)
-	(footprint "SDM_MiscFootprint:P091N2QC20BR10K"
+	(footprint "SDM:P091N2QC20BR10K"
 		(layer "F.Cu")
 		(at 162.68 84.25)
@@
 		)
 	)
-	(footprint "SDM_MiscFootprint:QFN50P500X500X80-29N-D"
+	(footprint "SDM:QFN50P500X500X80-29N-D"
 		(layer "F.Cu")
 		(at 125.6545 160.0124 90)
@@
 		)
 	)
-	(footprint "SDM_MiscFootprint:SOT95P280X145-5L"
+	(footprint "SDM:SOT95P280X145-5L"
 		(layer "F.Cu")
 		(at 112.3 59.5 90)
@@
 		)
 	)
-	(footprint "SDM_MiscFootprint:SOT65P210X110-3N"
+	(footprint "SDM:SOT65P210X110-3N"
 		(layer "F.Cu")
 		(at 162.1 174.4998 90)
