File: 2026/Wheelboard/SDM26_Wheelboard_V1.2/SDM26_Wheelboard_V1.2.kicad_pcb (KiCad board)
At the start: 4 copper layers, 39.5 x 56.5 mm, 80 parts, among them IC1 TPS259250DRCR, IC10 MCP2518FDT-E_SL, IC2 ESP32-S3-WROOM-1-N8R8, IC3 TLP175A_TPL,E, IC4 MIC37100-3.3WS, IC5 TPS2116DRLR, IC6 TLP175A_TPL,E, IC7 ISM330DHCXTR, IC8 CP2102N-A02-GQFN28, IC9 MAX9924UAUB+, J1 Conn_01x04_Socket, J2 Conn_01x04_Socket, J3 Conn_01x04_Socket, J4 Conn_01x04_Socket, J5 Conn_01x02_Socket, J6 ESP_USB, J7 Conn_01x02_Socket, Q1 SOT96P237X111-3N, Q2 SOT96P237X111-3N, U1 SN65HVD230, U2 SN65HVD230, U4 USBLC6-2SC6, Y1 ABM3B-20.000MHZ-10-1-U-T

Commit message: Library maintenance
edited some 3dmodles to point to their footprints. edited symbols and footprints to link properly. edited footprint and symbol library names in all projects 2026-2027 to use the same library nick name "SDM" for both  symbol and footprint.
all users must delete their old lib and make a new one named SDM for symbol and footprint.
Parts:
- D1, D2: footprint SDM_MiscFootprint:SOT65P210X110-3N -> SDM:SOT65P210X110-3N
- IC10: footprint SDM_MiscFootprint:SOIC127P600X175-14L -> SDM:SOIC127P600X175-14L
- IC3, IC6: footprint SDM_MiscFootprint:TLP266J -> SDM:TLP266J
- IC8: footprint SDM_MiscFootprint:QFN50P500X500X80-29N-D -> SDM:QFN50P500X500X80-29N-D
- LED1, LED2, LED3: footprint SDM_MiscFootprint:LEDC1608X80N -> SDM:LEDC1608X80N
Changed lines of the file:
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@@
 		)
 		(embedded_fonts no)
-		(model "${KICAD9_3DMODEL_DIR}/Capacitor_SMD.3dshapes/C_0603_1608Metric.wrl"
+		(model "${SDM_MISC_3D}/KiCad-original/Capacitor_SMD.3dshapes/C_0603_1608Metric.wrl"
 			(offset
 				(xyz 0 0 0)
@@
 		)
 		(embedded_fonts no)
-		(model "${KICAD9_3DMODEL_DIR}/Resistor_SMD.3dshapes/R_0603_1608Metric.wrl"
+		(model "${SDM_MISC_3D}/KiCad-original/Resistor_SMD.3dshapes/R_0603_1608Metric.wrl"
 			(offset
 				(xyz 0 0 0)
@@
 		)
 		(embedded_fonts no)
-		(model "${KICAD9_3DMODEL_DIR}/Resistor_SMD.3dshapes/R_0603_1608Metric.wrl"
+		(model "${SDM_MISC_3D}/KiCad-original/Resistor_SMD.3dshapes/R_0603_1608Metric.wrl"
 			(offset
 				(xyz 0 0 0)
@@
 		)
 		(embedded_fonts no)
-		(model "${KICAD9_3DMODEL_DIR}/Capacitor_SMD.3dshapes/C_0603_1608Metric.wrl"
+		(model "${SDM_MISC_3D}/KiCad-original/Capacitor_SMD.3dshapes/C_0603_1608Metric.wrl"
 			(offset
 				(xyz 0 0 0)
@@
 		)
 	)
-	(footprint "SDM_MiscFootprint:QFN50P500X500X80-29N-D"
+	(footprint "SDM:QFN50P500X500X80-29N-D"
 		(layer "F.Cu")
 		(at 120.3 99.55)
@@
 		)
 		(embedded_fonts no)
-		(model "${KICAD9_3DMODEL_DIR}/Resistor_SMD.3dshapes/R_0603_1608Metric.wrl"
+		(model "${SDM_MISC_3D}/KiCad-original/Resistor_SMD.3dshapes/R_0603_1608Metric.wrl"
 			(offset
 				(xyz 0 0 0)
@@
 		)
 		(embedded_fonts no)
-		(model "${KICAD9_3DMODEL_DIR}/Resistor_SMD.3dshapes/R_0603_1608Metric.wrl"
+		(model "${SDM_MISC_3D}/KiCad-original/Resistor_SMD.3dshapes/R_0603_1608Metric.wrl"
 			(offset
 				(xyz 0 0 0)
@@
 		)
 	)
-	(footprint "SDM_MiscFootprint:SOIC127P600X175-14L"
+	(footprint "SDM:SOIC127P600X175-14L"
 		(layer "F.Cu")
 		(at 118.57825 114.85 90)
@@
 		)
 		(embedded_fonts no)
-		(model "${KICAD9_3DMODEL_DIR}/Resistor_SMD.3dshapes/R_0603_1608Metric.wrl"
+		(model "${SDM_MISC_3D}/KiCad-original/Resistor_SMD.3dshapes/R_0603_1608Metric.wrl"
 			(offset
 				(xyz 0 0 0)
@@
 		)
 		(embedded_fonts no)
-		(model "${KICAD9_3DMODEL_DIR}/Capacitor_SMD.3dshapes/C_0603_1608Metric.wrl"
+		(model "${SDM_MISC_3D}/KiCad-original/Capacitor_SMD.3dshapes/C_0603_1608Metric.wrl"
 			(offset
 				(xyz 0 0 0)
@@
 		)
 	)
-	(footprint "SDM_MiscFootprint:LEDC1608X80N"
+	(footprint "SDM:LEDC1608X80N"
 		(layer "F.Cu")
 		(at 25.46 131.15)
@@
 		)
 		(embedded_fonts no)
-		(model "${KICAD9_3DMODEL_DIR}/Capacitor_SMD.3dshapes/C_0603_1608Metric.wrl"
+		(model "${SDM_MISC_3D}/KiCad-original/Capacitor_SMD.3dshapes/C_0603_1608Metric.wrl"
 			(offset
 				(xyz 0 0 0)
@@
 		)
 	)
-	(footprint "SDM_MiscFootprint:LEDC1608X80N"
+	(footprint "SDM:LEDC1608X80N"
 		(layer "F.Cu")
 		(at 126.6 107.5 180)
@@
 		)
 		(embedded_fonts no)
-		(model "${KICAD9_3DMODEL_DIR}/Capacitor_SMD.3dshapes/C_0603_1608Metric.wrl"
+		(model "${SDM_MISC_3D}/KiCad-original/Capacitor_SMD.3dshapes/C_0603_1608Metric.wrl"
 			(offset
 				(xyz 0 0 0)
@@
 		(embedded_fonts no)
 	)
-	(footprint "SDM_MiscFootprint:LEDC1608X80N"
+	(footprint "SDM:LEDC1608X80N"
 		(layer "B.Cu")
 		(at 122.5 100.75 -90)
@@
 		)
 	)
-	(footprint "SDM_MiscFootprint:TLP266J"
+	(footprint "SDM:TLP266J"
 		(layer "B.Cu")
 		(at 130.97825 121.2)
@@
 		)
 	)
-	(footprint "SDM_MiscFootprint:SOT65P210X110-3N"
+	(footprint "SDM:SOT65P210X110-3N"
 		(layer "B.Cu")
 		(at 136.37825 120.5 -90)
@@
 		)
 		(embedded_fonts no)
-		(model "${KICAD9_3DMODEL_DIR}/Resistor_SMD.3dshapes/R_0603_1608Metric.wrl"
+		(model "${SDM_MISC_3D}/KiCad-original/Resistor_SMD.3dshapes/R_0603_1608Metric.wrl"
 			(offset
 				(xyz 0 0 0)
@@
 		)
 	)
-	(footprint "SDM_MiscFootprint:SOT65P210X110-3N"
+	(footprint "SDM:SOT65P210X110-3N"
 		(layer "B.Cu")
 		(at 111.07825 119.6 -90)
@@
 		(embedded_fonts no)
 	)
-	(footprint "SDM_MiscFootprint:TLP266J"
+	(footprint "SDM:TLP266J"
 		(layer "B.Cu")
 		(at 113.52825 115.25 180)
@@
 		)
 		(embedded_fonts no)
-		(model "${KICAD9_3DMODEL_DIR}/Resistor_SMD.3dshapes/R_0603_1608Metric.wrl"
+		(model "${SDM_MISC_3D}/KiCad-original/Resistor_SMD.3dshapes/R_0603_1608Metric.wrl"
 			(offset
 				(xyz 0 0 0)
