File: 2026/Wheelboard/SDM26_Wheelboard_V2.1/SDM26_Wheelboard_V2.1.kicad_sch (KiCad schematic)
At the start: 69 parts, among them IC1 MCP2518FDT-H_QBB, IC2 ESP32-S3-WROOM-1-N8R8, IC3 TLP175A_TPL,E, IC4 MIC37100-3.3WS, IC5 TPS2116DRLR, IC6 TLP175A_TPL,E, IC8 CP2102N-A02-GQFN28, IC9 MAX9924UAUB+, J1 Conn_01x04_Socket, J2 Conn_01x04_Socket, J3 Conn_01x04_Socket, J4 Conn_01x04_Socket, J5 Conn_01x02_Socket, J6 ESP_USB, J7 Conn_01x02_Socket, Q1 SOT96P237X111-3N, Q2 SOT96P237X111-3N, U1 SN65HVD230, U2 SN65HVD230, U4 USBLC6-2SC6, Y1 ABM3B-20.000MHZ-10-1-U-T

Commit message: Library maintenance
edited some 3dmodles to point to their footprints. edited symbols and footprints to link properly. edited footprint and symbol library names in all projects 2026-2027 to use the same library nick name "SDM" for both  symbol and footprint.
all users must delete their old lib and make a new one named SDM for symbol and footprint.
Parts:
- D1, D2: footprint SDM_MiscFootprint:SOT65P210X110-3N -> SDM:SOT65P210X110-3N; symbol SDM_ESD:ESDCAN03-2BWY -> SDM:ESDCAN03-2BWY
- IC1: footprint SDM_MiscFootprint:SON65P300X450X90-15L-D -> SDM:SON65P300X450X90-15L-D
- IC2: footprint SDM_MiscFootprint:ESP32S3WROOM1N8R8 -> SDM:ESP32S3WROOM1N8R8
- IC3, IC6: footprint SDM_MiscFootprint:TLP266J -> SDM:TLP266J
- IC4: footprint SDM_MiscFootprint:SOT230P700X180-4N -> SDM:SOT230P700X180-4N; symbol SDM_VOLTAGE_REGULATORS:MIC37100-3.3WS -> SDM:MIC37100-3.3WS
- IC5: footprint SDM_MiscFootprint:SOTFL50P160X60-8L -> SDM:SOTFL50P160X60-8L; symbol SDM_LOGIC:TPS2116DRLR -> SDM:TPS2116DRLR
- IC8: footprint SDM_MiscFootprint:QFN50P500X500X80-29N-D -> SDM:QFN50P500X500X80-29N-D; symbol USBUART:CP2102N-A02-GQFN28 -> SDM:CP2102N-A02-GQFN28
- IC9: footprint SDM_MiscFootprint:SOP50P490X110-10L -> SDM:SOP50P490X110-10L; symbol SDM_SENSOR:MAX9924UAUB+ -> SDM:MAX9924UAUB+
- LED1, LED3: footprint SDM_MiscFootprint:LEDC1608X80N -> SDM:LEDC1608X80N; symbol SDM_LED:150060RS75000 -> SDM:150060RS75000
- LED2: footprint SDM_MiscFootprint:LEDC1608X80N -> SDM:LEDC1608X80N; symbol SDM_LED:150060VS75000 -> SDM:150060VS75000
- Q1, Q2: footprint SDM_MiscFootprint:SOT96P237X111-3N -> SDM:SOT96P237X111-3N
- Y1: footprint SDM_MiscFootprint:ABM3B -> SDM:ABM3B; symbol SDM_CRYSTAL_HSE:ABM3B-20.000MHZ-10-1-U-T -> SDM:ABM3B-20.000MHZ-10-1-U-T
