File: 2027/SDM27_CANSniffer/CANSniffer V1/ESP-C5.kicad_sch (KiCad schematic)
At the start: 62 parts, among them J1 WEIPU SA12 7PIN, J2 USB_C_Receptacle_USB2.0_16P, SW1 SW_Push, SW2 SW_Push, U1 ESP32-C5HR8, U2 GD25Q32ESIG, U3 TPS2121RUXR, U4 TPS62901RPJR, U5 TCAN3403DRBRQ1, U6 TLP175A_TPL,E, U7 USBLC6-2SC6, Y3 CX1612DB48000D0FPJC1

Commit message: CAN sniffer updated
updated CAN sniffer
Connections:
- net GND: now also J2.A12 (GND), J2.B1 (GND), J2.B12 (GND)
Other:
- note added: "User Interface"
- moved on the sheet: C19, J1, J2, R5, R6, U7

Commit message: Library maintenance
edited some 3dmodles to point to their footprints. edited symbols and footprints to link properly. edited footprint and symbol library names in all projects 2026-2027 to use the same library nick name "SDM" for both  symbol and footprint.
all users must delete their old lib and make a new one named SDM for symbol and footprint.
Parts:
- D2: symbol SDM_ESD:ESDCAN03-2BWY -> SDM:ESDCAN03-2BWY
- J2: symbol SDM_USB:USB_C_Receptacle_USB2.0_16P -> SDM:USB_C_Receptacle_USB2.0_16P
- LED2: symbol SDM_LED:150060RS75000 -> SDM:150060RS75000
- U1: footprint SDM_Misc:QFN40P600X600X90-49N-D -> SDM:QFN40P600X600X90-49N-D
- U3: footprint SDM_Misc:TPS2121RUXR -> SDM:TPS2121RUXR
- U6: symbol SDM_OPTOCOUPLERS:TLP175A_TPL,E -> SDM:TLP175A_TPL,E
