File: 2027/SDM27_CANSniffer/CANSniffer V1/_restore_backup_2026-10-19T12-15-33-923/ESP-C5-CAN SNIFFER.kicad_pcb (KiCad board)
At the start: 4 copper layers, 80 x 86 mm, 73 parts, among them J1 WEIPU SA12 7PIN, J2 USB_C_Receptacle_USB2.0_16P, J3 ELECROW_2.8_ILI9341, J4 WEIPU SA12 7PIN, SW1 SW_Push, SW2 SW_Push, SW3 RotaryEncoder_Bourns_PEC11R-S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, U1 ESP32-C5HR8, U2 GD25Q32ESIG, U3 TPS2121RUXR, U4 TPS62901RPJR, U5 TCAN3403DRBRQ1, U6 TLP175A_TPL,E, U7 USBLC6-2SC6, Y3 CX1612DB48000D0FPJC1

Commit message: Library maintenance
edited some 3dmodles to point to their footprints. edited symbols and footprints to link properly. edited footprint and symbol library names in all projects 2026-2027 to use the same library nick name "SDM" for both  symbol and footprint.
all users must delete their old lib and make a new one named SDM for symbol and footprint.
Parts:
- LED2: footprint SDM_MISC:LEDC1608X80N -> SDM:LEDC1608X80N
- SW3: footprint SDM_MISC:XDCR_PEC11R-4220F-S0024 -> SDM:XDCR_PEC11R-4220F-S0024
- U1: footprint SDM_MISC:QFN40P600X600X90-49N-D -> SDM:QFN40P600X600X90-49N-D
- U3: footprint SDM_MISC:TPS2121RUXR -> SDM:TPS2121RUXR
- U4: footprint SDM_MISC:TPS62901RPJR -> SDM:TPS62901RPJR
- U6: footprint SDM_MISC:TLP266J -> SDM:TLP266J
Changed lines of the file:
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@@
 		)
 	)
-	(footprint "SDM_MISC:TLP266J"
+	(footprint "SDM:TLP266J"
 		(layer "F.Cu")
 		(at 198.26 105.99 180)
@@
 		)
 	)
-	(footprint "SDM_MISC:XDCR_PEC11R-4220F-S0024"
+	(footprint "SDM:XDCR_PEC11R-4220F-S0024"
 		(layer "F.Cu")
 		(at 255.55 120 180)
@@
 		)
 	)
-	(footprint "SDM_MISC:TPS2121RUXR"
+	(footprint "SDM:TPS2121RUXR"
 		(layer "F.Cu")
 		(at 231.25 55.9 -90)
@@
 		)
 		(embedded_fonts no)
-		(model "C:/Users/lazee/OneDrive/Documents/pcb-dev/MiscLibraries/SDM_Misc3D/TPS2121RUXR.stp"
+		(model "${SDM_MISC_3D}/TPS2121RUXR.stp"
 			(offset
 				(xyz 0 0 0)
@@
 		)
 		(embedded_fonts no)
-		(model "CX1612DB48000D0FPJC1.stp"
+		(model "${SDM_MISC_3D}/CX1612DB48000D0FPJC1.stp"
 			(offset
 				(xyz 0 0 0)
@@
 		)
 		(embedded_fonts no)
-		(model "TCAN3403DRBRQ1.stp"
+		(model "${SDM_MISC_3D}/TCAN3403DRBRQ1.stp"
 			(offset
 				(xyz 0 0 0)
@@
 		)
 		(embedded_fonts no)
-		(model "F1C1-201612-2R2M.stp"
+		(model "${SDM_MISC_3D}/F1C1-201612-2R2M.stp"
 			(offset
 				(xyz -0.1899999948 -0.9100000126 0.05999999776)
@@
 		)
 	)
-	(footprint "SDM_MISC:TPS62901RPJR"
+	(footprint "SDM:TPS62901RPJR"
 		(layer "F.Cu")
 		(at 237.9 62.1)
@@
 		)
 		(embedded_fonts no)
-		(model "TPS62901RPJR.stp"
+		(model "${SDM_MISC_3D}/TPS62901RPJR.stp"
 			(offset
 				(xyz 0 0 0)
@@
 		)
 	)
-	(footprint "SDM_MISC:LEDC1608X80N"
+	(footprint "SDM:LEDC1608X80N"
 		(layer "F.Cu")
 		(at 256.46 67.22)
@@
 		)
 	)
-	(footprint "SDM_MISC:QFN40P600X600X90-49N-D"
+	(footprint "SDM:QFN40P600X600X90-49N-D"
 		(layer "F.Cu")
 		(at 220.25 95.5)
@@
 		)
 		(embedded_fonts no)
-		(model "ESP32-C5HR8.stp"
+		(model "${SDM_MISC_3D}/ESP32-C5HR8.stp"
 			(offset
 				(xyz 0 0 0)
