File: 2027/SDM27_CANSplitter/SDM27_CANSplitter_V1.0/SDM27_CANSplitter_V1.0.kicad_pcb (KiCad board)
At the start: 2 copper layers, 46 x 11.5 mm, 10 parts, among them J1 SM04B-ULHK-1TA1-ETB_HF_, J2 SM04B-ULHK-1TA1-ETB_HF_, J3 SM04B-ULHK-1TA1-ETB_HF_, J4 SM04B-ULHK-1TA1-ETB_HF_, J5 SM04B-ULHK-1TA1-ETB_HF_, J6 SM04B-ULHK-1TA1-ETB_HF_

Commit message: Library maintenance
edited some 3dmodles to point to their footprints. edited symbols and footprints to link properly. edited footprint and symbol library names in all projects 2026-2027 to use the same library nick name "SDM" for both  symbol and footprint.
all users must delete their old lib and make a new one named SDM for symbol and footprint.
Parts:
- J1, J2, J3: footprint SDM_MiscFootprint:SM04BULHK1TA1ETBHF -> SDM:SM04BULHK1TA1ETBHF
- LED1: footprint SDM_MiscFootprint:LEDC1608X80N -> SDM:LEDC1608X80N
Changed lines of the file:
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@@
 		(embedded_fonts no)
 	)
-	(footprint "SDM_MiscFootprint:SM04BULHK1TA1ETBHF"
+	(footprint "SDM:SM04BULHK1TA1ETBHF"
 		(layer "F.Cu")
 		(at 119 56)
@@
 		)
 	)
-	(footprint "SDM_MiscFootprint:LEDC1608X80N"
+	(footprint "SDM:LEDC1608X80N"
 		(layer "F.Cu")
 		(at 138.9 52 180)
@@
 		(embedded_fonts no)
 	)
-	(footprint "SDM_MiscFootprint:SM04BULHK1TA1ETBHF"
+	(footprint "SDM:SM04BULHK1TA1ETBHF"
 		(layer "F.Cu")
 		(at 107 56)
@@
 		)
 	)
-	(footprint "SDM_MiscFootprint:SM04BULHK1TA1ETBHF"
+	(footprint "SDM:SM04BULHK1TA1ETBHF"
 		(layer "F.Cu")
 		(at 131 56)
