File: 2027/SDM27_SlipAngle/SensorMountV2/SensorMountV2.kicad_sch (KiCad schematic)
At the start: 23 parts, among them IC1 ADNS-3050, IC2 ADNS-3050, J2 Conn_01x07_Pin

Commit message: Library maintenance
edited some 3dmodles to point to their footprints. edited symbols and footprints to link properly. edited footprint and symbol library names in all projects 2026-2027 to use the same library nick name "SDM" for both  symbol and footprint.
all users must delete their old lib and make a new one named SDM for symbol and footprint.
Parts:
- IC1, IC2: footprint ADNS3050 -> SDM:ADNS3050; symbol SDM_MISC:ADNS-3050 -> SDM:ADNS-3050
Changed lines of the file:
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@@
 	)
 	(symbol
-		(lib_id "SDM_MISC:ADNS-3050")
+		(lib_id "SDM:ADNS-3050")
 		(at 119.38 113.03 0)
 		(unit 1)
@@
 			)
 		)
-		(property "Footprint" "ADNS3050"
+		(property "Footprint" "SDM:ADNS3050"
 			(at 146.05 207.95 0)
 			(hide yes)
@@
 	)
 	(symbol
-		(lib_id "SDM_MISC:ADNS-3050")
+		(lib_id "SDM:ADNS-3050")
 		(at 119.38 142.24 0)
 		(unit 1)
@@
 			)
 		)
-		(property "Footprint" "ADNS3050"
+		(property "Footprint" "SDM:ADNS3050"
 			(at 146.05 237.16 0)
 			(hide yes)
